File: circuit-boards/CAN-IO-expander/CAN-IO-expander.kicad_pcb (KiCad board)
At the start: 2 copper layers, 120 parts, among them J1 PROG, J2 CAN1, J3 CAN1, J4 Conn_01x06_Pin, J5 Conn_01x03_Pin, J6 Conn_01x06_Pin, J7 Conn_01x03_Pin, J8 Power, U1 RP2350_60QFN, U10 24LC01BT-I/OT, U11 MCP6006UT-E/OT, U2 W25Q128JVP, U3 12MHz, U4 MCP2518FDT-H/SL, U5 MCP2558FD, U6 4MHz, U7 TPS613222ADBVR, U8 MCP6006UT-E/OT, U9 LMR54410FDBVR

Commit message: Changed to 1 encoder, all connectors to SMD right angle SL
Signed-off-by: Scott Berman <sgberman1@gmail.com>
Parts:
- removed C22: 330uF-35V-20%-10mm, Capacitor_THT:CP_Radial_D10.0mm_P5.00mm
- removed C29, C33, C40, C41, C42, C43, C44: 1nF-50V-5%-0603, Capacitor_SMD:C_0603_1608Metric
- removed C31: 0.1uF-25V-10%-0603, Capacitor_SMD:C_0603_1608Metric
- removed D10, D11, D12, D5, D8: BAV199, Package_TO_SOT_SMD:SOT-23
- removed J7: Conn_01x03_Pin, CAN-IO-expander:70555-0002
- removed J8: Power, CAN-IO-expander:Wago-2604-3102
- removed R11, R14, R34, R35, R36, R37, R38: 1.00k-1%-0603, Resistor_SMD:R_0603_1608Metric
- removed R24, R29, R30, R31, R32: 100R-1%-0603, Resistor_SMD:R_0603_1608Metric
- removed R33: 1.00M-1%-0603, Resistor_SMD:R_0603_1608Metric
- removed R39: 2.00k-1%-0603, Resistor_SMD:R_0603_1608Metric
- removed U8: MCP6006UT-E/OT, Package_TO_SOT_SMD:SOT-23-5
- C10, C11, C12, C13, C14, C15, C17, C18, C19, C20, C21, C26, C27, C30, C34, C35, C37, C6, C7, C8, C9, D2, R13, R16, R7, R8, U5: moved to B.Cu
- J2, J3: footprint CAN-IO-expander:70555-0001 -> CAN-IO-expander:Molex-70634-0036
- J4: value Conn_01x06_Pin -> 12V; footprint CAN-IO-expander:70555-0005 -> CAN-IO-expander:Molex-70634-0038
- J5: value Conn_01x03_Pin -> POT; footprint CAN-IO-expander:70555-0002 -> CAN-IO-expander:Molex-70634-0037
- J6: value Conn_01x06_Pin -> ENCODER; footprint CAN-IO-expander:70555-0005 -> CAN-IO-expander:Molex-70634-0039
- moved C23 337.8 mm to (263.9, 91.9), turned to -90 degrees
- moved C24 336.6 mm to (262.4, 91.9), turned to -90 degrees
- moved C25 333.4 mm to (258.1, 87.4), turned to -90 degrees
- moved R13 327.1 mm to (255.8, 87.6), turned to 90 degrees
- moved D4 325.9 mm to (262.9, 87.6), turned to 180 degrees
- moved R7 324.9 mm to (254.3, 87.6), turned to -90 degrees
- moved R16 324.6 mm to (252.7, 87.6), turned to -90 degrees
- moved U7 324.1 mm to (259.8, 91.9), turned to 90 degrees
- moved R8 322.2 mm to (251.2, 87.6), turned to 90 degrees
- moved U9 321.6 mm to (255.5, 87.4), turned to -90 degrees
- moved L3 313.7 mm to (254.5, 94.5), turned to -90 degrees
- moved C38 312.8 mm to (252.0, 87.4), turned to -90 degrees
- moved L2 310.7 mm to (259.8, 96.5), turned to 90 degrees
- moved D3 310.6 mm to (248.4, 89.7), turned to -90 degrees
- moved C18 309.7 mm to (256.8, 97.0), turned to 90 degrees
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Connections:
- J4 pad 2: +5V_EXT -> GND
- J4 pad 3: /QA0 -> /V_{BAT}
- J4 pad 4: /QB0 -> /V_{BAT}
- J6 pad 1: GND -> /PWM_IN0
- J6 pad 2: +5V_EXT -> /QB0
- J6 pad 3: /QA1 -> /QA0
- J6 pad 4: /QB1 -> +5V_EXT
- J6 pad 5: /PWM_IN1 -> GND
- U1 pad 15: /DI30 -> unconnected-(U1-GPIO11-Pad15)
- U1 pad 17: /DI30 -> unconnected-(U1-GPIO13-Pad17)
- U1 pad 31: /DI31 -> unconnected-(U1-GPIO19-Pad31)
- U1 pad 32: /DI11 -> unconnected-(U1-GPIO20-Pad32)
- U1 pad 33: /DI31 -> unconnected-(U1-GPIO21-Pad33)
- U1 pad 34: /DI01 -> unconnected-(U1-GPIO22-Pad34)
- U1 pad 35: /DI21 -> unconnected-(U1-GPIO23-Pad35)
- U1 pad 37: /DI21 -> unconnected-(U1-GPIO25-Pad37)
- U1 pad 41: /AIN1_ADC -> unconnected-(U1-GPIO27_ADC1-Pad41)
Other:
- board outline added: 71.1 x 38.1 mm
