File: circuit-boards/CAN-IO-expander/in_out.kicad_sch (KiCad schematic)
At the start: 24 parts, among them U11 MCP6006UT-E/OT

Commit message: Changed to 1 encoder, all connectors to SMD right angle SL
Signed-off-by: Scott Berman <sgberman1@gmail.com>
Parts:
- removed C41: 1nF-50V-5%-0603, Capacitor_SMD:C_0603_1608Metric, symbol Device:C_Small_US
- removed D11: BAV199, Package_TO_SOT_SMD:SOT-23, symbol CAN-IO-expander:BAV199
- removed R14: 1.00k-1%-0603, Resistor_SMD:R_0603_1608Metric, symbol Device:R_US
- removed R24: 100R-1%-0603, Resistor_SMD:R_0603_1608Metric, symbol Device:R_US
