File: circuit-boards/Pico-CAN/Pico-CAN.kicad_sch (KiCad schematic)
At the start: 18 parts, among them J1 CAN1, J2 CAN1, J3 Expansion, U1 4.0 MHz, U2 MCP2558FD, U3 MCP2518FDT-H/SL

Commit message: Minor update to PicoCAN. Add JLC assembly docs
Signed-off-by: Scott Berman <sgberman1@gmail.com>
Parts:
- C1, C2, C3, C4, C5: JLCPCB C519981 -> (none); LCSC Part # (none) -> C519981
- D1: JLCPCB C2984756 -> (none); LCSC Part # (none) -> C2984756
- R1: JLCPCB C114555 -> (none); LCSC Part # (none) -> C114555
- U1: JLCPCB C2901552 -> (none); LCSC Part # (none) -> C2901552
- U2: JLCPCB C124015 -> (none); LCSC Part # (none) -> C124015
- U3: JLCPCB C626759 -> (none); LCSC Part # (none) -> C626759
Changed lines of the file:
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@@
 			)
 		)
-		(property "JLCPCB" "C519981"
+		(property "JLCPCB" ""
+			(at 289.56 83.82 0)
+			(effects
+				(font
+					(size 1.27 1.27)
+				)
+				(hide yes)
+			)
+		)
+		(property "LCSC Part #" "C519981"
 			(at 289.56 83.82 0)
 			(effects
@@
 			)
 		)
-		(property "JLCPCB" "C2901552"
+		(property "LCSC Part #" "C2901552"
 			(at 186.69 146.05 0)
 			(effects
@@
 			)
 		)
-		(property "JLCPCB" "C519981"
+		(property "JLCPCB" ""
+			(at 173.99 166.37 0)
+			(effects
+				(font
+					(size 1.27 1.27)
+				)
+				(hide yes)
+			)
+		)
+		(property "LCSC Part #" "C519981"
 			(at 173.99 166.37 0)
 			(effects
@@
 			)
 		)
-		(property "JLCPCB" "C114555"
+		(property "JLCPCB" ""
+			(at 71.12 87.63 0)
+			(effects
+				(font
+					(size 1.27 1.27)
+				)
+				(hide yes)
+			)
+		)
+		(property "LCSC Part #" "C114555"
 			(at 71.12 87.63 0)
 			(effects
@@
 			)
 		)
-		(property "JLCPCB" "C124015"
+		(property "JLCPCB" ""
+			(at 298.45 106.68 0)
+			(effects
+				(font
+					(size 1.27 1.27)
+				)
+				(hide yes)
+			)
+		)
+		(property "LCSC Part #" "C124015"
 			(at 298.45 106.68 0)
 			(effects
@@
 			)
 		)
-		(property "JLCPCB" "C519981"
+		(property "JLCPCB" ""
+			(at 214.63 99.06 0)
+			(effects
+				(font
+					(size 1.27 1.27)
+				)
+				(hide yes)
+			)
+		)
+		(property "LCSC Part #" "C519981"
 			(at 214.63 99.06 0)
 			(effects
@@
 			)
 		)
-		(property "JLCPCB" "C519981"
+		(property "JLCPCB" ""
+			(at 71.12 97.79 0)
+			(effects
+				(font
+					(size 1.27 1.27)
+				)
+				(hide yes)
+			)
+		)
+		(property "LCSC Part #" "C519981"
 			(at 71.12 97.79 0)
 			(effects
@@
 			)
 		)
-		(property "JLCPCB" "C2984756"
+		(property "JLCPCB" ""
+			(at 335.28 123.19 90)
+			(effects
+				(font
+					(size 1.27 1.27)
+				)
+				(hide yes)
+			)
+		)
+		(property "LCSC Part #" "C2984756"
 			(at 335.28 123.19 90)
 			(effects
@@
 			)
 		)
-		(property "JLCPCB" "C519981"
+		(property "JLCPCB" ""
+			(at 308.61 83.82 0)
+			(effects
+				(font
+					(size 1.27 1.27)
+				)
+				(hide yes)
+			)
+		)
+		(property "LCSC Part #" "C519981"
 			(at 308.61 83.82 0)
 			(effects
@@
 			)
 		)
-		(property "JLCPCB" "C626759 "
+		(property "JLCPCB" ""
 			(at 223.52 118.11 0)
 			(effects
+				(font
+					(size 1.27 1.27)
+				)
+				(hide yes)
+			)
+		)
+		(property "LCSC Part #" "C626759 "
+			(at 223.52 118.11 0)
+			(effects

Commit message: Checkin post review
Signed-off-by: Scott Berman <sgberman1@gmail.com>
Parts:
- D1: now not fitted
- renumbered C3 to C2, C2 to C3, J3 to J1, J1 to J2, J2 to J3, U2 to U1, U1 to U2
Connections:
- net START_OF_FRAME: now also A1.21 (GPIO16); no longer A1.22 (GPIO17)
- net ~{CAN_IRQ}: now also A1.22 (GPIO17); no longer A1.32 (GPIO27_ADC1)
Changed lines of the file:
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@@
 	)
 	(no_connect
-		(at 154.94 102.87)
+		(at 154.94 130.81)
 	)
 	(wire
@@
 	(wire
 		(pts
-			(xy 46.99 123.19) (xy 52.07 123.19)
+			(xy 154.94 102.87) (xy 189.23 102.87)
 		)
 		(stroke
@@
 	(wire
 		(pts
-			(xy 300.99 99.06) (xy 300.99 104.14)
+			(xy 46.99 123.19) (xy 52.07 123.19)
 		)
 		(stroke
@@
 	(wire
 		(pts
-			(xy 186.69 123.19) (xy 186.69 130.81)
+			(xy 300.99 99.06) (xy 300.99 104.14)
 		)
 		(stroke
@@
 	(wire
 		(pts
-			(xy 154.94 105.41) (xy 189.23 105.41)
-		)
-		(stroke
-			(width 0)
-			(type default)
-		)
-	)
-	(wire
-		(pts
 			(xy 46.99 128.27) (xy 52.07 128.27)
 		)
@@
 	(wire
 		(pts
+			(xy 186.69 105.41) (xy 154.94 105.41)
+		)
+		(stroke
+			(width 0)
+			(type default)
+		)
+	)
+	(wire
+		(pts
 			(xy 195.58 151.13) (xy 205.74 151.13)
 		)
@@
 	(wire
 		(pts
-			(xy 67.31 113.03) (xy 67.31 120.65)
+			(xy 189.23 102.87) (xy 189.23 87.63)
 		)
 		(stroke
@@
 	(wire
 		(pts
-			(xy 350.52 113.03) (xy 356.87 113.03)
+			(xy 67.31 113.03) (xy 67.31 120.65)
 		)
 		(stroke
@@
 	(wire
 		(pts
-			(xy 189.23 105.41) (xy 189.23 87.63)
+			(xy 350.52 113.03) (xy 356.87 113.03)
 		)
 		(stroke
@@
 	(wire
 		(pts
-			(xy 238.76 113.03) (xy 287.02 113.03)
+			(xy 186.69 123.19) (xy 186.69 105.41)
 		)
 		(stroke
@@
 	(wire
 		(pts
-			(xy 154.94 130.81) (xy 186.69 130.81)
+			(xy 238.76 113.03) (xy 287.02 113.03)
 		)
 		(stroke
@@
 		)
 	)
-	(label "START_OF_FRAME"
-		(at 157.48 105.41 0)
-		(effects
-			(font
-				(size 1.27 1.27)
-			)
-			(justify left bottom)
-		)
-	)
 	(label "GPIO3"
 		(at 109.22 107.95 180)
@@
 	)
 	(label "~{CAN_IRQ}"
-		(at 157.48 130.81 0)
+		(at 157.48 105.41 0)
 		(effects
 			(font
@@
 		)
 	)
+	(label "START_OF_FRAME"
+		(at 157.48 102.87 0)
+		(effects
+			(font
+				(size 1.27 1.27)
+			)
+			(justify left bottom)
+		)
+	)
 	(label "GPIO14"
 		(at 69.85 140.97 0)
@@
 		(on_board yes)
 		(dnp no)
-		(property "Reference" "C2"
+		(property "Reference" "C3"
 			(at 292.1 82.6769 0)
 			(effects
@@
 			(project "Pico-CAN"
 				(path "/7933eff1-4657-450a-9155-0a77075ba053"
-					(reference "C2")
+					(reference "C3")
 					(unit 1)
 				)
@@
 		(dnp no)
 		(fields_autoplaced yes)
-		(property "Reference" "U1"
+		(property "Reference" "U2"
 			(at 198.12 144.7098 0)
 			(effects
@@
 			(project ""
 				(path "/7933eff1-4657-450a-9155-0a77075ba053"
-					(reference "U1")
+					(reference "U2")
 					(unit 1)
 				)
@@
 		(on_board yes)
 		(dnp no)
-		(property "Reference" "C3"
+		(property "Reference" "C2"
 			(at 171.45 165.2269 0)
 			(effects
@@
 			(project "Pico-CAN"
 				(path "/7933eff1-4657-450a-9155-0a77075ba053"
-					(reference "C3")
+					(reference "C2")
 					(unit 1)
 				)
@@
 		(dnp no)
 		(fields_autoplaced yes)
-		(property "Reference" "U2"
+		(property "Reference" "U1"
 			(at 300.5933 120.65 0)
 			(effects
@@
 			(project ""
 				(path "/7933eff1-4657-450a-9155-0a77075ba053"
-					(reference "U2")
+					(reference "U1")
 					(unit 1)
 				)
@@
 		(on_board yes)
 		(dnp no)
-		(property "Reference" "J1"
+		(property "Reference" "J2"
 			(at 363.22 110.4899 0)
 			(effects
@@
 			(project "Pico-CAN"
 				(path "/7933eff1-4657-450a-9155-0a77075ba053"
-					(reference "J1")
+					(reference "J2")
 					(unit 1)
 				)
@@
 		)
 		(pin "7"
+			(alternate "GPIO5")
 		)
 		(pin "1"
@@
 		(in_bom yes)
 		(on_board yes)
-		(dnp no)
+		(dnp yes)
 		(fields_autoplaced yes)
 		(property "Reference" "D1"
@@
 		(dnp no)
 		(fields_autoplaced yes)
-		(property "Reference" "J3"
+		(property "Reference" "J1"
 			(at 58.42 106.68 0)
 			(effects
@@
 			(project ""
 				(path "/7933eff1-4657-450a-9155-0a77075ba053"
-					(reference "J3")
+					(reference "J1")
 					(unit 1)
 				)
@@
 		(on_board yes)
 		(dnp no)
-		(property "Reference" "J2"
+		(property "Reference" "J3"
 			(at 363.22 118.1099 0)
 			(effects
@@
 			(project "Pico-CAN"
 				(path "/7933eff1-4657-450a-9155-0a77075ba053"
-					(reference "J2")
+					(reference "J3")
 					(unit 1)
 				)

Commit message: Changed oscillator back to ECS5032
Signed-off-by: Scott Berman <sgberman1@gmail.com>
Parts:
- H1, H2, H3, H4: footprint MountingHole:MountingHole_3.5mm -> MountingHole:MountingHole_3.7mm
- U2: footprint Pico-CAN:JLC-OSC-SMD3225-4P -> Pico-CAN:ECS-5032MV; DIST JLCPCB -> Digikey; DIST P/N C2901552 -> XC3114CT-ND; LCSC Part # C2901552 -> (none); MFG Shenzhen SCTF Elec -> ECS Inc.; MFG P/N SX3M4.000M20F30TNN -> ECS-5032MV-40-CN-TR
Changed lines of the file:
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@@
 			)
 		)
-		(property "Footprint" "MountingHole:MountingHole_3.5mm"
+		(property "Footprint" "MountingHole:MountingHole_3.7mm"
 			(at 85.09 217.17 0)
 			(effects
@@
 			)
 		)
-		(property "Footprint" "Pico-CAN:JLC-OSC-SMD3225-4P"
+		(property "Footprint" "Pico-CAN:ECS-5032MV"
 			(at 186.69 146.05 0)
 			(effects
@@
 			)
 		)
-		(property "Datasheet" "Components/JLC-C2901552.pdf"
+		(property "Datasheet" "Components/ECS-5032MV.pdf"
 			(at 186.69 146.05 0)
 			(effects
@@
 			)
 		)
-		(property "MFG" "Shenzhen SCTF Elec"
+		(property "MFG" "ECS Inc."
 			(at 186.69 146.05 0)
 			(effects
@@
 			)
 		)
-		(property "MFG P/N" "SX3M4.000M20F30TNN"
+		(property "MFG P/N" "ECS-5032MV-40-CN-TR"
 			(at 186.69 146.05 0)
 			(effects
@@
 			)
 		)
-		(property "DIST" "JLCPCB"
+		(property "DIST" "Digikey"
 			(at 186.69 146.05 0)
 			(effects
@@
 			)
 		)
-		(property "DIST P/N" " C2901552"
+		(property "DIST P/N" "XC3114CT-ND"
 			(at 186.69 146.05 0)
 			(effects
@@
 			)
 		)
-		(property "LCSC Part #" "C2901552"
+		(property "LCSC Part #" ""
 			(at 186.69 146.05 0)
 			(effects
@@
 			)
 		)
-		(property "Footprint" "MountingHole:MountingHole_3.5mm"
+		(property "Footprint" "MountingHole:MountingHole_3.7mm"
 			(at 85.09 227.33 0)
 			(effects
@@
 			)
 		)
-		(property "Footprint" "MountingHole:MountingHole_3.5mm"
+		(property "Footprint" "MountingHole:MountingHole_3.7mm"
 			(at 85.09 232.41 0)
 			(effects
@@
 			)
 		)
-		(property "Footprint" "MountingHole:MountingHole_3.5mm"
+		(property "Footprint" "MountingHole:MountingHole_3.7mm"
 			(at 85.09 222.25 0)
 			(effects

Commit message: Missed schematic
Signed-off-by: Scott Berman <sgberman1@gmail.com>
Parts:
- removed D1: PESD1CAN, Package_TO_SOT_SMD:SOT-23, symbol Pico-CAN:PESD1CAN
Changed lines of the file:
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@@
 	)
 	(junction
-		(at 332.74 113.03)
-		(diameter 0)
-		(color 0 0 0 0)
-	)
-	(junction
 		(at 49.53 140.97)
 		(diameter 0)
@@
 	)
 	(junction
-		(at 327.66 110.49)
-		(diameter 0)
-		(color 0 0 0 0)
-	)
-	(junction
 		(at 67.31 128.27)
 		(diameter 0)
@@
 	(wire
 		(pts
-			(xy 309.88 110.49) (xy 327.66 110.49)
+			(xy 309.88 110.49) (xy 353.06 110.49)
 		)
 		(stroke
@@
 	(wire
 		(pts
-			(xy 327.66 110.49) (xy 353.06 110.49)
-		)
-		(stroke
-			(width 0)
-			(type default)
-		)
-	)
-	(wire
-		(pts
 			(xy 46.99 120.65) (xy 52.07 120.65)
 		)
@@
 	(wire
 		(pts
-			(xy 309.88 113.03) (xy 332.74 113.03)
+			(xy 309.88 113.03) (xy 350.52 113.03)
 		)
 		(stroke
@@
 	(wire
 		(pts
-			(xy 332.74 113.03) (xy 332.74 119.38)
-		)
-		(stroke
-			(width 0)
-			(type default)
-		)
-	)
-	(wire
-		(pts
 			(xy 49.53 140.97) (xy 52.07 140.97)
 		)
@@
 	(wire
 		(pts
-			(xy 332.74 113.03) (xy 350.52 113.03)
-		)
-		(stroke
-			(width 0)
-			(type default)
-		)
-	)
-	(wire
-		(pts
 			(xy 184.15 85.09) (xy 250.19 85.09)
 		)
@@
 	(wire
 		(pts
-			(xy 327.66 110.49) (xy 327.66 119.38)
-		)
-		(stroke
-			(width 0)
-			(type default)
-		)
-	)
-	(wire
-		(pts
 			(xy 46.99 130.81) (xy 52.07 130.81)
 		)
@@
 	(symbol
 		(lib_id "power:GND")
-		(at 330.2 132.08 0)
-		(unit 1)
-		(exclude_from_sim no)
-		(in_bom yes)
-		(on_board yes)
-		(dnp no)
-		(property "Reference" "#PWR023"
-			(at 330.2 138.43 0)
-			(effects
-				(font
-					(size 1.27 1.27)
-				)
-				(hide yes)
-			)
-		)
-		(property "Value" "GND"
-			(at 330.2 135.89 0)
-			(effects
-				(font
-					(size 1.27 1.27)
-				)
-			)
-		)
-		(property "Footprint" ""
-			(at 330.2 132.08 0)
-			(effects
-				(font
-					(size 1.27 1.27)
-				)
-				(hide yes)
-			)
-		)
-		(property "Datasheet" ""
-			(at 330.2 132.08 0)
-			(effects
-				(font
-					(size 1.27 1.27)
-				)
-				(hide yes)
-			)
-		)
-		(property "Description" ""
-			(at 330.2 132.08 0)
-			(effects
-				(font
-					(size 1.27 1.27)
-				)
-				(hide yes)
-			)
-		)
-		(pin "1"
-		)
-		(instances
-			(project "Pico-CAN"
-				(path "/7933eff1-4657-450a-9155-0a77075ba053"
-					(reference "#PWR023")
-					(unit 1)
-				)
-			)
-		)
-	)
-	(symbol
-		(lib_id "power:GND")
 		(at 308.61 86.36 0)
 		(unit 1)
@@
 					(unit 1)
 				)
-			)
-		)
-	)
-	(symbol
-		(lib_id "Pico-CAN:PESD1CAN")
-		(at 335.28 123.19 270)
-		(unit 1)
-		(exclude_from_sim no)
-		(in_bom yes)
-		(on_board yes)
-		(dnp yes)
-		(fields_autoplaced yes)
-		(property "Reference" "D1"
-			(at 335.28 124.4599 90)
-			(effects
-				(font
-					(size 1.27 1.27)
-				)
-				(justify left)
-			)
-		)
-		(property "Value" "PESD1CAN"
-			(at 335.28 123.19 0)
-			(effects
-				(font
-					(size 1.27 1.27)
-				)
-				(hide yes)
-			)
-		)
-		(property "Footprint" "Package_TO_SOT_SMD:SOT-23"
-			(at 335.28 123.19 0)
-			(effects
-				(font
-					(size 1.27 1.27)
-				)
-				(hide yes)
-			)
-		)
-		(property "Datasheet" "Components/Nexperia-PESD1CAN.pdf"
-			(at 335.28 123.19 0)
-			(effects
-				(font
-					(size 1.27 1.27)
-				)
-				(hide yes)
-			)
-		)
-		(property "Description" ""
-			(at 335.28 123.19 0)
-			(effects
-				(font
-					(size 1.27 1.27)
-				)
-				(hide yes)
-			)
-		)
-		(property "MFG" "Nexperia"
-			(at 335.28 123.19 0)
-			(effects
-				(font
-					(size 1.27 1.27)
-				)
-				(hide yes)
-			)
-		)
-		(property "MFG P/N" "PESD1CAN,215"
-			(at 335.28 126.9999 90)
-			(effects
-				(font
-					(size 1.27 1.27)
-				)
-				(justify left)
-			)
-		)
-		(property "DIST" "Digikey"
-			(at 335.28 123.19 0)
-			(effects
-				(font
-					(size 1.27 1.27)
-				)
-				(hide yes)
-			)
-		)
-		(property "DIST P/N" "1727-3817-1-ND"
-			(at 335.28 123.19 0)
-			(effects
-				(font
-					(size 1.27 1.27)
-				)
-				(hide yes)
-			)
-		)
-		(property "JLCPCB" ""
-			(at 335.28 123.19 90)
-			(effects
-				(font
-					(size 1.27 1.27)
-				)
-				(hide yes)
-			)
-		)
-		(property "LCSC Part #" "C2984756"
-			(at 335.28 123.19 90)
-			(effects
-				(font
-					(size 1.27 1.27)
-				)
-				(hide yes)
-			)
-		)
-		(pin "2"
-		)
-		(pin "1"
-		)
-		(pin "3"
-		)
-		(instances
-			(project ""
-				(path "/7933eff1-4657-450a-9155-0a77075ba053"
-					(reference "D1")
-					(unit 1)
-				)

Commit message: Update BOM
Signed-off-by: Scott Berman <sgberman1@gmail.com>
Parts:
- added J4, J5: 20 Pos Header, symbol Graphic:SYM_Arrow_Large
- added J6: 3 Pos Header, symbol Graphic:SYM_Arrow_Large
- A1: DIST (none) -> Digikey; DIST P/N (none) -> 2648-SC1631CT-ND; MFG (none) -> Raspberry Pi; MFG P/N (none) -> SC1631
- C1, C2, C3, C4, C5: DIST (none) -> Digikey; DIST P/N (none) -> CC0805KRX7R8BB104; MFG (none) -> YAGEO; MFG P/N (none) -> 311-1141-1-ND
- J1: DIST (none) -> Digikey; DIST P/N (none) -> S2011EC-13-ND; MFG (none) -> Sullins Connector Solutions; MFG P/N (none) -> PRPC013DAAN-RC
- J2, J3: value CAN1 -> CAN; DIST P/N WM1340-ND -> WM4175-ND; MFG P/N 0015912025 -> 0705550036
- R1: DIST (none) -> Digikey; DIST P/N (none) -> 311-1.50KCRCT-ND; LCSC Part # C114555 -> (none); MFG (none) -> YAGEO; MFG P/N (none) -> RC0805FR-071K5L
