File: circuit-boards/mini-pdb-V2/mini-pdb.kicad_pcb (KiCad board)
At the start: 2 copper layers, 84.4 x 36.8 mm, 25 parts, among them J1 2604-1102, J2 2604-1102, J3 2604-1110

Commit message: Fix name on PCB
Signed-off-by: Scott Berman <sgberman1@gmail.com>
Parts:
- moved G*** 9.15 mm to (220.2, 115.6)
Other:
- board text added: "Mini Power Board"
- board text removed: "Mini Power Distribution Board"
Changed lines of the file:
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@@
 	(footprint "Logos:WCP-Logo_250"
 		(layer "B.Cu")
-		(at 229.362 115.824 180)
+		(at 220.218 115.57 180)
 		(property "Reference" "G***"
 			(at 0 0 0)
@@
 		)
 	)
-	(gr_text "Mini Power Distribution Board"
-		(at 224.663 116.967 0)
+	(gr_text "Mini Power Board"
+		(at 215.519 116.713 0)
 		(layer "B.SilkS")
 		(effects
