File: circuit-boards/NX-J401-Adapter-v5/NX-J401-Adapter.kicad_pcb (KiCad board)
At the start: 2 copper layers, 100 x 79 mm, 56 parts, among them J1 18V_OUT, J2 NX BUTTON, J3 Power, J4 USB_C_Receptacle_USB2.0_14P, Q1 CSD16322Q5, Q2 SI4483ADY-T1-GE3, SW1 RECOVERY, SW2 RESET, U1 LM3478MA, U2 ISO6721BDR, U3 FT232RNL

Commit message: Change NX-J401-Adapter to reduce the PCB standoff spacing.
Signed-off-by: Scott Berman <sgberman1@gmail.com>
Parts:
- removed the C8 at (291.6, 115.1)
- added C10: 120uF 25V, NX-J401-Adapter:CP_Radial_D8.0mm_P3.50mm_H7.0mm, F.Cu at (309.9, 107.8)
- added C17: 4.7uF-10%-50V-0805, Capacitor_SMD:C_0805_2012Metric, F.Cu at (280.2, 147.3)
- added C3: 120uF 25V, NX-J401-Adapter:CP_Radial_D8.0mm_P3.50mm_H7.0mm, F.Cu at (305.3, 99.9)
- added C4: 120uF 25V, NX-J401-Adapter:CP_Radial_D8.0mm_P3.50mm_H7.0mm, F.Cu at (314.5, 99.9)
- added D3: 15V, Diode_SMD:D_SOD-123F, F.Cu at (290.9, 125.4)
- added D4: 15V, Diode_SMD:D_SOD-123F, F.Cu at (298.7, 134.0)
- added Q3: MMBT3906LT1G, Package_TO_SOT_SMD:SOT-23, F.Cu at (290.9, 122.3)
- added Q4: SQM40061EL_GE3, NX-J401-Adapter:TO-263-2, F.Cu at (286.9, 133.7)
- added R10: 5.10k-1%-0805, Resistor_SMD:R_0805_2012Metric, F.Cu at (301.2, 134.0)
- added R14: 5.10k-1%-0805, Resistor_SMD:R_0805_2012Metric, F.Cu at (280.2, 151.4)
- added R9: 1.05k-1%-0805, Resistor_SMD:R_0805_2012Metric, F.Cu at (286.5, 125.4)
- C1, C2: value 82uF 35V -> 56uF 25V; footprint Capacitor_THT:CP_Radial_D8.0mm_P3.50mm -> NX-J401-Adapter:CP_Radial_D8.0mm_P3.50mm_H7.0mm
- C5: value 330uF 35V -> 56uF 25V; footprint Capacitor_THT:CP_Radial_D10.0mm_P5.00mm -> NX-J401-Adapter:CP_Radial_D8.0mm_P3.50mm_H7.0mm
- D2: value 15V -> 20V
- D5: renamed from D3; value 15V -> 24V; footprint Diode_SMD:D_SMB -> NX-J401-Adapter:D_SMC_Littelfuse_DO-214AB
- J1: value 18V_OUT -> V_OUT; footprint NX-J401-Adapter:CONN_69140872_WRE -> NX-J401-Adapter:Weidmuller-1824740000
- J3: footprint NX-J401-Adapter:Wurth-691406510002B -> NX-J401-Adapter:Weidmuller-1824740000
- Q2: value SI4483ADY-T1-GE3 -> SQM40061EL_GE3; footprint Package_SO:SOIC-8_3.9x4.9mm_P1.27mm -> NX-J401-Adapter:TO-263-2
- R11: value 4.99k-1%-0805 -> 1.00R-1%-0805
- R7: value 1.05k-1%-0805 -> 5.10k-1%-0805
- R8: value 20.0k-1%-0805 -> 5.10k-1%-0805
- moved LOGO1 42.6 mm to (239.9, 114.9)
- moved C5 34.2 mm to (275.8, 101.0), turned to -90 degrees
- moved D2 18.2 mm to (281.4, 123.3), turned to 180 degrees
- moved Q2 15.6 mm to (303.7, 122.0), turned to 0 degrees
- moved J1 12.9 mm to (269.3, 84.2), turned to -90 degrees
- moved J2 12.7 mm to (242.5, 101.6)
- moved R8 11.1 mm to (286.5, 121.3), turned to 0 degrees
- moved R7 8.31 mm to (286.5, 119.3), turned to 0 degrees
- moved R11 5.62 mm to (283.9, 147.3)
- moved C2 1.92 mm to (275.8, 92.1)
- moved C1 1.62 mm to (275.8, 83.2)
- moved D5 0.85 mm to (303.0, 145.3)
- moved J3 0.63 mm to (290.6, 149.0)
- renumbered C9 to C11, C10 to C12, C11 to C13, C12 to C14, C13 to C15, C14 to C16, C15 to C18, C3 to C6, C4 to C7, C6 to C8, C7 to C9, D4 to D6, D5 to D7, R9 to R12, R10 to R13
Connections:
- C5 pad 1: /Power Supply/V_IN -> +18V
- D2 pad 1: /Power Supply/V_IN -> Net-(D2-K)
- D2 pad 2: Net-(D2-A) -> GND
- D7 pad 1: Net-(D5-KA) -> Net-(D7-KA)
- Q2 pad 1: /Power Supply/V_IN -> Net-(D3-A)
- Q2 pad 3: /Power Supply/V_IN -> /Power Supply/V_P
- R11 pad 1: Net-(D5-KA) -> Net-(C17-Pad1)
- R7 pad 2: Net-(D2-A) -> Net-(D3-A)
- R8 pad 1: Net-(D2-A) -> Net-(D2-K)
- R8 pad 2: /Power Supply/V_IN -> Net-(Q3-B)
Routing:
- net /Power Supply/V_IN: track 27.9 -> 111.5 mm
- net /V_BAT: track 13.3 -> 38.5 mm
- net /Power Supply/V_P: track 0.00 -> 24.5 mm
- net Net-(D3-A): track 0.00 -> 17.7 mm
- net Net-(D2-A): track 14.0 -> 0.00 mm
- net /PC_LED+: track 96.2 -> 83.2 mm
- net /PC_LED-: track 104.8 -> 92.0 mm
- net /3V3: track 41.5 -> 28.8 mm
- net /~{SYS_RESET}: track 68.8 -> 56.1 mm
- net /~{REC}: track 67.8 -> 55.1 mm
- net /UART2_RXD: track 55.0 -> 43.2 mm
- net /UART2_TXD: track 51.3 -> 39.6 mm
- net Net-(D4-A): track 0.00 -> 11.0 mm
- net GND: track 36.5 -> 45.8 mm, vias 12 -> 17
- net Net-(D2-K): track 0.00 -> 7.66 mm
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- added copper zone on F.Cu, net /Power Supply/V_P
Other:
- outline, holes or cut-outs redrawn
- board text removed: "${LAYER}"
