File: circuit-boards/NX-J401-Adapter-v5/PowerSupply.kicad_sch (KiCad schematic)
At the start: 23 parts, among them Q1 CSD16322Q5, Q2 SI4483ADY-T1-GE3, U1 LM3478MA

Commit message: Add over voltage protection to NX adapter circuit. Also reduce component height
Signed-off-by: Scott Berman <sgberman1@gmail.com>
Parts:
- removed Q2: SI4483ADY-T1-GE3, Package_SO:SOIC-8_3.9x4.9mm_P1.27mm, symbol Device:Q_PMOS_SGD
- removed R8: 20.0k-1%-0805, Resistor_SMD:R_0805_2012Metric, symbol Device:R_US
- added C16: 56uF 25V, Capacitor_THT:CP_Radial_D8.0mm_P3.50mm, symbol Device:C_Polarized_US
- added C17, C18: 120uF 25V, Capacitor_THT:CP_Radial_D8.0mm_P3.50mm, symbol Device:C_Polarized_US
- added D7: 15V, Diode_SMD:D_SOD-123F, symbol Device:D_Zener
- added Q2, Q6: SQM40061EL_GE3, NX-J401-Adapter:TO-263-2, symbol Simulation_SPICE:PMOS
- added Q3: MMBT3906LT1G, Package_TO_SOT_SMD:SOT-23, symbol Transistor_BJT:MMBT3906
- added R12: 5.10k-1%-0805, Resistor_SMD:R_0805_2012Metric, symbol Device:R_US
- added R14: 100R-1%-0805, Resistor_SMD:R_0805_2012Metric, symbol Device:R_US
- added R15, R17: 1.05k-1%-0805, Resistor_SMD:R_0805_2012Metric, symbol Device:R_US
- added R18: 6.98k-1%-0805, Resistor_SMD:R_0805_2012Metric, symbol Device:R_US
- added U4: TL431DBZ, Package_TO_SOT_SMD:SOT-23, symbol Reference_Voltage:TL431DBZ
- C1, C2: value 82uF 35V -> 56uF 25V; DIST Digikey -> Mouser; DIST P/N P16345-ND -> 667-25SEPF56M; MFG P/N 35SEPF82M -> 25SEPF56M
- C5: value 330uF 35V -> 120uF 25V; footprint Capacitor_THT:CP_Radial_D10.0mm_P5.00mm -> Capacitor_THT:CP_Radial_D8.0mm_P3.50mm; DIST P/N 1189-35PZJ330M10X9-ND -> P122635-ND; MFG Rubycon -> Panasonic; MFG P/N 35PZJ330M10X9 -> 25SEK120M
Connections:
- net +18V: now also C16.1
- net GND: now also C16.2, C17.2, C18.2, R15.1, R17.1, U4.3 (A)
- net V_IN: now also C17.1, C18.1, Q6.1 (D), R18.1; no longer D2.1 (K)
- net V_{BAT}: now also Q2.1 (D)
- net at D2.2 (A), R7.2: now also Q2.2 (G)
- new net: Q3.1 (B), R12.1, R14.2
- new net: D2.1 (K), D7.1 (K), Q2.3 (S), Q3.2 (E), Q6.3 (S), R14.1
- new net: D7.2 (A), Q3.3 (C), Q6.2 (G), R15.2
- new net: R17.2, R18.2, U4.2 (REF)
- new net: R12.2, U4.1 (K)
Other:
- note added: "18V Boost Converter"
- note added: "2.495V"
- note added: "Fix polymer cap step files"
- note added: "Overvoltage Limiter"
- note added: "Reverse Polarity Protector"
- note added: "Setpoint 19V"
- moved on the sheet: C1, C3, C4, C6, C7, C8, D1, D3, L1, Q1, R1, R2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

Commit message: Change NX-J401-Adapter to reduce the PCB standoff spacing.
Signed-off-by: Scott Berman <sgberman1@gmail.com>
Parts:
- removed C8: 22uF-20%-25V-0805, Capacitor_SMD:C_0805_2012Metric, symbol Device:C
- removed Q2, Q6: SQM40061EL_GE3, NX-J401-Adapter:TO-263-2, symbol Simulation_SPICE:PMOS
- removed R12: 5.10k-1%-0805, Resistor_SMD:R_0805_2012Metric, symbol Device:R_US
- removed R14: 100R-1%-0805, Resistor_SMD:R_0805_2012Metric, symbol Device:R_US
- removed R15, R17: 1.05k-1%-0805, Resistor_SMD:R_0805_2012Metric, symbol Device:R_US
- removed R18: 6.98k-1%-0805, Resistor_SMD:R_0805_2012Metric, symbol Device:R_US
- removed U4: TL431DBZ, Package_TO_SOT_SMD:SOT-23, symbol Reference_Voltage:TL431DBZ
- added C17: 4.7uF-10%-50V-0805, Capacitor_SMD:C_0805_2012Metric, symbol Device:C
- added D2: 20V, Diode_SMD:D_SOD-123F, symbol Device:D_Zener
- added Q2, Q4: SQM40061EL_GE3, NX-J401-Adapter:TO-263-2, symbol NX-AdapterBoard:SQM40061EL_GE3
- added R10, R8: 5.10k-1%-0805, Resistor_SMD:R_0805_2012Metric, symbol Device:R_US
- added R11: 1.00R-1%-0805, Resistor_SMD:R_0805_2012Metric, symbol Device:R_US
- added R9: 1.05k-1%-0805, Resistor_SMD:R_0805_2012Metric, symbol Device:R_US
- C1: renamed from C2; footprint Capacitor_THT:CP_Radial_D8.0mm_P3.50mm -> NX-J401-Adapter:CP_Radial_D8.0mm_P3.50mm_H7.0mm
- C10: renamed from C18; footprint Capacitor_THT:CP_Radial_D8.0mm_P3.50mm -> NX-J401-Adapter:CP_Radial_D8.0mm_P3.50mm_H7.0mm
- C2: renamed from C16; footprint Capacitor_THT:CP_Radial_D8.0mm_P3.50mm -> NX-J401-Adapter:CP_Radial_D8.0mm_P3.50mm_H7.0mm
- C3: renamed from C5; footprint Capacitor_THT:CP_Radial_D8.0mm_P3.50mm -> NX-J401-Adapter:CP_Radial_D8.0mm_P3.50mm_H7.0mm
- C4: renamed from C17; footprint Capacitor_THT:CP_Radial_D8.0mm_P3.50mm -> NX-J401-Adapter:CP_Radial_D8.0mm_P3.50mm_H7.0mm
- C5: renamed from C1; footprint Capacitor_THT:CP_Radial_D8.0mm_P3.50mm -> NX-J401-Adapter:CP_Radial_D8.0mm_P3.50mm_H7.0mm
- D5: renamed from D3; value 15V -> 24V; footprint Diode_SMD:D_SMB -> NX-J401-Adapter:D_SMC_Littelfuse_DO-214AB; DIST P/N F11544CT-ND -> SMDJ24CACT-ND; MFG P/N SZ1SMB15CAT3G -> SMDJ24CA
- R7: value 1.05k-1%-0805 -> 5.10k-1%-0805; DIST P/N 311-1.05KCRCT-ND -> 311-5.10KCRCT-ND; MFG P/N RC0805FR-071K05L -> RC0805FR-075K1L
- renumbered C3 to C6, C4 to C7, C6 to C8, C7 to C9, D7 to D3, D2 to D4
Connections:
- net GND: now also C17.2, D2.2 (A), R10.1
- net V_IN: now also Q2.2 (D)
- net V_{BAT}: now also Q4.2 (D), R11.2
- net at Q3.1 (B): now also R8.2
- net V_P: now reaches D3.1 (K), D4.1 (K), Q3.2 (E)
- net V_P: now also Q2.3 (S), Q4.3 (S), R9.2
- net at D3.2 (A), Q3.3 (C): now also R7.2, Q2.1 (G)
- net at D4.2 (A): now also Q4.1 (G), R10.2; no longer R7.2
- new net: D2.1 (K), R8.1, R9.1
- new net: C17.1, R11.1
Other:
- note added: "Overvoltage Shutdown"
- note added: "V_trip = 21V"
- note removed: "2.495V"
- note removed: "Fix polymer cap step files"
- note removed: "Overvoltage Limiter"
- note removed: "Setpoint 19V"
- moved on the sheet: C8, D3, R6

Commit message: Fixed IDC connector part number
Signed-off-by: Scott Berman <scott.berman@bluerivertech.com>
Parts:
- Q3: value MMBT3906LT1G -> MMBT3906LT3G; DIST P/N MMBT3906LT1GOSCT-ND -> MMBT3906LT3GOSCT-ND; MFG P/N MMBT3906LT1G -> MMBT3906LT3G
- R10, R7, R8: DIST P/N 311-5.10KCRCT-ND -> 13-RC0805FR-135K1LCT-ND; MFG P/N RC0805FR-075K1L -> RC0805FR-135K1L
Changed lines of the file:
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@@
 			)
 		)
-		(property "Value" "MMBT3906LT1G"
+		(property "Value" "MMBT3906LT3G"
 			(at 131.572 96.52 0)
 			(effects
@@
 			)
 		)
-		(property "MFG P/N" "MMBT3906LT1G"
+		(property "MFG P/N" "MMBT3906LT3G"
 			(at 127 95.25 0)
 			(effects
@@
 			)
 		)
-		(property "DIST P/N" "MMBT3906LT1GOSCT-ND"
+		(property "DIST P/N" "MMBT3906LT3GOSCT-ND"
 			(at 127 95.25 0)
 			(effects
@@
 			)
 		)
-		(property "MFG P/N" "RC0805FR-075K1L"
+		(property "MFG P/N" "RC0805FR-135K1L"
 			(at 116.84 95.25 0)
 			(effects
@@
 			)
 		)
-		(property "DIST P/N" "311-5.10KCRCT-ND"
+		(property "DIST P/N" "13-RC0805FR-135K1LCT-ND"
 			(at 116.84 95.25 0)
 			(effects
@@
 			)
 		)
-		(property "MFG P/N" "RC0805FR-075K1L"
+		(property "MFG P/N" "RC0805FR-135K1L"
 			(at 69.85 127 0)
 			(effects
@@
 			)
 		)
-		(property "DIST P/N" "311-5.10KCRCT-ND"
+		(property "DIST P/N" "13-RC0805FR-135K1LCT-ND"
 			(at 69.85 127 0)
 			(effects
@@
 			)
 		)
-		(property "MFG P/N" "RC0805FR-075K1L"
+		(property "MFG P/N" "RC0805FR-135K1L"
 			(at 162.56 127 0)
 			(effects
@@
 			)
 		)
-		(property "DIST P/N" "311-5.10KCRCT-ND"
+		(property "DIST P/N" "13-RC0805FR-135K1LCT-ND"
 			(at 162.56 127 0)
 			(effects
