File: circuit-boards/NX-J401-Adapter-v5/usb-serial.kicad_sch (KiCad schematic)
At the start: 13 parts, among them J4 USB_C_Receptacle_USB2.0_14P, U2 ISO6721BDR, U3 FT232RNL

Commit message: Change NX-J401-Adapter to reduce the PCB standoff spacing.
Signed-off-by: Scott Berman <sgberman1@gmail.com>
Parts:
- renumbered C9 to C11, C10 to C12, C11 to C13, C12 to C14, C13 to C15, C14 to C16, C15 to C18, R9 to R12, R10 to R13
Changed lines of the file:
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@@
 	(title_block
 		(title "NX J401 Adapter")
-		(date "2025-09-13")
+		(date "2025-10-19")
 		(rev "5")
 	)
@@
 		(on_board yes)
 		(dnp no)
-		(property "Reference" "C12"
+		(property "Reference" "C14"
 			(at 210.82 189.23 0)
 			(effects
@@
 			(project "NX-J401-Adapter"
 				(path "/cc31ce4b-09ab-4aea-a1d3-ed84696ba658/0fdfc19c-5516-450c-b6f2-10dc3e7a4edc"
-					(reference "C12")
+					(reference "C14")
 					(unit 1)
 				)
@@
 		(on_board yes)
 		(dnp no)
-		(property "Reference" "C11"
+		(property "Reference" "C13"
 			(at 153.67 130.81 0)
 			(effects
@@
 			(project "NX-J401-Adapter"
 				(path "/cc31ce4b-09ab-4aea-a1d3-ed84696ba658/0fdfc19c-5516-450c-b6f2-10dc3e7a4edc"
-					(reference "C11")
+					(reference "C13")
 					(unit 1)
 				)
@@
 		(on_board yes)
 		(dnp no)
-		(property "Reference" "C15"
+		(property "Reference" "C18"
 			(at 115.57 130.81 0)
 			(effects
@@
 			(project "NX-J401-Adapter"
 				(path "/cc31ce4b-09ab-4aea-a1d3-ed84696ba658/0fdfc19c-5516-450c-b6f2-10dc3e7a4edc"
-					(reference "C15")
+					(reference "C18")
 					(unit 1)
 				)
@@
 		(on_board yes)
 		(dnp no)
-		(property "Reference" "C14"
+		(property "Reference" "C16"
 			(at 128.27 189.23 0)
 			(effects
@@
 			(project "NX-J401-Adapter"
 				(path "/cc31ce4b-09ab-4aea-a1d3-ed84696ba658/0fdfc19c-5516-450c-b6f2-10dc3e7a4edc"
-					(reference "C14")
+					(reference "C16")
 					(unit 1)
 				)
@@
 		(on_board yes)
 		(dnp no)
-		(property "Reference" "C9"
+		(property "Reference" "C11"
 			(at 320.04 106.68 0)
 			(effects
@@
 			(project "NX-J401-Adapter"
 				(path "/cc31ce4b-09ab-4aea-a1d3-ed84696ba658/0fdfc19c-5516-450c-b6f2-10dc3e7a4edc"
-					(reference "C9")
+					(reference "C11")
 					(unit 1)
 				)
@@
 		(on_board yes)
 		(dnp no)
-		(property "Reference" "C10"
+		(property "Reference" "C12"
 			(at 280.67 93.98 0)
 			(effects
@@
 			(project "NX-J401-Adapter"
 				(path "/cc31ce4b-09ab-4aea-a1d3-ed84696ba658/0fdfc19c-5516-450c-b6f2-10dc3e7a4edc"
-					(reference "C10")
+					(reference "C12")
 					(unit 1)
 				)
@@
 		(on_board yes)
 		(dnp no)
-		(property "Reference" "R10"
+		(property "Reference" "R13"
 			(at 123.698 156.21 90)
 			(effects
@@
 			(project "NX-J401-Adapter"
 				(path "/cc31ce4b-09ab-4aea-a1d3-ed84696ba658/0fdfc19c-5516-450c-b6f2-10dc3e7a4edc"
-					(reference "R10")
+					(reference "R13")
 					(unit 1)
 				)
@@
 		(on_board yes)
 		(dnp no)
-		(property "Reference" "R9"
+		(property "Reference" "R12"
 			(at 113.538 158.75 90)
 			(effects
@@
 			(project "NX-J401-Adapter"
 				(path "/cc31ce4b-09ab-4aea-a1d3-ed84696ba658/0fdfc19c-5516-450c-b6f2-10dc3e7a4edc"
-					(reference "R9")
+					(reference "R12")
 					(unit 1)
 				)
@@
 		(on_board yes)
 		(dnp no)
-		(property "Reference" "C13"
+		(property "Reference" "C15"
 			(at 138.43 189.23 0)
 			(effects
@@
 			(project "NX-J401-Adapter"
 				(path "/cc31ce4b-09ab-4aea-a1d3-ed84696ba658/0fdfc19c-5516-450c-b6f2-10dc3e7a4edc"
-					(reference "C13")
+					(reference "C15")
 					(unit 1)
 				)

Commit message: Fix bom to reduce line items. Addd zip tie slots. Add 1.5mm tooling holes
Signed-off-by: Scott Berman <sgberman1@gmail.com>
Parts:
- C11, C12, C14: value 0.1uF-10%-25V-0805 -> 0.22uF-10%-50V-0805; DIST P/N 399-C0805C104K3RACTUCT-ND -> 399-C0805C224K5RACTUCT-ND; MFG P/N C0805C104K3RACTU -> C0805C224K5RAC7800
- C13: value 4.7uF-10%-25V-0805 -> 4.7uF-10%-50V-0805; DIST P/N 1276-1244-1-ND -> 490-10751-1-ND; MFG Samsung Electro-Mechanics -> Murata Electronics; MFG P/N CL21A475KAQNNNE -> GRM21BR61H475KE51L
Changed lines of the file:
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@@
 	(title_block
 		(title "NX J401 Adapter")
-		(date "2025-10-19")
+		(date "2025-10-24")
 		(rev "5")
 	)
@@
 			)
 		)
-		(property "Value" "0.1uF-10%-25V-0805"
+		(property "Value" "0.22uF-10%-50V-0805"
 			(at 205.74 191.77 90)
 			(effects
@@
 			)
 		)
-		(property "Datasheet" ""
+		(property "Datasheet" "Components/KEMET_C1002_X7R_SMD.pdf"
 			(at 209.55 191.77 0)
 			(effects
@@
 			)
 		)
-		(property "MFG P/N" "C0805C104K3RACTU"
+		(property "MFG P/N" "C0805C224K5RAC7800"
 			(at 209.55 191.77 0)
 			(effects
@@
 			)
 		)
-		(property "DIST P/N" "399-C0805C104K3RACTUCT-ND"
+		(property "DIST P/N" "399-C0805C224K5RACTUCT-ND"
 			(at 209.55 191.77 0)
 			(effects
@@
 			)
 		)
-		(property "Value" "4.7uF-10%-25V-0805"
+		(property "Value" "4.7uF-10%-50V-0805"
 			(at 158.75 133.35 90)
 			(effects
@@
 			)
 		)
-		(property "Datasheet" ""
+		(property "Datasheet" "Components/KEMET_C1002_X7R_SMD.pdf"
 			(at 154.94 133.35 0)
 			(effects
@@
 			)
 		)
-		(property "MFG" "Samsung Electro-Mechanics"
+		(property "MFG" "Murata Electronics"
 			(at 154.94 133.35 0)
 			(effects
@@
 			)
 		)
-		(property "MFG P/N" "CL21A475KAQNNNE"
+		(property "MFG P/N" "GRM21BR61H475KE51L"
 			(at 154.94 133.35 0)
 			(effects
@@
 			)
 		)
-		(property "DIST P/N" "1276-1244-1-ND"
+		(property "DIST P/N" "490-10751-1-ND"
 			(at 154.94 133.35 0)
 			(effects
@@
 			)
 		)
-		(property "Value" "0.1uF-10%-25V-0805"
+		(property "Value" "0.22uF-10%-50V-0805"
 			(at 325.12 109.22 0)
 			(effects
@@
 			)
 		)
-		(property "Datasheet" ""
+		(property "Datasheet" "Components/KEMET_C1002_X7R_SMD.pdf"
 			(at 321.31 109.22 0)
 			(effects
@@
 			)
 		)
-		(property "MFG P/N" "C0805C104K3RACTU"
+		(property "MFG P/N" "C0805C224K5RAC7800"
 			(at 321.31 109.22 0)
 			(effects
@@
 			)
 		)
-		(property "DIST P/N" "399-C0805C104K3RACTUCT-ND"
+		(property "DIST P/N" "399-C0805C224K5RACTUCT-ND"
 			(at 321.31 109.22 0)
 			(effects
@@
 			)
 		)
-		(property "Value" "0.1uF-10%-25V-0805"
+		(property "Value" "0.22uF-10%-50V-0805"
 			(at 275.59 96.52 90)
 			(effects
@@
 			)
 		)
-		(property "Datasheet" ""
+		(property "Datasheet" "Components/KEMET_C1002_X7R_SMD.pdf"
 			(at 279.4 96.52 0)
 			(effects
@@
 			)
 		)
-		(property "MFG P/N" "C0805C104K3RACTU"
+		(property "MFG P/N" "C0805C224K5RAC7800"
 			(at 279.4 96.52 0)
 			(effects
@@
 			)
 		)
-		(property "DIST P/N" "399-C0805C104K3RACTUCT-ND"
+		(property "DIST P/N" "399-C0805C224K5RACTUCT-ND"
 			(at 279.4 96.52 0)
 			(effects

Commit message: Fixed IDC connector part number
Signed-off-by: Scott Berman <scott.berman@bluerivertech.com>
Parts:
- R12, R13: DIST P/N 311-5.10KCRCT-ND -> 13-RC0805FR-135K1LCT-ND; MFG P/N RC0805FR-075K1L -> RC0805FR-135K1L
- U3: DIST Digikey -> Mouser; DIST P/N 768-FT232RNL-REELCT-ND -> 895-FT232RNL-TUBE
Changed lines of the file:
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@@
 			)
 		)
-		(property "MFG P/N" "RC0805FR-075K1L"
+		(property "MFG P/N" "RC0805FR-135K1L"
 			(at 118.11 154.94 0)
 			(effects
@@
 			)
 		)
-		(property "DIST P/N" "311-5.10KCRCT-ND"
+		(property "DIST P/N" "13-RC0805FR-135K1LCT-ND"
 			(at 118.11 154.94 0)
 			(effects
@@
 			)
 		)
-		(property "DIST" "Digikey"
+		(property "DIST" "Mouser"
 			(at 237.49 166.37 0)
 			(effects
@@
 			)
 		)
-		(property "DIST P/N" "768-FT232RNL-REELCT-ND"
+		(property "DIST P/N" "895-FT232RNL-TUBE "
 			(at 237.49 166.37 0)
 			(effects
@@
 			)
 		)
-		(property "MFG P/N" "RC0805FR-075K1L"
+		(property "MFG P/N" "RC0805FR-135K1L"
 			(at 118.11 160.02 0)
 			(effects
@@
 			)
 		)
-		(property "DIST P/N" "311-5.10KCRCT-ND"
+		(property "DIST P/N" "13-RC0805FR-135K1LCT-ND"
 			(at 118.11 160.02 0)
 			(effects
