File: circuit-boards/Pico-ButtonBoard-v1/Pico-ButtonBoard-v1.kicad_pcb (KiCad board)
At the start: 2 copper layers, 179 parts, among them J101 DC_IN, J102 BATT, J103 CAN, J104 CAN, J201 B0, J202 B1, J203 B2, J204 B3, J205 B4, J206 B5, J207 B6, J208 B7, J209 B8, J210 B9, J211 B10, J212 B11, J213 B12, J214 B13, J215 B14, J216 B15, J301 XY1-L, J302 XY0-R, J501 ID, Q401 BSS123, Q402 BSS123, U101 4.0 MHz, U102 MCP2518FDT-H/SL, U103 MCP2558FD, U201 SN74HC165DR, U202 SN74HC165DR, U301 TLV77033DDC, U302 SN74LVC1G3157DBVR, U401 ITS41k0S-ME-N, U402 TPS54202DDC

Commit message: Pico Button Board initial placement
Signed-off-by: Scott Berman <sgberman1@gmail.com>
Parts:
- added FID101: Fiducial, Fiducial:Fiducial_Cross_1.5mm_Mask2mm, F.Cu at (278.3, 47.9)
- added FID102: Fiducial, Fiducial:Fiducial_Cross_1.5mm_Mask2mm, F.Cu at (278.3, 51.4)
- added FID103: Fiducial, Fiducial:Fiducial_Cross_1.5mm_Mask2mm, F.Cu at (281.8, 47.9)
- added FID104: Fiducial, Fiducial:Fiducial_Cross_1.5mm_Mask2mm, F.Cu at (281.8, 51.4)
- added FID105: Fiducial, Fiducial:Fiducial_Cross_1.5mm_Mask2mm, F.Cu at (285.4, 47.9)
- added FID106: Fiducial, Fiducial:Fiducial_Cross_1.5mm_Mask2mm, F.Cu at (285.4, 51.4)
- added H101: MountingHole, MountingHole:MountingHole_3.2mm_M3, F.Cu at (179.7, 73.0)
- added H102: MountingHole, MountingHole:MountingHole_3.2mm_M3, F.Cu at (179.7, 177.2)
- added H103: MountingHole, MountingHole:MountingHole_3.2mm_M3, F.Cu at (228.0, 177.2)
- added H104: MountingHole, MountingHole:MountingHole_3.2mm_M3, F.Cu at (228.0, 73.0)
- added J601: ENC0, Pico-ButtonBoard:Molex-70543-0039, F.Cu at (227.3, 90.8)
- added J602: ENC1, Pico-ButtonBoard:Molex-70543-0039, F.Cu at (180.4, 82.8)
- added J603: ENC2, Pico-ButtonBoard:Molex-70543-0039, F.Cu at (180.4, 98.0)
- added J604: ENC PWR, Connector_PinHeader_2.54mm:PinHeader_1x03_P2.54mm_Vertical, F.Cu at (220.5, 71.9)
- added R601: 20k-1%-0805, Resistor_SMD:R_0805_2012Metric_Pad1.20x1.40mm_HandSolder, F.Cu at (64.7, 81.8)
- added R602: 49.9R-1%-0805, Resistor_SMD:R_0805_2012Metric_Pad1.20x1.40mm_HandSolder, F.Cu at (64.7, 84.8)
- added R603: 20k-1%-0805, Resistor_SMD:R_0805_2012Metric_Pad1.20x1.40mm_HandSolder, F.Cu at (64.7, 87.7)
- added R604: 20k-1%-0805, Resistor_SMD:R_0805_2012Metric_Pad1.20x1.40mm_HandSolder, F.Cu at (64.7, 90.7)
- added R605: 49.9R-1%-0805, Resistor_SMD:R_0805_2012Metric_Pad1.20x1.40mm_HandSolder, F.Cu at (64.7, 93.6)
- added R606: 49.9R-1%-0805, Resistor_SMD:R_0805_2012Metric_Pad1.20x1.40mm_HandSolder, F.Cu at (64.7, 96.6)
- added R607: 20k-1%-0805, Resistor_SMD:R_0805_2012Metric_Pad1.20x1.40mm_HandSolder, F.Cu at (64.7, 99.5)
- added R608: 20k-1%-0805, Resistor_SMD:R_0805_2012Metric_Pad1.20x1.40mm_HandSolder, F.Cu at (69.4, 81.8)
- added R609: 20k-1%-0805, Resistor_SMD:R_0805_2012Metric_Pad1.20x1.40mm_HandSolder, F.Cu at (69.4, 84.8)
- added R610: 49.9R-1%-0805, Resistor_SMD:R_0805_2012Metric_Pad1.20x1.40mm_HandSolder, F.Cu at (69.4, 87.7)
- added R611: 49.9R-1%-0805, Resistor_SMD:R_0805_2012Metric_Pad1.20x1.40mm_HandSolder, F.Cu at (69.4, 90.7)
- added R612: 49.9R-1%-0805, Resistor_SMD:R_0805_2012Metric_Pad1.20x1.40mm_HandSolder, F.Cu at (69.4, 93.6)
- added R613: 20k-1%-0805, Resistor_SMD:R_0805_2012Metric_Pad1.20x1.40mm_HandSolder, F.Cu at (69.4, 96.6)
- added R614: 20k-1%-0805, Resistor_SMD:R_0805_2012Metric_Pad1.20x1.40mm_HandSolder, F.Cu at (69.4, 99.5)
- added R615: 20k-1%-0805, Resistor_SMD:R_0805_2012Metric_Pad1.20x1.40mm_HandSolder, F.Cu at (74.2, 81.8)
- added R616: 49.9R-1%-0805, Resistor_SMD:R_0805_2012Metric_Pad1.20x1.40mm_HandSolder, F.Cu at (74.2, 84.8)
- added R617: 49.9R-1%-0805, Resistor_SMD:R_0805_2012Metric_Pad1.20x1.40mm_HandSolder, F.Cu at (74.2, 87.7)
- added R618: 49.9R-1%-0805, Resistor_SMD:R_0805_2012Metric_Pad1.20x1.40mm_HandSolder, F.Cu at (74.2, 90.7)
- J101, J102, J103, J104, J201, J202, J203, J204, J205, J206, J207, J208, J209, J210, J211, J212, J213, J214, J215, J216: footprint Pico-ButtonBoard:Molex-70555-0036 -> Pico-ButtonBoard:Molex-70543-0001
- J501: footprint Pico-ButtonBoard:Molex-70555-0038 -> Pico-ButtonBoard:Molex-70543-0003
- moved C102 477.1 mm to (299.7, 126.1)
- moved C103 477.1 mm to (299.7, 129.1)
- moved C104 477.1 mm to (299.7, 132.1)
- moved C105 477.1 mm to (299.7, 135.2)
- moved U102 469.6 mm to (301.6, 109.6)
- moved TP101 468.7 mm to (304.3, 123.8)
- moved TP102 468.7 mm to (304.3, 128.1)
- moved U101 457.5 mm to (301.6, 118.1)
- moved U103 456.1 mm to (301.6, 101.2)
- moved J301 445.8 mm to (229.1, 103.5), turned to 90 degrees
- moved J102 427.5 mm to (227.3, 138.7), turned to 90 degrees
- moved J302 426.8 mm to (229.1, 114.7), turned to 90 degrees
- moved C101 407.3 mm to (234.6, 85.9)
- moved J501 397.3 mm to (188.6, 73.7), turned to 90 degrees
- moved A101 389.3 mm to (203.8, 95.9)
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Connections:
- net /Joystick Inputs/ADC0 renamed /X0_ADC
- net /Joystick Inputs/ADC1 renamed /Y0_ADC
- net /Joystick Inputs/ADC2 renamed /XY1_ADC
- A101 pad 1: unconnected-(A101-GPIO0-Pad1)_1 -> /ENC0_A
- A101 pad 10: unconnected-(A101-GPIO7-Pad10)_1 -> /ENC1_PWM
- A101 pad 11: unconnected-(A101-GPIO8-Pad11) -> /ENC2_A
- A101 pad 12: unconnected-(A101-GPIO9-Pad12) -> /ENC2_B
- A101 pad 15: /ADC3/~{ADC2} -> /ENC2_PWM
- A101 pad 2: unconnected-(A101-GPIO1-Pad2) -> /ENC0_B
- A101 pad 21: /START_OF_FRAME -> /ADC3/~{ADC2}
- A101 pad 6: unconnected-(A101-GPIO4-Pad6)_1 -> /ENC0_PWM
- A101 pad 7: unconnected-(A101-GPIO5-Pad7)_1 -> /ENC1_A
- A101 pad 9: unconnected-(A101-GPIO6-Pad9)_1 -> /ENC1_B
- U102 pad 3: /START_OF_FRAME -> unconnected-(U102-CLKO/SOF-Pad3)
Other:
- board outline added: 55.9 x 111.8 mm

Commit message: Pico Button Board initial pcb checkin
Signed-off-by: Scott Berman <sgberman1@gmail.com>
Parts:
- removed L302: 10uH-10%-500mA-0805, Inductor_SMD:L_0805_2012Metric_Pad1.05x1.20mm_HandSolder
- A1: renamed from A101; footprint Module:RaspberryPi_Pico_Common_Unspecified -> Pico-ButtonBoard:RaspberryPi_Pico_Common_Unspecified
- C10: renamed from C302; moved to B.Cu
- C11: renamed from C305; moved to B.Cu
- C12: renamed from C216; moved to B.Cu
- C13: renamed from C214; moved to B.Cu
- C14: renamed from C212; moved to B.Cu
- C15: renamed from C210; moved to B.Cu
- C16: renamed from C301; moved to B.Cu
- C17: renamed from C306; moved to B.Cu
- C18: renamed from C309; moved to B.Cu
- C19: renamed from C310; moved to B.Cu
- C20: renamed from C104; moved to B.Cu
- C21: renamed from C308; moved to B.Cu
- C22: renamed from C105; moved to B.Cu
- C23: renamed from C103; moved to B.Cu
- C24: renamed from C401; moved to B.Cu
- C25: renamed from C208; moved to B.Cu
- C26: renamed from C101; moved to B.Cu
- C27: renamed from C404; moved to B.Cu
- C28: renamed from C206; moved to B.Cu
- C29: renamed from C403; moved to B.Cu
- C30: renamed from C204; moved to B.Cu
- C31: renamed from C502; moved to B.Cu
- C32: renamed from C501; moved to B.Cu
- C33: renamed from C202; moved to B.Cu
- C34: renamed from C201; moved to B.Cu
- C35: renamed from C203; moved to B.Cu
- C36: renamed from C205; moved to B.Cu
- C37: renamed from C207; moved to B.Cu
- C38: renamed from C209; moved to B.Cu
- C39: renamed from C211; moved to B.Cu
- C40: renamed from C213; moved to B.Cu
- C41: renamed from C215; moved to B.Cu
- D22: renamed from D406; moved to B.Cu
- D23: renamed from D404; moved to B.Cu
- FID1: renamed from FID105; footprint Fiducial:Fiducial_Cross_1.5mm_Mask2mm -> Pico-ButtonBoard:Fiducial_1.6mm_Mask3mm
- FID2: renamed from FID103; footprint Fiducial:Fiducial_Cross_1.5mm_Mask2mm -> Pico-ButtonBoard:Fiducial_1.6mm_Mask3mm
- FID3: renamed from FID101; footprint Fiducial:Fiducial_Cross_1.5mm_Mask2mm -> Pico-ButtonBoard:Fiducial_1.6mm_Mask3mm
- FID4: renamed from FID102; footprint Fiducial:Fiducial_Cross_1.5mm_Mask2mm -> Pico-ButtonBoard:Fiducial_1.6mm_Mask3mm; moved to B.Cu
- FID5: renamed from FID104; footprint Fiducial:Fiducial_Cross_1.5mm_Mask2mm -> Pico-ButtonBoard:Fiducial_1.6mm_Mask3mm; moved to B.Cu
- FID6: renamed from FID106; footprint Fiducial:Fiducial_Cross_1.5mm_Mask2mm -> Pico-ButtonBoard:Fiducial_1.6mm_Mask3mm; moved to B.Cu
- Q1: renamed from Q401; footprint Package_TO_SOT_SMD:SOT-23 -> Package_TO_SOT_SMD:SOT-23-3
- Q2: renamed from Q402; footprint Package_TO_SOT_SMD:SOT-23 -> Package_TO_SOT_SMD:SOT-23-3; moved to B.Cu
- R40: renamed from R301; moved to B.Cu
- R41: renamed from R303; moved to B.Cu
- R42: renamed from R302; moved to B.Cu
- R43: renamed from R304; moved to B.Cu
- R44: renamed from R230; moved to B.Cu
- R45: renamed from R248; moved to B.Cu
- R46: renamed from R226; moved to B.Cu
- R47: renamed from R247; moved to B.Cu
- R48: renamed from R246; moved to B.Cu
- R49: renamed from R222; moved to B.Cu
- R50: renamed from R604; moved to B.Cu
- R51: renamed from R603; moved to B.Cu
- R52: renamed from R601; moved to B.Cu
- R53: renamed from R218; moved to B.Cu
- R54: renamed from R245; moved to B.Cu
- R55: renamed from R244; moved to B.Cu
- R56: renamed from R404; moved to B.Cu
- R57: renamed from R401; moved to B.Cu
- R58: renamed from R214; moved to B.Cu
- R59: renamed from R101; moved to B.Cu
- R60: renamed from R243; moved to B.Cu
- R61: renamed from R210; moved to B.Cu
- R62: renamed from R408; moved to B.Cu
- R63: renamed from R242; moved to B.Cu
- R64: renamed from R206; moved to B.Cu
- R65: renamed from R241; moved to B.Cu
- R66: renamed from R202; moved to B.Cu
- R67: renamed from R607; moved to B.Cu
- R68: renamed from R608; moved to B.Cu
- R69: renamed from R609; moved to B.Cu
- R70: renamed from R613; moved to B.Cu
- R71: renamed from R614; moved to B.Cu
- R72: renamed from R615; moved to B.Cu
- R73: renamed from R233; moved to B.Cu
- R74: renamed from R201; moved to B.Cu
- R75: renamed from R234; moved to B.Cu
- R76: renamed from R205; moved to B.Cu
- R77: renamed from R235; moved to B.Cu
- R78: renamed from R209; moved to B.Cu
- R79: renamed from R236; moved to B.Cu
- R80: renamed from R213; moved to B.Cu
- R81: renamed from R237; moved to B.Cu
- R82: renamed from R217; moved to B.Cu
- R83: renamed from R238; moved to B.Cu
- R84: renamed from R221; moved to B.Cu
- R85: renamed from R239; moved to B.Cu
- R86: renamed from R225; moved to B.Cu
- R87: renamed from R240; moved to B.Cu
- R88: renamed from R229; moved to B.Cu
- moved R27 220.7 mm to (214.8, 153.2), turned to 180 degrees
- moved Q1 220.2 mm to (214.8, 150.4), turned to 180 degrees
- moved D23 220.0 mm to (208.4, 150.4)
- moved R57 218.9 mm to (211.6, 148.6)
- moved TP1 217.2 mm to (195.7, 146.1)
- moved D13 215.6 mm to (208.4, 150.4)
- moved D17 213.4 mm to (220.5, 143.8)
- moved D18 212.7 mm to (220.5, 147.6)
- moved TP3 211.2 mm to (204.3, 149.6)
- moved R26 211.0 mm to (211.6, 146.6)
- moved D22 211.0 mm to (214.8, 150.4), turned to 180 degrees
- moved R56 208.1 mm to (211.6, 146.6), turned to 180 degrees
- moved Q2 207.3 mm to (211.6, 141.7)
- moved R22 205.1 mm to (200.5, 146.6), turned to 180 degrees
- moved TP2 200.9 mm to (196.1, 134.0)
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- renumbered C402 to C1, C217 to C2, C405 to C3, C102 to C4, C218 to C5, C311 to C6, C307 to C7, C304 to C8, C303 to C9, D201 to D1, D407 to D10, D204 to D11, D206 to D12, D405 to D13, D208 to D14, D210 to D15, D403 to D16, D401 to D17, D402 to D18, D216 to D19, D203 to D2, D214 to D20, D212 to D21, D205 to D3, D207 to D4, D209 to D5, D211 to D6, D213 to D7, D215 to D8, D202 to D9, H101 to H1, H102 to H2, H104 to H3, H103 to H4, J602 to J1, J208 to J10, J209 to J11, J501 to J12, J210 to J13, J211 to J14, J212 to J15, J213 to J16, J604 to J17, J601 to J18, J104 to J19, J603 to J2, J103 to J20, J102 to J21, J101 to J22, J216 to J23, J215 to J24, J214 to J25, J301 to J26, J302 to J27, J201 to J3, J202 to J4, J203 to J5, J204 to J6, J205 to J7, J206 to J8, J207 to J9, L401 to L1, L301 to L2, R203 to R1, R503 to R10, R501 to R11, R610 to R12, R611 to R13, R612 to R14, R616 to R15, R617 to R16, R618 to R17, R231 to R18, R204 to R19, R207 to R2, R208 to R20, R407 to R21, R405 to R22, R406 to R23, R212 to R24, R216 to R25, R403 to R26, R402 to R27, R309 to R28, R220 to R29, R211 to R3, R606 to R30, R605 to R31, R602 to R32, R232 to R33, R228 to R34, R224 to R35, R305 to R36, R306 to R37, R307 to R38, R308 to R39, R215 to R4, R219 to R5, R223 to R6, R227 to R7, R504 to R8, R502 to R9, TP401 to TP1, TP402 to TP2, TP403 to TP3, TP101 to TP4, TP102 to TP5, TP301 to TP6, TP302 to TP7, U201 to U1, U402 to U2, U202 to U3, U101 to U4, U102 to U5, U401 to U6, U302 to U7, U103 to U8, U301 to U9
Routing:
- net +5V: track 0.00 -> 133.0 mm, vias 0 -> 2
- net +3V3: track 0.00 -> 111.3 mm, vias 0 -> 24
- net GND: track 0.00 -> 110.0 mm, vias 0 -> 41
- net /BUTTON_MISO: track 0.00 -> 72.6 mm, vias 0 -> 1
- net /BUTTON_SCK: track 0.00 -> 69.1 mm, vias 0 -> 2
- net Net-(U1-D0): track 0.00 -> 60.4 mm, vias 0 -> 1
- net /~{BUTTON_LD}: track 0.00 -> 59.5 mm, vias 0 -> 2
- net Net-(U1-D1): track 0.00 -> 48.3 mm, vias 0 -> 1
- net /SPI0_SCK: track 0.00 -> 47.5 mm
- net /~{SPI0_CS}: track 0.00 -> 43.1 mm, vias 0 -> 1
- net /SPI0_MISO: track 0.00 -> 40.0 mm, vias 0 -> 1
- net Net-(U1-D2): track 0.00 -> 39.4 mm, vias 0 -> 3
- net Net-(U1-D3): track 0.00 -> 38.0 mm, vias 0 -> 1
- net /SPI0_MOSI: track 0.00 -> 37.3 mm
- net Net-(D16-K): track 0.00 -> 36.4 mm, vias 0 -> 3
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- added copper zone on In1.Cu, net +3V3
- added copper zone on In1.Cu, net +3V3A
- added copper zone on In1.Cu, net /Encoder Inputs/ENC_VCC
- added copper zone on In2.Cu, net GND
- added copper zone on In2.Cu, net GNDA
Other:
- outline, holes or cut-outs redrawn
- copper layers 2 -> 4
- board text added: "3V3"
- board text added: "5V"
