File: circuit-boards/Pico-ButtonBoard-v1/button-input.kicad_sch (KiCad schematic)
At the start: 100 parts, among them J1 B1, J10 B9, J11 B10, J12 B11, J13 B12, J14 B13, J15 B14, J16 B15, J2 B0, J3 B2, J4 B3, J5 B4, J6 B5, J7 B6, J8 B7, J9 B8, U1 SN74HC165DR, U2 SN74HC165DR

Commit message: Update footprints
Signed-off-by: Scott Berman <sgberman1@gmail.com>
Parts:
- D201: renamed from D1; DIST (none) -> Digikey; DIST P/N (none) -> 1080-1419-1-ND; MFG (none) -> Everlight; MFG P/N (none) -> QTLP650D4TR/QT15-21SYGD/S530-E2/TR8
- D202: renamed from D9; DIST (none) -> Digikey; DIST P/N (none) -> 1080-1419-1-ND; MFG (none) -> Everlight; MFG P/N (none) -> QTLP650D4TR/QT15-21SYGD/S530-E2/TR8
- D203: renamed from D2; DIST (none) -> Digikey; DIST P/N (none) -> 1080-1419-1-ND; MFG (none) -> Everlight; MFG P/N (none) -> QTLP650D4TR/QT15-21SYGD/S530-E2/TR8
- D204: renamed from D10; DIST (none) -> Digikey; DIST P/N (none) -> 1080-1419-1-ND; MFG (none) -> Everlight; MFG P/N (none) -> QTLP650D4TR/QT15-21SYGD/S530-E2/TR8
- D205: renamed from D3; DIST (none) -> Digikey; DIST P/N (none) -> 1080-1419-1-ND; MFG (none) -> Everlight; MFG P/N (none) -> QTLP650D4TR/QT15-21SYGD/S530-E2/TR8
- D206: renamed from D11; DIST (none) -> Digikey; DIST P/N (none) -> 1080-1419-1-ND; MFG (none) -> Everlight; MFG P/N (none) -> QTLP650D4TR/QT15-21SYGD/S530-E2/TR8
- D207: renamed from D4; DIST (none) -> Digikey; DIST P/N (none) -> 1080-1419-1-ND; MFG (none) -> Everlight; MFG P/N (none) -> QTLP650D4TR/QT15-21SYGD/S530-E2/TR8
- D208: renamed from D12; DIST (none) -> Digikey; DIST P/N (none) -> 1080-1419-1-ND; MFG (none) -> Everlight; MFG P/N (none) -> QTLP650D4TR/QT15-21SYGD/S530-E2/TR8
- D209: renamed from D5; DIST (none) -> Digikey; DIST P/N (none) -> 1080-1419-1-ND; MFG (none) -> Everlight; MFG P/N (none) -> QTLP650D4TR/QT15-21SYGD/S530-E2/TR8
- D210: renamed from D13; DIST (none) -> Digikey; DIST P/N (none) -> 1080-1419-1-ND; MFG (none) -> Everlight; MFG P/N (none) -> QTLP650D4TR/QT15-21SYGD/S530-E2/TR8
- D211: renamed from D6; DIST (none) -> Digikey; DIST P/N (none) -> 1080-1419-1-ND; MFG (none) -> Everlight; MFG P/N (none) -> QTLP650D4TR/QT15-21SYGD/S530-E2/TR8
- D212: renamed from D14; DIST (none) -> Digikey; DIST P/N (none) -> 1080-1419-1-ND; MFG (none) -> Everlight; MFG P/N (none) -> QTLP650D4TR/QT15-21SYGD/S530-E2/TR8
- D213: renamed from D7; DIST (none) -> Digikey; DIST P/N (none) -> 1080-1419-1-ND; MFG (none) -> Everlight; MFG P/N (none) -> QTLP650D4TR/QT15-21SYGD/S530-E2/TR8
- D214: renamed from D15; DIST (none) -> Digikey; DIST P/N (none) -> 1080-1419-1-ND; MFG (none) -> Everlight; MFG P/N (none) -> QTLP650D4TR/QT15-21SYGD/S530-E2/TR8
- D215: renamed from D8; DIST (none) -> Digikey; DIST P/N (none) -> 1080-1419-1-ND; MFG (none) -> Everlight; MFG P/N (none) -> QTLP650D4TR/QT15-21SYGD/S530-E2/TR8
- D216: renamed from D16; DIST (none) -> Digikey; DIST P/N (none) -> 1080-1419-1-ND; MFG (none) -> Everlight; MFG P/N (none) -> QTLP650D4TR/QT15-21SYGD/S530-E2/TR8
- R233: renamed from R2; DIST (none) -> Digikey; DIST P/N (none) -> 541-10.0KCCT-ND; MFG (none) -> Vishay Dale; MFG P/N (none) -> CRCW080510K0FKEA
- R234: renamed from R3; DIST (none) -> Digikey; DIST P/N (none) -> 541-10.0KCCT-ND; MFG (none) -> Vishay Dale; MFG P/N (none) -> CRCW080510K0FKEA
- R235: renamed from R4; DIST (none) -> Digikey; DIST P/N (none) -> 541-10.0KCCT-ND; MFG (none) -> Vishay Dale; MFG P/N (none) -> CRCW080510K0FKEA
- R236: renamed from R5; DIST (none) -> Digikey; DIST P/N (none) -> 541-10.0KCCT-ND; MFG (none) -> Vishay Dale; MFG P/N (none) -> CRCW080510K0FKEA
- R237: renamed from R6; DIST (none) -> Digikey; DIST P/N (none) -> 541-10.0KCCT-ND; MFG (none) -> Vishay Dale; MFG P/N (none) -> CRCW080510K0FKEA
- R238: renamed from R7; DIST (none) -> Digikey; DIST P/N (none) -> 541-10.0KCCT-ND; MFG (none) -> Vishay Dale; MFG P/N (none) -> CRCW080510K0FKEA
- R239: renamed from R8; DIST (none) -> Digikey; DIST P/N (none) -> 541-10.0KCCT-ND; MFG (none) -> Vishay Dale; MFG P/N (none) -> CRCW080510K0FKEA
- R240: renamed from R9; DIST (none) -> Digikey; DIST P/N (none) -> 541-10.0KCCT-ND; MFG (none) -> Vishay Dale; MFG P/N (none) -> CRCW080510K0FKEA
- R241: renamed from R41; DIST (none) -> Digikey; DIST P/N (none) -> 541-10.0KCCT-ND; MFG (none) -> Vishay Dale; MFG P/N (none) -> CRCW080510K0FKEA
- R242: renamed from R42; DIST (none) -> Digikey; DIST P/N (none) -> 541-10.0KCCT-ND; MFG (none) -> Vishay Dale; MFG P/N (none) -> CRCW080510K0FKEA
- R243: renamed from R43; DIST (none) -> Digikey; DIST P/N (none) -> 541-10.0KCCT-ND; MFG (none) -> Vishay Dale; MFG P/N (none) -> CRCW080510K0FKEA
- R244: renamed from R44; DIST (none) -> Digikey; DIST P/N (none) -> 541-10.0KCCT-ND; MFG (none) -> Vishay Dale; MFG P/N (none) -> CRCW080510K0FKEA
- R245: renamed from R45; DIST (none) -> Digikey; DIST P/N (none) -> 541-10.0KCCT-ND; MFG (none) -> Vishay Dale; MFG P/N (none) -> CRCW080510K0FKEA
- R246: renamed from R46; DIST (none) -> Digikey; DIST P/N (none) -> 541-10.0KCCT-ND; MFG (none) -> Vishay Dale; MFG P/N (none) -> CRCW080510K0FKEA
- R247: renamed from R47; DIST (none) -> Digikey; DIST P/N (none) -> 541-10.0KCCT-ND; MFG (none) -> Vishay Dale; MFG P/N (none) -> CRCW080510K0FKEA
- R248: renamed from R48; DIST (none) -> Digikey; DIST P/N (none) -> 541-10.0KCCT-ND; MFG (none) -> Vishay Dale; MFG P/N (none) -> CRCW080510K0FKEA
- renumbered C2 to C201, C11 to C202, C3 to C203, C12 to C204, C4 to C205, C13 to C206, C6 to C207, C14 to C208, C7 to C209, C15 to C210, C8 to C211, C16 to C212, C9 to C213, C17 to C214, C10 to C215, C18 to C216, C5 to C217, C1 to C218, J2 to J201, J1 to J202, J3 to J203, J4 to J204, J5 to J205, J6 to J206, J7 to J207, J8 to J208, J9 to J209, J10 to J210, J11 to J211, J12 to J212, J13 to J213, J14 to J214, J15 to J215, J16 to J216, R1 to R201, R25 to R202, R10 to R203, R26 to R204, R11 to R205, R27 to R206, R12 to R207, R28 to R208, R13 to R209, R29 to R210, R14 to R211, R30 to R212, R15 to R213, R31 to R214, R16 to R215, R32 to R216, R17 to R217, R33 to R218, R18 to R219, R34 to R220, R19 to R221, R35 to R222, R20 to R223, R36 to R224, R21 to R225, R37 to R226, R22 to R227, R38 to R228, R23 to R229, R39 to R230, R24 to R231, R40 to R232, U1 to U201, U2 to U202
Other:
- title: (none) -> Pico Button Board

Commit message: Pico Button Board initial placement
Signed-off-by: Scott Berman <sgberman1@gmail.com>
Parts:
- C201, C202, C203, C204, C205, C206, C207, C208, C209, C210, C211, C212, C213, C214, C215, C216, C217, C218: LCSC Part # C519981 -> (none)
- J201, J202, J203, J204, J205, J206, J207, J208, J209, J210, J211, J212, J213, J214, J215, J216: footprint Pico-ButtonBoard:Molex-70555-0036 -> Pico-ButtonBoard:Molex-70543-0001; DIST P/N WM4175-ND -> WM4824-ND; MFG P/N 70555-0036 -> 70543-0036

Commit message: Pico Button Board initial pcb checkin
Signed-off-by: Scott Berman <sgberman1@gmail.com>
Parts:
- renumbered C216 to C12, C214 to C13, C212 to C14, C210 to C15, C217 to C2, C208 to C25, C206 to C28, C204 to C30, C202 to C33, C201 to C34, C203 to C35, C205 to C36, C207 to C37, C209 to C38, C211 to C39, C213 to C40, C215 to C41, C218 to C5, D201 to D1, D204 to D11, D206 to D12, D208 to D14, D210 to D15, D216 to D19, D203 to D2, D214 to D20, D212 to D21, D205 to D3, D207 to D4, D209 to D5, D211 to D6, D213 to D7, D215 to D8, D202 to D9, J208 to J10, J209 to J11, J210 to J13, J211 to J14, J212 to J15, J213 to J16, J216 to J23, J215 to J24, J214 to J25, J201 to J3, J202 to J4, J203 to J5, J204 to J6, J205 to J7, J206 to J8, J207 to J9, R203 to R1, R231 to R18, R204 to R19, R207 to R2, R208 to R20, R212 to R24, R216 to R25, R220 to R29, R211 to R3, R232 to R33, R228 to R34, R224 to R35, R215 to R4, R230 to R44, R248 to R45, R226 to R46, R247 to R47, R246 to R48, R222 to R49, R219 to R5, R218 to R53, R245 to R54, R244 to R55, R214 to R58, R223 to R6, R243 to R60, R210 to R61, R242 to R63, R206 to R64, R241 to R65, R202 to R66, R227 to R7, R233 to R73, R201 to R74, R234 to R75, R205 to R76, R235 to R77, R209 to R78, R236 to R79, R213 to R80, R237 to R81, R217 to R82, R238 to R83, R221 to R84, R239 to R85, R225 to R86, R240 to R87, R229 to R88, U201 to U1, U202 to U3

Commit message: Changed button input circuit to use mux. Changed ADC3 to an external SPI ADC
Signed-off-by: Scott Berman <sgberman1@gmail.com>
Parts:
- removed U1, U3: SN74HC165DR, Package_SO:SO-16_3.9x9.9mm_P1.27mm, symbol 74xx:74HC165
- added U1, U3: SN74HC151DR, Package_SO:SOIC-16_3.9x9.9mm_P1.27mm, symbol 74xx:74LS151
- renumbered C12 to C11, C13 to C12, C14 to C13, C15 to C14, C25 to C24, C28 to C27, C30 to C29, C33 to C32, C34 to C33, C35 to C34, C36 to C35, C37 to C36, C38 to C37, C39 to C38, C40 to C39, C41 to C40, J13 to J12, J14 to J13, J15 to J14, J16 to J15, J23 to J22, J24 to J23, J25 to J24, R18 to R15, R19 to R16, R20 to R17, R24 to R21, R25 to R22, R29 to R25, R33 to R29, R34 to R30, R35 to R31, R44 to R40, R45 to R41, R46 to R42, R47 to R43, R48 to R44, R49 to R45, R53 to R49, R54 to R50, R55 to R51, R58 to R54, R60 to R56, R61 to R57, R63 to R59, R64 to R60, R65 to R61, R66 to R62, R73 to R66, R74 to R67, R75 to R68, R76 to R69, R77 to R70, R78 to R71, R79 to R72, R80 to R73, R81 to R74, R82 to R75, R83 to R76, R84 to R77, R85 to R78, R86 to R79, R87 to R80, R88 to R81
Connections:
- net +3V3: now also U1.16 (VCC), U3.16 (VCC)
- net GND: now also U1.7 (~{E}), U1.8 (GND), U3.7 (~{E}), U3.8 (GND)
- net at R76.2: now also U1.14 (I5)
- net at R74.2: now also U1.15 (I4)
- net at R80.2: now also U1.12 (I7)
- net at R72.2: now also U1.1 (I3)
- net at R61.2: now also U3.4 (I0)
- net at R50.2: now also U3.15 (I4)
- net at R43.2: now also U3.13 (I6)
- net at R59.2: now also U3.3 (I1)
- net at R56.2: now also U3.2 (I2)
- net at R51.2: now also U3.1 (I3)
- net at R44.2: now also U3.14 (I5)
- net at R41.2: now also U3.12 (I7)
- net at R66.2: now also U1.4 (I0)
- net at R68.2: now also U1.3 (I1)
- net at R78.2: now also U1.13 (I6)
- net at R70.2: now also U1.2 (I2)
- new net BUTTON_DA: U1.6 (~{Z})
- new net BUTTON_DB: U3.6 (~{Z})
- new net BUTTON_S0: U1.11 (S0), U3.11 (S0)
- new net BUTTON_S1: U1.10 (S1), U3.10 (S1)
- new net BUTTON_S2: U1.9 (S2), U3.9 (S2)
Other:
- moved on the sheet: C2

Commit message: Add power over CAN to supply joystick from button interfaces.
Signed-off-by: Scott Berman <sgberman1@gmail.com>
Parts:
- renumbered C12 to C10, C13 to C11, C14 to C12, C11 to C9, D12 to D13, D14 to D15, D15 to D16, D19 to D20, D20 to D21, D21 to D22, R25 to R28, R29 to R32, R30 to R33, R31 to R34, R40 to R35, R41 to R36, R42 to R37, R43 to R38, R44 to R39, R45 to R40, R49 to R44, R50 to R49, R51 to R50
Changed lines of the file:
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@@
 	(title_block
 		(title "Pico Button Board")
-		(date "2025-12-29")
+		(date "2025-12-30")
 		(rev "1")
 	)
@@
 		(on_board yes)
 		(dnp no)
-		(property "Reference" "R29"
+		(property "Reference" "R32"
 			(at 209.55 156.972 90)
 			(effects
@@
 			(project "Pico-ButtonBoard-v1"
 				(path "/644201a9-3a2f-4df3-9c93-2ae55394df4b/0ff2bd57-0772-402e-b5ad-a11115b3bfe5"
-					(reference "R29")
+					(reference "R32")
 					(unit 1)
 				)
@@
 		(on_board yes)
 		(dnp no)
-		(property "Reference" "R49"
+		(property "Reference" "R44"
 			(at 171.196 162.052 90)
 			(effects
@@
 			(project "Pico-ButtonBoard-v1"
 				(path "/644201a9-3a2f-4df3-9c93-2ae55394df4b/0ff2bd57-0772-402e-b5ad-a11115b3bfe5"
-					(reference "R49")
+					(reference "R44")
 					(unit 1)
 				)
@@
 		(on_board yes)
 		(dnp no)
-		(property "Reference" "D21"
+		(property "Reference" "D22"
 			(at 184.15 170.434 0)
 			(effects
@@
 			(project "Pico-ButtonBoard-v1"
 				(path "/644201a9-3a2f-4df3-9c93-2ae55394df4b/0ff2bd57-0772-402e-b5ad-a11115b3bfe5"
-					(reference "D21")
+					(reference "D22")
 					(unit 1)
 				)
@@
 		(on_board yes)
 		(dnp no)
-		(property "Reference" "C11"
+		(property "Reference" "C9"
 			(at 204.47 236.22 90)
 			(effects
@@
 			(project "Pico-ButtonBoard-v1"
 				(path "/644201a9-3a2f-4df3-9c93-2ae55394df4b/0ff2bd57-0772-402e-b5ad-a11115b3bfe5"
-					(reference "C11")
+					(reference "C9")
 					(unit 1)
 				)
@@
 		(on_board yes)
 		(dnp no)
-		(property "Reference" "D20"
+		(property "Reference" "D21"
 			(at 194.31 170.434 0)
 			(effects
@@
 			(project "Pico-ButtonBoard-v1"
 				(path "/644201a9-3a2f-4df3-9c93-2ae55394df4b/0ff2bd57-0772-402e-b5ad-a11115b3bfe5"
-					(reference "D20")
+					(reference "D21")
 					(unit 1)
 				)
@@
 		(on_board yes)
 		(dnp no)
-		(property "Reference" "R25"
+		(property "Reference" "R28"
 			(at 176.53 156.972 90)
 			(effects
@@
 			(project "Pico-ButtonBoard-v1"
 				(path "/644201a9-3a2f-4df3-9c93-2ae55394df4b/0ff2bd57-0772-402e-b5ad-a11115b3bfe5"
-					(reference "R25")
+					(reference "R28")
 					(unit 1)
 				)
@@
 		(on_board yes)
 		(dnp no)
-		(property "Reference" "R45"
+		(property "Reference" "R40"
 			(at 182.626 162.052 90)
 			(effects
@@
 			(project "Pico-ButtonBoard-v1"
 				(path "/644201a9-3a2f-4df3-9c93-2ae55394df4b/0ff2bd57-0772-402e-b5ad-a11115b3bfe5"
-					(reference "R45")
+					(reference "R40")
 					(unit 1)
 				)
@@
 		(on_board yes)
 		(dnp no)
-		(property "Reference" "R50"
+		(property "Reference" "R49"
 			(at 227.33 207.264 90)
 			(effects
@@
 			(project "Pico-ButtonBoard-v1"
 				(path "/644201a9-3a2f-4df3-9c93-2ae55394df4b/0ff2bd57-0772-402e-b5ad-a11115b3bfe5"
-					(reference "R50")
+					(reference "R49")
 					(unit 1)
 				)
@@
 		(on_board yes)
 		(dnp no)
-		(property "Reference" "R30"
+		(property "Reference" "R33"
 			(at 198.12 156.972 90)
 			(effects
@@
 			(project "Pico-ButtonBoard-v1"
 				(path "/644201a9-3a2f-4df3-9c93-2ae55394df4b/0ff2bd57-0772-402e-b5ad-a11115b3bfe5"
-					(reference "R30")
+					(reference "R33")
 					(unit 1)
 				)
@@
 		(on_board yes)
 		(dnp no)
-		(property "Reference" "R43"
+		(property "Reference" "R38"
 			(at 227.33 219.964 90)
 			(effects
@@
 			(project "Pico-ButtonBoard-v1"
 				(path "/644201a9-3a2f-4df3-9c93-2ae55394df4b/0ff2bd57-0772-402e-b5ad-a11115b3bfe5"
-					(reference "R43")
+					(reference "R38")
 					(unit 1)
 				)
@@
 		(on_board yes)
 		(dnp no)
-		(property "Reference" "C14"
+		(property "Reference" "C12"
 			(at 171.45 236.22 90)
 			(effects
@@
 			(project "Pico-ButtonBoard-v1"
 				(path "/644201a9-3a2f-4df3-9c93-2ae55394df4b/0ff2bd57-0772-402e-b5ad-a11115b3bfe5"
-					(reference "C14")
+					(reference "C12")
 					(unit 1)
 				)
@@
 		(on_board yes)
 		(dnp no)
-		(property "Reference" "D14"
+		(property "Reference" "D15"
 			(at 161.29 170.434 0)
 			(effects
@@
 			(project "Pico-ButtonBoard-v1"
 				(path "/644201a9-3a2f-4df3-9c93-2ae55394df4b/0ff2bd57-0772-402e-b5ad-a11115b3bfe5"
-					(reference "D14")
+					(reference "D15")
 					(unit 1)
 				)
@@
 		(on_board yes)
 		(dnp no)
-		(property "Reference" "D19"
+		(property "Reference" "D20"
 			(at 205.74 170.434 0)
 			(effects
@@
 			(project "Pico-ButtonBoard-v1"
 				(path "/644201a9-3a2f-4df3-9c93-2ae55394df4b/0ff2bd57-0772-402e-b5ad-a11115b3bfe5"
-					(reference "D19")
+					(reference "D20")
 					(unit 1)
 				)
@@
 		(on_board yes)
 		(dnp no)
-		(property "Reference" "C12"
+		(property "Reference" "C10"
 			(at 193.04 236.22 90)
 			(effects
@@
 			(project "Pico-ButtonBoard-v1"
 				(path "/644201a9-3a2f-4df3-9c93-2ae55394df4b/0ff2bd57-0772-402e-b5ad-a11115b3bfe5"
-					(reference "C12")
+					(reference "C10")
 					(unit 1)
 				)
@@
 		(on_board yes)
 		(dnp no)
-		(property "Reference" "C13"
+		(property "Reference" "C11"
 			(at 182.88 236.22 90)
 			(effects
@@
 			(project "Pico-ButtonBoard-v1"
 				(path "/644201a9-3a2f-4df3-9c93-2ae55394df4b/0ff2bd57-0772-402e-b5ad-a11115b3bfe5"
-					(reference "C13")
+					(reference "C11")
 					(unit 1)
 				)
@@
 		(on_board yes)
 		(dnp no)
-		(property "Reference" "D12"
+		(property "Reference" "D13"
 			(at 149.86 170.434 0)
 			(effects
@@
 			(project "Pico-ButtonBoard-v1"
 				(path "/644201a9-3a2f-4df3-9c93-2ae55394df4b/0ff2bd57-0772-402e-b5ad-a11115b3bfe5"
-					(reference "D12")
+					(reference "D13")
 					(unit 1)
 				)
@@
 		(on_board yes)
 		(dnp no)
-		(property "Reference" "R41"
+		(property "Reference" "R36"
 			(at 227.33 226.314 90)
 			(effects
@@
 			(project "Pico-ButtonBoard-v1"
 				(path "/644201a9-3a2f-4df3-9c93-2ae55394df4b/0ff2bd57-0772-402e-b5ad-a11115b3bfe5"
-					(reference "R41")
+					(reference "R36")
 					(unit 1)
 				)
@@
 		(on_board yes)
 		(dnp no)
-		(property "Reference" "R31"
+		(property "Reference" "R34"
 			(at 187.96 156.972 90)
 			(effects
@@
 			(project "Pico-ButtonBoard-v1"
 				(path "/644201a9-3a2f-4df3-9c93-2ae55394df4b/0ff2bd57-0772-402e-b5ad-a11115b3bfe5"
-					(reference "R31")
+					(reference "R34")
 					(unit 1)
 				)
@@
 		(on_board yes)
 		(dnp no)
-		(property "Reference" "R44"
+		(property "Reference" "R39"
 			(at 227.33 213.614 90)
 			(effects
@@
 			(project "Pico-ButtonBoard-v1"
 				(path "/644201a9-3a2f-4df3-9c93-2ae55394df4b/0ff2bd57-0772-402e-b5ad-a11115b3bfe5"
-					(reference "R44")
+					(reference "R39")
 					(unit 1)
 				)
@@
 		(on_board yes)
 		(dnp no)
-		(property "Reference" "D15"
+		(property "Reference" "D16"
 			(at 172.72 170.434 0)
 			(effects
@@
 			(project "Pico-ButtonBoard-v1"
 				(path "/644201a9-3a2f-4df3-9c93-2ae55394df4b/0ff2bd57-0772-402e-b5ad-a11115b3bfe5"
-					(reference "D15")
+					(reference "D16")
 					(unit 1)
 				)
@@
 		(on_board yes)
 		(dnp no)
-		(property "Reference" "R51"
+		(property "Reference" "R50"
 			(at 227.33 200.914 90)
 			(effects
@@
 			(project "Pico-ButtonBoard-v1"
 				(path "/644201a9-3a2f-4df3-9c93-2ae55394df4b/0ff2bd57-0772-402e-b5ad-a11115b3bfe5"
-					(reference "R51")
+					(reference "R50")
 					(unit 1)
 				)
@@
 		(on_board yes)
 		(dnp no)
-		(property "Reference" "R40"
+		(property "Reference" "R35"
 			(at 204.216 162.052 90)
 			(effects
@@
 			(project "Pico-ButtonBoard-v1"
 				(path "/644201a9-3a2f-4df3-9c93-2ae55394df4b/0ff2bd57-0772-402e-b5ad-a11115b3bfe5"
-					(reference "R40")
+					(reference "R35")
 					(unit 1)
 				)
@@
 		(on_board yes)
 		(dnp no)
-		(property "Reference" "R42"
+		(property "Reference" "R37"
 			(at 192.786 162.052 90)
 			(effects
@@
 			(project "Pico-ButtonBoard-v1"
 				(path "/644201a9-3a2f-4df3-9c93-2ae55394df4b/0ff2bd57-0772-402e-b5ad-a11115b3bfe5"
-					(reference "R42")
+					(reference "R37")
 					(unit 1)
 				)

Commit message: Change diodes to schottky. Change 5V setpoint to 5.18V
Signed-off-by: Scott Berman <sgberman1@gmail.com>
Other:
- note added: "1-Button Pressed 0-Button Open"
Changed lines of the file:
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@@
 	(title_block
 		(title "Pico Button Board")
-		(date "2025-12-30")
+		(date "2025-12-31")
 		(rev "1")
 	)
+	(text "1-Button Pressed\n0-Button Open"
+		(exclude_from_sim no)
+		(at 378.46 112.522 0)
+		(effects
+			(font
+				(size 1.27 1.27)
+			)
+			(justify left)
+		)
+	)
 	(junction
 		(at 138.43 151.13)
@@
 		)
 		(property "Value" "0.1uF-25V-10%-0805"
-			(at 329.184 100.33 90)
+			(at 328.168 100.33 0)
 			(effects
 				(font
 					(size 1.27 1.27)
 				)
+				(justify right)
 			)
 		)

Commit message: Added power indicator to button board
Signed-off-by: Scott Berman <sgberman1@gmail.com>
Parts:
- renumbered C29 to C30, C32 to C33, C33 to C34, C34 to C35, C35 to C36, C36 to C37, C37 to C38, C38 to C39, C39 to C40, C40 to C41, D13 to D14, D15 to D16, D16 to D17, R59 to R63, R60 to R65, R61 to R66, R62 to R67, R66 to R71, R67 to R72, R68 to R73, R69 to R74, R70 to R75, R71 to R76, R72 to R77, R73 to R78, R74 to R79, R75 to R80, R76 to R81, R77 to R82, R78 to R83, R79 to R84, R80 to R85, R81 to R86
