File: circuit-boards/Pico-ButtonBoard-v1/power-supply.kicad_sch (KiCad schematic)
At the start: 25 parts, among them Q1 BSS123, Q3 BSS123, U7 ITS41k0S-ME-N, U9 TPS54202DDC

Commit message: Update footprints
Signed-off-by: Scott Berman <sgberman1@gmail.com>
Parts:
- removed C34: 0.22uF-50V-10%-0805, Capacitor_SMD:C_0805_2012Metric_Pad1.18x1.45mm_HandSolder, symbol Device:C_Small_US
- added C401: 10uF-10%-50V-1206, Capacitor_SMD:C_1206_3216Metric_Pad1.33x1.80mm_HandSolder, symbol Device:C_US
- added TP401, TP402, TP403: CAN_RX, TestPoint:TestPoint_Keystone_5000-5004_Miniature, symbol Connector:TestPoint
- C404: renamed from C35; DIST (none) -> Digikey; DIST P/N (none) -> 311-1109-1-ND; MFG (none) -> YAGEO; MFG P/N (none) -> CC0805JRNPO9BN680
- C405: renamed from C41; value 47uF-10%-16V-1206 -> 47uF-10%-16V-1210
- L401: renamed from L3; footprint (none) -> Pico-ButtonBoard:Cyntec-MS6-Inductor
- R401: renamed from R64; DIST (none) -> Digikey; DIST P/N (none) -> 541-10.0KCCT-ND; MFG (none) -> Vishay Dale; MFG P/N (none) -> CRCW080510K0FKEA
- R402: renamed from R63; DIST (none) -> Digikey; DIST P/N (none) -> 541-10.0KCCT-ND; MFG (none) -> Vishay Dale; MFG P/N (none) -> CRCW080510K0FKEA
- R403: renamed from R61; DIST (none) -> Digikey; DIST P/N (none) -> P20.0KCCT-ND; MFG (none) -> Panasonic; MFG P/N (none) -> ERJ-6ENF2002V
- R404: renamed from R62; DIST (none) -> Digikey; DIST P/N (none) -> P20.0KCCT-ND; MFG (none) -> Panasonic; MFG P/N (none) -> ERJ-6ENF2002V
- R405: renamed from R65; DIST (none) -> Digikey; DIST P/N (none) -> 311-100KCRCT-ND; MFG (none) -> YAGEO; MFG P/N (none) -> RC0805FR-07100KL
- R406: renamed from R66; value 20.0k-1%-0805 -> 20k-1%-0805; DIST (none) -> Digikey; DIST P/N (none) -> P20.0KCCT-ND; MFG (none) -> Panasonic; MFG P/N (none) -> ERJ-6ENF2002V
- R407: renamed from R60; DIST (none) -> Digikey; DIST P/N (none) -> RMCF0805FT12K4CT-ND; MFG (none) -> Stackpole; MFG P/N (none) -> RMCF0805FT12K4
- R408: renamed from R59; DIST (none) -> Digikey; DIST P/N (none) -> 311-100KCRCT-ND; MFG (none) -> YAGEO; MFG P/N (none) -> RC0805FR-07100KL
- renumbered C40 to C402, C36 to C403, D26 to D401, D21 to D402, D17 to D403, D20 to D404, D18 to D405, D19 to D406, D22 to D407, Q3 to Q401, Q1 to Q402, U7 to U401, U9 to U402
Connections:
- net GND: now also C401.2
- net V_PS: now also TP401.1
- net at C404.1, C405.1, D407.2 (A)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: now also TP402.1
- net at D403.1 (K), R403.2, U401.2 (Vs): now also C401.1, TP403.1
Other:
- note added: "5V Power Supply"
- note added: "Battery Backup"
- note removed: "Hot Plug"
- title: (none) -> Pico Button Board

Commit message: Pico Button Board initial placement
Signed-off-by: Scott Berman <sgberman1@gmail.com>
Parts:
- C403: LCSC Part # C519981 -> (none)

Commit message: Pico Button Board initial pcb checkin
Signed-off-by: Scott Berman <sgberman1@gmail.com>
Parts:
- Q1: renamed from Q401; footprint Package_TO_SOT_SMD:SOT-23 -> Package_TO_SOT_SMD:SOT-23-3
- Q2: renamed from Q402; footprint Package_TO_SOT_SMD:SOT-23 -> Package_TO_SOT_SMD:SOT-23-3
- renumbered C402 to C1, C401 to C24, C404 to C27, C403 to C29, C405 to C3, D407 to D10, D405 to D13, D403 to D16, D401 to D17, D402 to D18, D406 to D22, D404 to D23, L401 to L1, R407 to R21, R405 to R22, R406 to R23, R403 to R26, R402 to R27, R404 to R56, R401 to R57, R408 to R62, TP401 to TP1, TP402 to TP2, TP403 to TP3, U402 to U2, U401 to U6
Changed lines of the file:
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@@
 		(dnp no)
 		(fields_autoplaced yes)
-		(property "Reference" "U402"
+		(property "Reference" "U2"
 			(at 251.46 113.03 0)
 			(effects
@@
 			(project ""
 				(path "/644201a9-3a2f-4df3-9c93-2ae55394df4b/dd046a3a-8e17-4277-b6b1-7e4df1560d2f"
-					(reference "U402")
+					(reference "U2")
 					(unit 1)
 				)
@@
 		(on_board yes)
 		(dnp no)
-		(property "Reference" "C404"
+		(property "Reference" "C27"
 			(at 285.75 135.89 90)
 			(effects
@@
 			(project "Pico-ButtonBoard-v1"
 				(path "/644201a9-3a2f-4df3-9c93-2ae55394df4b/dd046a3a-8e17-4277-b6b1-7e4df1560d2f"
-					(reference "C404")
+					(reference "C27")
 					(unit 1)
 				)
@@
 		(on_board yes)
 		(dnp no)
-		(property "Reference" "R408"
+		(property "Reference" "R62"
 			(at 288.29 128.016 90)
 			(effects
@@
 			(project "Pico-ButtonBoard-v1"
 				(path "/644201a9-3a2f-4df3-9c93-2ae55394df4b/dd046a3a-8e17-4277-b6b1-7e4df1560d2f"
-					(reference "R408")
+					(reference "R62")
 					(unit 1)
 				)
@@
 		(on_board yes)
 		(dnp no)
-		(property "Reference" "D405"
+		(property "Reference" "D13"
 			(at 112.268 152.4 90)
 			(effects
@@
 			(project "Pico-ButtonBoard-v1"
 				(path "/644201a9-3a2f-4df3-9c93-2ae55394df4b/dd046a3a-8e17-4277-b6b1-7e4df1560d2f"
-					(reference "D405")
+					(reference "D13")
 					(unit 1)
 				)
@@
 		(on_board yes)
 		(dnp no)
-		(property "Reference" "D403"
+		(property "Reference" "D16"
 			(at 68.072 117.602 0)
 			(effects
@@
 			(project ""
 				(path "/644201a9-3a2f-4df3-9c93-2ae55394df4b/dd046a3a-8e17-4277-b6b1-7e4df1560d2f"
-					(reference "D403")
+					(reference "D16")
 					(unit 1)
 				)
@@
 		(on_board yes)
 		(dnp no)
-		(property "Reference" "C401"
+		(property "Reference" "C24"
 			(at 81.28 143.7639 0)
 			(effects
@@
 			(project "Pico-ButtonBoard-v1"
 				(path "/644201a9-3a2f-4df3-9c93-2ae55394df4b/dd046a3a-8e17-4277-b6b1-7e4df1560d2f"
-					(reference "C401")
+					(reference "C24")
 					(unit 1)
 				)
@@
 		(on_board yes)
 		(dnp no)
-		(property "Reference" "R405"
+		(property "Reference" "R22"
 			(at 231.14 124.206 90)
 			(effects
@@
 			(project "Pico-ButtonBoard-v1"
 				(path "/644201a9-3a2f-4df3-9c93-2ae55394df4b/dd046a3a-8e17-4277-b6b1-7e4df1560d2f"
-					(reference "R405")
+					(reference "R22")
 					(unit 1)
 				)
@@
 		(on_board yes)
 		(dnp no)
-		(property "Reference" "L401"
+		(property "Reference" "L1"
 			(at 288.29 124.714 90)
 			(effects
@@
 			(project ""
 				(path "/644201a9-3a2f-4df3-9c93-2ae55394df4b/dd046a3a-8e17-4277-b6b1-7e4df1560d2f"
-					(reference "L401")
+					(reference "L1")
 					(unit 1)
 				)
@@
 		(on_board yes)
 		(dnp no)
-		(property "Reference" "R401"
+		(property "Reference" "R57"
 			(at 104.394 115.57 90)
 			(effects
@@
 			(project "Pico-ButtonBoard-v1"
 				(path "/644201a9-3a2f-4df3-9c93-2ae55394df4b/dd046a3a-8e17-4277-b6b1-7e4df1560d2f"
-					(reference "R401")
+					(reference "R57")
 					(unit 1)
 				)
@@
 		(on_board yes)
 		(dnp no)
-		(property "Reference" "R404"
+		(property "Reference" "R56"
 			(at 139.954 157.48 90)
 			(effects
@@
 			(project "Pico-ButtonBoard-v1"
 				(path "/644201a9-3a2f-4df3-9c93-2ae55394df4b/dd046a3a-8e17-4277-b6b1-7e4df1560d2f"
-					(reference "R404")
+					(reference "R56")
 					(unit 1)
 				)
@@
 		(on_board yes)
 		(dnp no)
-		(property "Reference" "D401"
+		(property "Reference" "D17"
 			(at 68.072 90.932 0)
 			(effects
@@
 			(project "Pico-ButtonBoard-v1"
 				(path "/644201a9-3a2f-4df3-9c93-2ae55394df4b/dd046a3a-8e17-4277-b6b1-7e4df1560d2f"
-					(reference "D401")
+					(reference "D17")
 					(unit 1)
 				)
@@
 		(on_board yes)
 		(dnp no)
-		(property "Reference" "D406"
+		(property "Reference" "D22"
 			(at 147.828 152.4 90)
 			(effects
@@
 			(project "Pico-ButtonBoard-v1"
 				(path "/644201a9-3a2f-4df3-9c93-2ae55394df4b/dd046a3a-8e17-4277-b6b1-7e4df1560d2f"
-					(reference "D406")
+					(reference "D22")
 					(unit 1)
 				)
@@
 		(on_board yes)
 		(dnp no)
-		(property "Reference" "D407"
+		(property "Reference" "D10"
 			(at 334.772 120.142 0)
 			(effects
@@
 			(project "Pico-ButtonBoard-v1"
 				(path "/644201a9-3a2f-4df3-9c93-2ae55394df4b/dd046a3a-8e17-4277-b6b1-7e4df1560d2f"
-					(reference "D407")
+					(reference "D10")
 					(unit 1)
 				)
@@
 		(on_board yes)
 		(dnp no)
-		(property "Reference" "C402"
+		(property "Reference" "C1"
 			(at 207.01 139.9539 0)
 			(effects
@@
 			(project ""
 				(path "/644201a9-3a2f-4df3-9c93-2ae55394df4b/dd046a3a-8e17-4277-b6b1-7e4df1560d2f"
-					(reference "C402")
+					(reference "C1")
 					(unit 1)
 				)
@@
 		(on_board yes)
 		(dnp yes)
-		(property "Reference" "TP403"
+		(property "Reference" "TP3"
 			(at 120.65 115.316 0)
 			(effects
@@
 			(project "Pico-ButtonBoard-v1"
 				(path "/644201a9-3a2f-4df3-9c93-2ae55394df4b/dd046a3a-8e17-4277-b6b1-7e4df1560d2f"
-					(reference "TP403")
+					(reference "TP3")
 					(unit 1)
 				)
@@
 		(on_board yes)
 		(dnp no)
-		(property "Reference" "R407"
+		(property "Reference" "R21"
 			(at 270.764 143.51 90)
 			(effects
@@
 			(project "Pico-ButtonBoard-v1"
 				(path "/644201a9-3a2f-4df3-9c93-2ae55394df4b/dd046a3a-8e17-4277-b6b1-7e4df1560d2f"
-					(reference "R407")
+					(reference "R21")
 					(unit 1)
 				)
@@
 		(on_board yes)
 		(dnp no)
-		(property "Reference" "C403"
+		(property "Reference" "C29"
 			(at 268.986 119.38 0)
 			(effects
@@
 			(project "Pico-ButtonBoard-v1"
 				(path "/644201a9-3a2f-4df3-9c93-2ae55394df4b/dd046a3a-8e17-4277-b6b1-7e4df1560d2f"
-					(reference "C403")
+					(reference "C29")
 					(unit 1)
 				)
@@
 		(on_board yes)
 		(dnp yes)
-		(property "Reference" "TP401"
+		(property "Reference" "TP1"
 			(at 184.15 88.646 0)
 			(effects
@@
 			(project "Pico-ButtonBoard-v1"
 				(path "/644201a9-3a2f-4df3-9c93-2ae55394df4b/dd046a3a-8e17-4277-b6b1-7e4df1560d2f"
-					(reference "TP401")
+					(reference "TP1")
 					(unit 1)
 				)
@@
 		(on_board yes)
 		(dnp no)
-		(property "Reference" "C405"
+		(property "Reference" "C3"
 			(at 314.96 139.9539 0)
 			(effects
@@
 			(project "Pico-ButtonBoard-v1"
 				(path "/644201a9-3a2f-4df3-9c93-2ae55394df4b/dd046a3a-8e17-4277-b6b1-7e4df1560d2f"
-					(reference "C405")
+					(reference "C3")
 					(unit 1)
 				)
@@
 		(on_board yes)
 		(dnp yes)
-		(property "Reference" "TP402"
+		(property "Reference" "TP2"
 			(at 316.23 117.856 0)
 			(effects
@@
 			(project "Pico-ButtonBoard-v1"
 				(path "/644201a9-3a2f-4df3-9c93-2ae55394df4b/dd046a3a-8e17-4277-b6b1-7e4df1560d2f"
-					(reference "TP402")
+					(reference "TP2")
 					(unit 1)
 				)
@@
 		(dnp no)
 		(fields_autoplaced yes)
-		(property "Reference" "U401"
+		(property "Reference" "U6"
 			(at 158.75 113.03 0)
 			(effects
@@
 			(project ""
 				(path "/644201a9-3a2f-4df3-9c93-2ae55394df4b/dd046a3a-8e17-4277-b6b1-7e4df1560d2f"
-					(reference "U401")
+					(reference "U6")
 					(unit 1)
 				)
@@
 		(on_board yes)
 		(dnp no)
-		(property "Reference" "R403"
+		(property "Reference" "R26"
 			(at 139.954 133.35 90)
 			(effects
@@
 			(project "Pico-ButtonBoard-v1"
 				(path "/644201a9-3a2f-4df3-9c93-2ae55394df4b/dd046a3a-8e17-4277-b6b1-7e4df1560d2f"
-					(reference "R403")
+					(reference "R26")
 					(unit 1)
 				)
@@
 		(on_board yes)
 		(dnp no)
-		(property "Reference" "D402"
+		(property "Reference" "D18"
 			(at 68.072 99.822 0)
 			(effects
@@
 			(project "Pico-ButtonBoard-v1"
 				(path "/644201a9-3a2f-4df3-9c93-2ae55394df4b/dd046a3a-8e17-4277-b6b1-7e4df1560d2f"
-					(reference "D402")
+					(reference "D18")
 					(unit 1)
 				)
@@
 		(on_board yes)
 		(dnp no)
-		(property "Reference" "D404"
+		(property "Reference" "D23"
 			(at 100.584 134.874 90)
 			(effects
@@
 			(project "Pico-ButtonBoard-v1"
 				(path "/644201a9-3a2f-4df3-9c93-2ae55394df4b/dd046a3a-8e17-4277-b6b1-7e4df1560d2f"
-					(reference "D404")
+					(reference "D23")
 					(unit 1)
 				)
@@
 		(on_board yes)
 		(dnp no)
-		(property "Reference" "R402"
+		(property "Reference" "R27"
 			(at 104.394 157.48 90)
 			(effects
@@
 			(project "Pico-ButtonBoard-v1"
 				(path "/644201a9-3a2f-4df3-9c93-2ae55394df4b/dd046a3a-8e17-4277-b6b1-7e4df1560d2f"
-					(reference "R402")
+					(reference "R27")
 					(unit 1)
 				)
@@
 		(on_board yes)
 		(dnp no)
-		(property "Reference" "R406"
+		(property "Reference" "R23"
 			(at 239.014 143.51 90)
 			(effects
@@
 			(project "Pico-ButtonBoard-v1"
 				(path "/644201a9-3a2f-4df3-9c93-2ae55394df4b/dd046a3a-8e17-4277-b6b1-7e4df1560d2f"
-					(reference "R406")
+					(reference "R23")
 					(unit 1)
 				)
@@
 		(dnp no)
 		(fields_autoplaced yes)
-		(property "Reference" "Q401"
+		(property "Reference" "Q1"
 			(at 124.46 143.5099 0)
 			(effects
@@
 			)
 		)
-		(property "Footprint" "Package_TO_SOT_SMD:SOT-23"
+		(property "Footprint" "Package_TO_SOT_SMD:SOT-23-3"
 			(at 123.19 146.685 0)
 			(effects
@@
 			(project "Pico-ButtonBoard-v1"
 				(path "/644201a9-3a2f-4df3-9c93-2ae55394df4b/dd046a3a-8e17-4277-b6b1-7e4df1560d2f"
-					(reference "Q401")
+					(reference "Q1")
 					(unit 1)
 				)
@@
 		(dnp no)
 		(fields_autoplaced yes)
-		(property "Reference" "Q402"
+		(property "Reference" "Q2"
 			(at 160.02 143.5099 0)
 			(effects
@@
 			)
 		)
-		(property "Footprint" "Package_TO_SOT_SMD:SOT-23"
+		(property "Footprint" "Package_TO_SOT_SMD:SOT-23-3"
 			(at 158.75 146.685 0)
 			(effects
@@
 			(project ""
 				(path "/644201a9-3a2f-4df3-9c93-2ae55394df4b/dd046a3a-8e17-4277-b6b1-7e4df1560d2f"
-					(reference "Q402")
+					(reference "Q2")
 					(unit 1)
 				)

Commit message: Changed button input circuit to use mux. Changed ADC3 to an external SPI ADC
Signed-off-by: Scott Berman <sgberman1@gmail.com>
Parts:
- renumbered C24 to C22, C27 to C26, C29 to C28, R21 to R18, R22 to R19, R23 to R20, R26 to R23, R27 to R24, R56 to R52, R57 to R53, R62 to R58
Changed lines of the file:
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@@
 	(title_block
 		(title "Pico Button Board")
-		(date "2025-12-28")
+		(date "2025-12-29")
 		(rev "1")
 	)
@@
 		(on_board yes)
 		(dnp no)
-		(property "Reference" "C27"
+		(property "Reference" "C26"
 			(at 285.75 135.89 90)
 			(effects
@@
 			(project "Pico-ButtonBoard-v1"
 				(path "/644201a9-3a2f-4df3-9c93-2ae55394df4b/dd046a3a-8e17-4277-b6b1-7e4df1560d2f"
-					(reference "C27")
+					(reference "C26")
 					(unit 1)
 				)
@@
 		(on_board yes)
 		(dnp no)
-		(property "Reference" "R62"
+		(property "Reference" "R58"
 			(at 288.29 128.016 90)
 			(effects
@@
 			(project "Pico-ButtonBoard-v1"
 				(path "/644201a9-3a2f-4df3-9c93-2ae55394df4b/dd046a3a-8e17-4277-b6b1-7e4df1560d2f"
-					(reference "R62")
+					(reference "R58")
 					(unit 1)
 				)
@@
 		(on_board yes)
 		(dnp no)
-		(property "Reference" "C24"
+		(property "Reference" "C22"
 			(at 81.28 143.7639 0)
 			(effects
@@
 			(project "Pico-ButtonBoard-v1"
 				(path "/644201a9-3a2f-4df3-9c93-2ae55394df4b/dd046a3a-8e17-4277-b6b1-7e4df1560d2f"
-					(reference "C24")
+					(reference "C22")
 					(unit 1)
 				)
@@
 		(on_board yes)
 		(dnp no)
-		(property "Reference" "R22"
+		(property "Reference" "R19"
 			(at 231.14 124.206 90)
 			(effects
@@
 			(project "Pico-ButtonBoard-v1"
 				(path "/644201a9-3a2f-4df3-9c93-2ae55394df4b/dd046a3a-8e17-4277-b6b1-7e4df1560d2f"
-					(reference "R22")
+					(reference "R19")
 					(unit 1)
 				)
@@
 		(on_board yes)
 		(dnp no)
-		(property "Reference" "R57"
+		(property "Reference" "R53"
 			(at 104.394 115.57 90)
 			(effects
@@
 			(project "Pico-ButtonBoard-v1"
 				(path "/644201a9-3a2f-4df3-9c93-2ae55394df4b/dd046a3a-8e17-4277-b6b1-7e4df1560d2f"
-					(reference "R57")
+					(reference "R53")
 					(unit 1)
 				)
@@
 		(on_board yes)
 		(dnp no)
-		(property "Reference" "R56"
+		(property "Reference" "R52"
 			(at 139.954 157.48 90)
 			(effects
@@
 			(project "Pico-ButtonBoard-v1"
 				(path "/644201a9-3a2f-4df3-9c93-2ae55394df4b/dd046a3a-8e17-4277-b6b1-7e4df1560d2f"
-					(reference "R56")
+					(reference "R52")
 					(unit 1)
 				)
@@
 		(on_board yes)
 		(dnp no)
-		(property "Reference" "R21"
+		(property "Reference" "R18"
 			(at 270.764 143.51 90)
 			(effects
@@
 			(project "Pico-ButtonBoard-v1"
 				(path "/644201a9-3a2f-4df3-9c93-2ae55394df4b/dd046a3a-8e17-4277-b6b1-7e4df1560d2f"
-					(reference "R21")
+					(reference "R18")
 					(unit 1)
 				)
@@
 		(on_board yes)
 		(dnp no)
-		(property "Reference" "C29"
+		(property "Reference" "C28"
 			(at 268.986 119.38 0)
 			(effects
@@
 			(project "Pico-ButtonBoard-v1"
 				(path "/644201a9-3a2f-4df3-9c93-2ae55394df4b/dd046a3a-8e17-4277-b6b1-7e4df1560d2f"
-					(reference "C29")
+					(reference "C28")
 					(unit 1)
 				)
@@
 		(on_board yes)
 		(dnp no)
-		(property "Reference" "R26"
+		(property "Reference" "R23"
 			(at 139.954 133.35 90)
 			(effects
@@
 			(project "Pico-ButtonBoard-v1"
 				(path "/644201a9-3a2f-4df3-9c93-2ae55394df4b/dd046a3a-8e17-4277-b6b1-7e4df1560d2f"
-					(reference "R26")
+					(reference "R23")
 					(unit 1)
 				)
@@
 		(on_board yes)
 		(dnp no)
-		(property "Reference" "R27"
+		(property "Reference" "R24"
 			(at 104.394 157.48 90)
 			(effects
@@
 			(project "Pico-ButtonBoard-v1"
 				(path "/644201a9-3a2f-4df3-9c93-2ae55394df4b/dd046a3a-8e17-4277-b6b1-7e4df1560d2f"
-					(reference "R27")
+					(reference "R24")
 					(unit 1)
 				)
@@
 		(on_board yes)
 		(dnp no)
-		(property "Reference" "R23"
+		(property "Reference" "R20"
 			(at 239.014 143.51 90)
 			(effects
@@
 			(project "Pico-ButtonBoard-v1"
 				(path "/644201a9-3a2f-4df3-9c93-2ae55394df4b/dd046a3a-8e17-4277-b6b1-7e4df1560d2f"
-					(reference "R23")
+					(reference "R20")
 					(unit 1)
 				)
