File: circuit-boards/mag-encoder/mag-encoder.kicad_sch (KiCad schematic)
At the start: 25 parts, among them J1 CONFIG, J2 0015912055, U1 AP2120N-3.3TRG1, U2 SN74LVC7032ABQAR, U3 MA732GQ

Commit message: Update silk to new part number
Signed-off-by: Scott Berman <sgberman1@gmail.com>
Other:
- title: Mag Encoder (WCP-1971) -> WCP Mag Encoder (WCP-2435)
Changed lines of the file:
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@@
 	(paper "B")
 	(title_block
-		(title "Mag Encoder (WCP-1971)")
+		(title "WCP Mag Encoder (WCP-2435)")
 		(date "2025-09-20")
 		(rev "1")

Commit message: Add open source license to mag encoder.
Signed-off-by: Scott Berman <sgberman1@gmail.com>
Parts:
- C1, C2, C3, C4, C5: footprint Capacitor_SMD:C_0603_1608Metric -> mag-encoder:C_0603_1608Metric
- D1, D2, D3, D4: footprint LED_SMD:LED_0603_1608Metric -> mag-encoder:LED_0603_1608Metric
- D5: footprint Diode_SMD:D_SOD-123 -> mag-encoder:D_SOD-123
- J1: footprint Connector_PinHeader_2.54mm:PinHeader_1x06_P2.54mm_Vertical -> mag-encoder:PinHeader_1x06_P2.54mm_Vertical
- R1, R2, R3, R4, R5, R6, R7, R8: footprint Resistor_SMD:R_0603_1608Metric -> mag-encoder:R_0603_1608Metric
- U1: footprint Package_TO_SOT_SMD:SOT-23 -> mag-encoder:SOT-23
Other:
- company: (none) -> Space Cookies FRC Team 1868
