File: circuit-boards/NX-J401-usb-m2-key-e-V1/NX-J401-usb-m2-key-e-V1.kicad_sch (KiCad schematic)
At the start: 3 parts, among them J1 USB1, J2 Bus_M.2_Socket_E

Commit message: Prepare USB-m2 for manufacture
Signed-off-by: Scott Berman <sgberman1@gmail.com>
Parts:
- J1: footprint usb-m2-key-e-adapter:Molex-PicoLatch-5040500491 -> nx-j401-usb-m2-key-e:Molex-PicoLatch-5040500491; symbol Connector_Generic:Conn_01x04 -> NX-J401-usb-m2-key-e:Conn_01x04
- J2: footprint Connector_PCBEdge:M.2_2230-xx-E -> nx-j401-usb-m2-key-e:M.2_2230-xx-E; symbol Connector:Bus_M.2_Socket_E -> NX-J401-usb-m2-key-e:Bus_M.2_Socket_E; now left out of the parts list
- LOGO1: footprint usb-m2-key-e-adapter:SPACE_COOKIES_LOGO_7mm -> nx-j401-usb-m2-key-e:SPACE_COOKIES_LOGO_7mm; symbol Graphic:SYM_Arrow_Large -> NX-J401-usb-m2-key-e:SYM_Arrow_Large
Changed lines of the file:
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@@
 	)
 	(symbol
-		(lib_id "Graphic:SYM_Arrow_Large")
+		(lib_id "NX-J401-usb-m2-key-e:SYM_Arrow_Large")
 		(at 71.4685 200.2297 0)
 		(unit 1)
@@
 			)
 		)
-		(property "Footprint" "usb-m2-key-e-adapter:SPACE_COOKIES_LOGO_7mm"
+		(property "Footprint" "nx-j401-usb-m2-key-e:SPACE_COOKIES_LOGO_7mm"
 			(at 71.4685 200.2297 0)
 			(hide yes)
@@
 	)
 	(symbol
-		(lib_id "Connector:Bus_M.2_Socket_E")
+		(lib_id "NX-J401-usb-m2-key-e:Bus_M.2_Socket_E")
 		(at 236.22 134.62 0)
 		(unit 1)
 		(body_style 1)
 		(exclude_from_sim no)
-		(in_bom yes)
+		(in_bom no)
 		(on_board yes)
 		(in_pos_files yes)
@@
 			)
 		)
-		(property "Footprint" "Connector_PCBEdge:M.2_2230-xx-E"
+		(property "Footprint" "nx-j401-usb-m2-key-e:M.2_2230-xx-E"
 			(at 236.22 107.95 0)
 			(hide yes)
@@
 	)
 	(symbol
-		(lib_id "Connector_Generic:Conn_01x04")
+		(lib_id "NX-J401-usb-m2-key-e:Conn_01x04")
 		(at 162.56 129.54 180)
 		(unit 1)
@@
 			)
 		)
-		(property "Footprint" "usb-m2-key-e-adapter:Molex-PicoLatch-5040500491"
+		(property "Footprint" "nx-j401-usb-m2-key-e:Molex-PicoLatch-5040500491"
 			(at 162.56 129.54 0)
 			(hide yes)
