File: circuit-boards/NX-J401-Adapter-v6/usb-serial.kicad_sch (KiCad schematic)
At the start: 14 parts, among them J14 USB_C_Receptacle_USB2.0_14P, U8 FT232RNL, U9 ISO6721BDR

Commit message: Improved placement.  Pre-routing
Signed-off-by: Scott Berman <sgberman1@gmail.com>
Parts:
- removed C60: 10uF-50V-10%-X7R-1210, Capacitor_SMD:C_1210_3225Metric, symbol Device:C_US
- added C49: 22uF-10%-16V-0805, Capacitor_SMD:C_0805_2012Metric, symbol Device:C_US
Connections:
- net GND_USB: now also C49.2
- net at C61.1, L2.2, U8.20 (VCC)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: now also C49.1
Changed lines of the file:
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@@
-	)
-	(symbol
-		(lib_id "Device:C_US")
-		(at 154.94 133.35 0)
-		(unit 1)
-		(body_style 1)
-		(exclude_from_sim no)
-		(in_bom yes)
-		(on_board yes)
-		(in_pos_files yes)
-		(dnp no)
-		(property "Reference" "C60"
-			(at 156.718 131.318 90)
-			(show_name no)
-			(do_not_autoplace no)
-			(effects
-				(font
-					(size 1.27 1.27)
-				)
-				(justify left)
-			)
-		)
-		(property "Value" "10uF-50V-10%-X7R-1210"
-			(at 151.384 133.604 90)
-			(show_name no)
-			(do_not_autoplace no)
-			(effects
-				(font
-					(size 1.27 1.27)
-				)
-			)
-		)
-		(property "Footprint" "Capacitor_SMD:C_1210_3225Metric"
-			(at 154.94 133.35 0)
-			(hide yes)
-			(show_name no)
-			(do_not_autoplace no)
-			(effects
-				(font
-					(size 1.27 1.27)
-				)
-			)
-		)
-		(property "Datasheet" "Components/Murata-GRM32ER71H106KA12-01.pdf"
-			(at 154.94 133.35 0)
-			(hide yes)
-			(show_name no)
-			(do_not_autoplace no)
-			(effects
-				(font
-					(size 1.27 1.27)
-				)
-			)
-		)
-		(property "Description" "capacitor, US symbol"
-			(at 154.94 133.35 0)
-			(hide yes)
-			(show_name no)
-			(do_not_autoplace no)
-			(effects
-				(font
-					(size 1.27 1.27)
-				)
-			)
-		)
-		(property "MFG" "Murata Eelectronics"
-			(at 154.94 133.35 0)
-			(hide yes)
-			(show_name no)
-			(do_not_autoplace no)
-			(effects
-				(font
-					(size 1.27 1.27)
-				)
-			)
-		)
-		(property "MFG P/N" " GRM32ER71H106KA12L"
-			(at 154.94 133.35 0)
-			(hide yes)
-			(show_name no)
-			(do_not_autoplace no)
-			(effects
-				(font
-					(size 1.27 1.27)
-				)
-			)
-		)
-		(property "JLCPCB P/N" "C77102"
-			(at 154.94 133.35 0)
-			(hide yes)
-			(show_name no)
-			(do_not_autoplace no)
-			(effects
-				(font
-					(size 1.27 1.27)
-				)
-			)
-		)
-		(pin "1"
-		)
-		(pin "2"
-		)
-		(instances
-			(project "NX-J401-Adapter-v6"
-				(path "/3c9fa76f-2b37-4666-8575-58caa65def04/7f338915-7b6e-40c1-9733-742b14680646"
-					(reference "C60")
-					(unit 1)
-				)
-			)
-		)
 	)
 	(symbol
@@
 					(unit 1)
 				)
+			)
+		)
+	)
+	(symbol
+		(lib_id "Device:C_US")
+		(at 154.94 133.35 0)
+		(unit 1)
+		(body_style 1)
+		(exclude_from_sim no)
+		(in_bom yes)
+		(on_board yes)
+		(in_pos_files yes)
+		(dnp no)
+		(property "Reference" "C49"
+			(at 155.956 130.556 0)
+			(show_name no)
+			(do_not_autoplace no)
+			(effects
+				(font
+					(size 1.27 1.27)
+				)
+				(justify left)
+			)
+		)
+		(property "Value" "22uF-10%-16V-0805"
+			(at 151.384 133.604 90)
+			(show_name no)
+			(do_not_autoplace no)
+			(effects
+				(font
+					(size 1.27 1.27)
+				)
+			)
+		)
+		(property "Footprint" "Capacitor_SMD:C_0805_2012Metric"
+			(at 154.94 133.35 0)
+			(hide yes)
+			(show_name no)
+			(do_not_autoplace no)
+			(effects
+				(font
+					(size 1.27 1.27)
+				)
+			)
+		)
+		(property "Datasheet" ""
+			(at 154.94 133.35 0)
+			(hide yes)
+			(show_name no)
+			(do_not_autoplace no)
+			(effects
+				(font
+					(size 1.27 1.27)
+				)
+			)
+		)
+		(property "Description" "16V 22uF X5R ±10% 0805 Multilayer Ceramic Capacitors MLCC - SMD/SMT ROHS"
+			(at 154.94 133.35 0)
+			(hide yes)
+			(show_name no)
+			(do_not_autoplace no)
+			(effects
+				(font
+					(size 1.27 1.27)
+				)
+			)
+		)
+		(property "MFG" "Samsung Electro-Mechanics"
+			(at 154.94 133.35 0)
+			(hide yes)
+			(show_name no)
+			(do_not_autoplace no)
+			(effects
+				(font
+					(size 1.27 1.27)
+				)
+			)
+		)
+		(property "MFG P/N" "CL21A226KOQNNNE"
+			(at 154.94 133.35 0)
+			(hide yes)
+			(show_name no)
+			(do_not_autoplace no)
+			(effects
+				(font
+					(size 1.27 1.27)
+				)
+			)
+		)
+		(property "JLCPCB P/N" "C296720"
+			(at 154.94 133.35 0)
+			(hide yes)
+			(show_name no)
+			(do_not_autoplace no)
+			(effects
+				(font
+					(size 1.27 1.27)
+				)
+			)
+		)
+		(pin "1"
+		)
+		(pin "2"
+		)
+		(instances
+			(project "NX-J401-Adapter-v6"
+				(path "/3c9fa76f-2b37-4666-8575-58caa65def04/7f338915-7b6e-40c1-9733-742b14680646"
+					(reference "C49")
+					(unit 1)
+				)

Commit message: Initial complete routing
Signed-off-by: Scott Berman <sgberman1@gmail.com>
Parts:
- C38: renamed from C63; KiLib_Generator (none) -> SMD_2terminal_chip_molded
- C39: renamed from C64; KiLib_Generator (none) -> SMD_2terminal_chip_molded
- C45: renamed from C49; KiLib_Generator (none) -> SMD_2terminal_chip_molded
- C46: renamed from C57; KiLib_Generator (none) -> SMD_2terminal_chip_molded
- C53: renamed from C61; KiLib_Generator (none) -> SMD_2terminal_chip_molded
- C54: renamed from C62; KiLib_Generator (none) -> SMD_2terminal_chip_molded
- C55: renamed from C59; KiLib_Generator (none) -> SMD_2terminal_chip_molded
- C56: renamed from C58; KiLib_Generator (none) -> SMD_2terminal_chip_molded
- L3: renamed from L2; KiLib_Generator (none) -> SMD_2terminal_chip_molded
- R24: renamed from R30; KiLib_Generator (none) -> SMD_2terminal_chip_molded
- R25: renamed from R31; KiLib_Generator (none) -> SMD_2terminal_chip_molded
- U7: renamed from U9; KiLib_Generator (none) -> package/gullwing
- U8: KiLib_Generator (none) -> package/gullwing
- renumbered J14 to J11
Changed lines of the file:
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@@
 		(in_pos_files yes)
 		(dnp no)
-		(property "Reference" "R31"
+		(property "Reference" "R25"
 			(at 114.808 158.75 90)
 			(show_name no)
@@
 		(property "JLCPCB P/N" "C105580"
 			(at 118.11 160.02 90)
+			(hide yes)
+			(show_name no)
+			(do_not_autoplace no)
+			(effects
+				(font
+					(size 1.27 1.27)
+				)
+			)
+		)
+		(property "KiLib_Generator" "SMD_2terminal_chip_molded"
+			(at 118.11 160.02 0)
 			(hide yes)
 			(show_name no)
@@
 			(project "NX-J401-Adapter-v6"
 				(path "/3c9fa76f-2b37-4666-8575-58caa65def04/7f338915-7b6e-40c1-9733-742b14680646"
-					(reference "R31")
+					(reference "R25")
 					(unit 1)
 				)
@@
 		(in_pos_files yes)
 		(dnp no)
-		(property "Reference" "C64"
+		(property "Reference" "C39"
 			(at 325.12 108.2039 0)
 			(show_name no)
@@
 		)
 		(property "JLCPCB P/N" "C14663"
+			(at 321.31 109.22 0)
+			(hide yes)
+			(show_name no)
+			(do_not_autoplace no)
+			(effects
+				(font
+					(size 1.27 1.27)
+				)
+			)
+		)
+		(property "KiLib_Generator" "SMD_2terminal_chip_molded"
 			(at 321.31 109.22 0)
 			(hide yes)
@@
 			(project "NX-J401-Adapter-v6"
 				(path "/3c9fa76f-2b37-4666-8575-58caa65def04/7f338915-7b6e-40c1-9733-742b14680646"
-					(reference "C64")
+					(reference "C39")
 					(unit 1)
 				)
@@
 		(in_pos_files yes)
 		(dnp no)
-		(property "Reference" "C61"
+		(property "Reference" "C53"
 			(at 204.47 128.5239 0)
 			(show_name no)
@@
 		)
 		(property "JLCPCB P/N" "C14663"
+			(at 208.28 129.54 0)
+			(hide yes)
+			(show_name no)
+			(do_not_autoplace no)
+			(effects
+				(font
+					(size 1.27 1.27)
+				)
+			)
+		)
+		(property "KiLib_Generator" "SMD_2terminal_chip_molded"
 			(at 208.28 129.54 0)
 			(hide yes)
@@
 			(project "NX-J401-Adapter-v6"
 				(path "/3c9fa76f-2b37-4666-8575-58caa65def04/7f338915-7b6e-40c1-9733-742b14680646"
-					(reference "C61")
+					(reference "C53")
 					(unit 1)
 				)
@@
 		(in_pos_files yes)
 		(dnp no)
-		(property "Reference" "J14"
+		(property "Reference" "J11"
 			(at 85.09 139.7 0)
 			(show_name no)
@@
 			(project "NX-J401-Adapter-v6"
 				(path "/3c9fa76f-2b37-4666-8575-58caa65def04/7f338915-7b6e-40c1-9733-742b14680646"
-					(reference "J14")
+					(reference "J11")
 					(unit 1)
 				)
@@
 		(in_pos_files yes)
 		(dnp no)
-		(property "Reference" "C57"
+		(property "Reference" "C46"
 			(at 118.618 131.572 90)
 			(show_name no)
@@
 		)
 		(property "JLCPCB P/N" "C107076"
+			(at 116.84 133.35 0)
+			(hide yes)
+			(show_name no)
+			(do_not_autoplace no)
+			(effects
+				(font
+					(size 1.27 1.27)
+				)
+			)
+		)
+		(property "KiLib_Generator" "SMD_2terminal_chip_molded"
 			(at 116.84 133.35 0)
 			(hide yes)
@@
 			(project "NX-J401-Adapter-v6"
 				(path "/3c9fa76f-2b37-4666-8575-58caa65def04/7f338915-7b6e-40c1-9733-742b14680646"
-					(reference "C57")
+					(reference "C46")
 					(unit 1)
 				)
@@
 		(in_pos_files yes)
 		(dnp no)
-		(property "Reference" "C59"
+		(property "Reference" "C55"
 			(at 140.716 189.23 0)
 			(show_name no)
@@
 		)
 		(property "JLCPCB P/N" "C2168903"
+			(at 139.7 191.77 0)
+			(hide yes)
+			(show_name no)
+			(do_not_autoplace no)
+			(effects
+				(font
+					(size 1.27 1.27)
+				)
+			)
+		)
+		(property "KiLib_Generator" "SMD_2terminal_chip_molded"
 			(at 139.7 191.77 0)
 			(hide yes)
@@
 			(project "NX-J401-Adapter-v6"
 				(path "/3c9fa76f-2b37-4666-8575-58caa65def04/7f338915-7b6e-40c1-9733-742b14680646"
-					(reference "C59")
+					(reference "C55")
 					(unit 1)
 				)
@@
 		(in_pos_files yes)
 		(dnp no)
-		(property "Reference" "C49"
+		(property "Reference" "C45"
 			(at 155.956 130.556 0)
 			(show_name no)
@@
 		)
 		(property "JLCPCB P/N" "C296720"
+			(at 154.94 133.35 0)
+			(hide yes)
+			(show_name no)
+			(do_not_autoplace no)
+			(effects
+				(font
+					(size 1.27 1.27)
+				)
+			)
+		)
+		(property "KiLib_Generator" "SMD_2terminal_chip_molded"
 			(at 154.94 133.35 0)
 			(hide yes)
@@
 			(project "NX-J401-Adapter-v6"
 				(path "/3c9fa76f-2b37-4666-8575-58caa65def04/7f338915-7b6e-40c1-9733-742b14680646"
-					(reference "C49")
+					(reference "C45")
 					(unit 1)
 				)
@@
 		(in_pos_files yes)
 		(dnp no)
-		(property "Reference" "C63"
+		(property "Reference" "C38"
 			(at 275.59 95.5039 0)
 			(show_name no)
@@
 		)
 		(property "JLCPCB P/N" "C14663"
+			(at 279.4 96.52 0)
+			(hide yes)
+			(show_name no)
+			(do_not_autoplace no)
+			(effects
+				(font
+					(size 1.27 1.27)
+				)
+			)
+		)
+		(property "KiLib_Generator" "SMD_2terminal_chip_molded"
 			(at 279.4 96.52 0)
 			(hide yes)
@@
 			(project "NX-J401-Adapter-v6"
 				(path "/3c9fa76f-2b37-4666-8575-58caa65def04/7f338915-7b6e-40c1-9733-742b14680646"
-					(reference "C63")
+					(reference "C38")
 					(unit 1)
 				)
@@
 		(in_pos_files yes)
 		(dnp no)
-		(property "Reference" "C62"
+		(property "Reference" "C54"
 			(at 205.74 190.7539 0)
 			(show_name no)
@@
 		)
 		(property "JLCPCB P/N" "C14663"
+			(at 209.55 191.77 0)
+			(hide yes)
+			(show_name no)
+			(do_not_autoplace no)
+			(effects
+				(font
+					(size 1.27 1.27)
+				)
+			)
+		)
+		(property "KiLib_Generator" "SMD_2terminal_chip_molded"
 			(at 209.55 191.77 0)
 			(hide yes)
@@
 			(project "NX-J401-Adapter-v6"
 				(path "/3c9fa76f-2b37-4666-8575-58caa65def04/7f338915-7b6e-40c1-9733-742b14680646"
-					(reference "C62")
+					(reference "C54")
 					(unit 1)
 				)
@@
 		(in_pos_files yes)
 		(dnp no)
-		(property "Reference" "C58"
+		(property "Reference" "C56"
 			(at 130.556 189.23 0)
 			(show_name no)
@@
 		)
 		(property "JLCPCB P/N" "C2168903"
+			(at 129.54 191.77 0)
+			(hide yes)
+			(show_name no)
+			(do_not_autoplace no)
+			(effects
+				(font
+					(size 1.27 1.27)
+				)
+			)
+		)
+		(property "KiLib_Generator" "SMD_2terminal_chip_molded"
 			(at 129.54 191.77 0)
 			(hide yes)
@@
 			(project "NX-J401-Adapter-v6"
 				(path "/3c9fa76f-2b37-4666-8575-58caa65def04/7f338915-7b6e-40c1-9733-742b14680646"
-					(reference "C58")
+					(reference "C56")
 					(unit 1)
 				)
@@
 		(in_pos_files yes)
 		(dnp no)
-		(property "Reference" "R30"
+		(property "Reference" "R24"
 			(at 114.808 152.4 90)
 			(show_name no)
@@
 		(property "JLCPCB P/N" "C105580"
 			(at 118.11 153.67 90)
+			(hide yes)
+			(show_name no)
+			(do_not_autoplace no)
+			(effects
+				(font
+					(size 1.27 1.27)
+				)
+			)
+		)
+		(property "KiLib_Generator" "SMD_2terminal_chip_molded"
+			(at 118.11 153.67 0)
 			(hide yes)
 			(show_name no)
@@
 			(project "NX-J401-Adapter-v6"
 				(path "/3c9fa76f-2b37-4666-8575-58caa65def04/7f338915-7b6e-40c1-9733-742b14680646"
-					(reference "R30")
+					(reference "R24")
 					(unit 1)
 				)
@@
 			)
 		)
+		(property "KiLib_Generator" "package/gullwing"
+			(at 237.49 166.37 0)
+			(hide yes)
+			(show_name no)
+			(do_not_autoplace no)
+			(effects
+				(font
+					(size 1.27 1.27)
+				)
+			)
+		)
 		(pin "16"
 		)
@@
 		(dnp no)
 		(fields_autoplaced yes)
-		(property "Reference" "U9"
+		(property "Reference" "U7"
 			(at 293.37 118.11 0)
 			(show_name no)
@@
 		)
 		(property "JLCPCB P/N" "C5216430"
+			(at 293.37 123.19 0)
+			(hide yes)
+			(show_name no)
+			(do_not_autoplace no)
+			(effects
+				(font
+					(size 1.27 1.27)
+				)
+			)
+		)
+		(property "KiLib_Generator" "package/gullwing"
 			(at 293.37 123.19 0)
 			(hide yes)
@@
 			(project "NX-J401-Adapter-v6"
 				(path "/3c9fa76f-2b37-4666-8575-58caa65def04/7f338915-7b6e-40c1-9733-742b14680646"
-					(reference "U9")
+					(reference "U7")
 					(unit 1)
 				)
@@
 		(in_pos_files yes)
 		(dnp no)
-		(property "Reference" "L2"
+		(property "Reference" "L3"
 			(at 134.62 116.332 90)
 			(show_name no)
@@
 		(property "JLCPCB P/N" "C2441364"
 			(at 134.62 119.38 90)
+			(hide yes)
+			(show_name no)
+			(do_not_autoplace no)
+			(effects
+				(font
+					(size 1.27 1.27)
+				)
+			)
+		)
+		(property "KiLib_Generator" "SMD_2terminal_chip_molded"
+			(at 134.62 119.38 0)
 			(hide yes)
 			(show_name no)
@@
 			(project "NX-J401-Adapter-v6"
 				(path "/3c9fa76f-2b37-4666-8575-58caa65def04/7f338915-7b6e-40c1-9733-742b14680646"
-					(reference "L2")
-					(unit 1)
-				)
+					(reference "L3")
+					(unit 1)
+				)

Commit message: minor fixes
Signed-off-by: Scott Berman <sgberman1@gmail.com>
Other:
- company: (none) -> SPACE COOKIES FRC TEAM 1868
Changed lines of the file:
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@@
 	(title_block
 		(title "NX J401 Adapter")
-		(date "2025-11-24")
-		(rev "5")
+		(date "2026-05-25")
+		(rev "6")
+		(company "SPACE COOKIES FRC TEAM 1868")
 	)
 	(text "https://hackaday.com/2023/08/07/all-about-usb-c-example-circuits/"

Commit message: Updates
Signed-off-by: Scott Berman <sgberman1@gmail.com>
Parts:
- C38, C39, C46, C53, C54, C55, C56: footprint Capacitor_SMD:C_0603_1608Metric -> NX-J401-Adapter:C_0603_1608Metric; symbol Device:C_US -> NX-J401-Adapter:C_US
- C45: footprint Capacitor_SMD:C_0805_2012Metric -> NX-J401-Adapter:C_0805_2012Metric; symbol Device:C_US -> NX-J401-Adapter:C_US
- L3: footprint Inductor_SMD:L_0805_2012Metric -> NX-J401-Adapter:L_0805_2012Metric; symbol Device:L_Iron -> NX-J401-Adapter:L_Iron
- R24, R25: footprint Resistor_SMD:R_0603_1608Metric -> NX-J401-Adapter:R_0603_1608Metric; symbol Device:R_US -> NX-J401-Adapter:R_US
- U7: footprint Package_SO:SOIC-8_3.9x4.9mm_P1.27mm -> NX-J401-Adapter:SOIC-8_3.9x4.9mm_P1.27mm
- U8: footprint Package_SO:SSOP-28_5.3x10.2mm_P0.65mm -> NX-J401-Adapter:SSOP-28_5.3x10.2mm_P0.65mm
Changed lines of the file:
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@@
 	(title_block
 		(title "NX J401 Adapter")
-		(date "2026-05-25")
+		(date "2026-06-02")
 		(rev "6")
 		(company "SPACE COOKIES FRC TEAM 1868")
@@
 	)
 	(symbol
-		(lib_id "Device:R_US")
+		(lib_id "NX-J401-Adapter:R_US")
 		(at 118.11 160.02 90)
 		(mirror x)
@@
 			)
 		)
-		(property "Footprint" "Resistor_SMD:R_0603_1608Metric"
+		(property "Footprint" "NX-J401-Adapter:R_0603_1608Metric"
 			(at 118.364 161.036 90)
 			(hide yes)
@@
 	)
 	(symbol
-		(lib_id "Device:C_US")
+		(lib_id "NX-J401-Adapter:C_US")
 		(at 321.31 109.22 0)
 		(unit 1)
@@
 			)
 		)
-		(property "Footprint" "Capacitor_SMD:C_0603_1608Metric"
+		(property "Footprint" "NX-J401-Adapter:C_0603_1608Metric"
 			(at 321.31 109.22 0)
 			(hide yes)
@@
 	)
 	(symbol
-		(lib_id "Device:C_US")
+		(lib_id "NX-J401-Adapter:C_US")
 		(at 208.28 129.54 0)
 		(mirror y)
@@
 			)
 		)
-		(property "Footprint" "Capacitor_SMD:C_0603_1608Metric"
+		(property "Footprint" "NX-J401-Adapter:C_0603_1608Metric"
 			(at 208.28 129.54 0)
 			(hide yes)
@@
 	)
 	(symbol
-		(lib_id "Device:C_US")
+		(lib_id "NX-J401-Adapter:C_US")
 		(at 116.84 133.35 0)
 		(mirror y)
@@
 			)
 		)
-		(property "Footprint" "Capacitor_SMD:C_0603_1608Metric"
+		(property "Footprint" "NX-J401-Adapter:C_0603_1608Metric"
 			(at 116.84 133.35 0)
 			(hide yes)
@@
 	)
 	(symbol
-		(lib_id "Device:C_US")
+		(lib_id "NX-J401-Adapter:C_US")
 		(at 139.7 191.77 0)
 		(mirror y)
@@
 			)
 		)
-		(property "Footprint" "Capacitor_SMD:C_0603_1608Metric"
+		(property "Footprint" "NX-J401-Adapter:C_0603_1608Metric"
 			(at 139.7 191.77 0)
 			(hide yes)
@@
 	)
 	(symbol
-		(lib_id "Device:C_US")
+		(lib_id "NX-J401-Adapter:C_US")
 		(at 154.94 133.35 0)
 		(unit 1)
@@
 			)
 		)
-		(property "Footprint" "Capacitor_SMD:C_0805_2012Metric"
+		(property "Footprint" "NX-J401-Adapter:C_0805_2012Metric"
 			(at 154.94 133.35 0)
 			(hide yes)
@@
 	)
 	(symbol
-		(lib_id "Device:C_US")
+		(lib_id "NX-J401-Adapter:C_US")
 		(at 279.4 96.52 0)
 		(mirror y)
@@
 			)
 		)
-		(property "Footprint" "Capacitor_SMD:C_0603_1608Metric"
+		(property "Footprint" "NX-J401-Adapter:C_0603_1608Metric"
 			(at 279.4 96.52 0)
 			(hide yes)
@@
 	)
 	(symbol
-		(lib_id "Device:C_US")
+		(lib_id "NX-J401-Adapter:C_US")
 		(at 209.55 191.77 0)
 		(mirror y)
@@
 			)
 		)
-		(property "Footprint" "Capacitor_SMD:C_0603_1608Metric"
+		(property "Footprint" "NX-J401-Adapter:C_0603_1608Metric"
 			(at 209.55 191.77 0)
 			(hide yes)
@@
 	)
 	(symbol
-		(lib_id "Device:C_US")
+		(lib_id "NX-J401-Adapter:C_US")
 		(at 129.54 191.77 0)
 		(mirror y)
@@
 			)
 		)
-		(property "Footprint" "Capacitor_SMD:C_0603_1608Metric"
+		(property "Footprint" "NX-J401-Adapter:C_0603_1608Metric"
 			(at 129.54 191.77 0)
 			(hide yes)
@@
 	)
 	(symbol
-		(lib_id "Device:R_US")
+		(lib_id "NX-J401-Adapter:R_US")
 		(at 118.11 153.67 90)
 		(mirror x)
@@
 			)
 		)
-		(property "Footprint" "Resistor_SMD:R_0603_1608Metric"
+		(property "Footprint" "NX-J401-Adapter:R_0603_1608Metric"
 			(at 118.364 154.686 90)
 			(hide yes)
@@
 			)
 		)
-		(property "Footprint" "Package_SO:SSOP-28_5.3x10.2mm_P0.65mm"
+		(property "Footprint" "NX-J401-Adapter:SSOP-28_5.3x10.2mm_P0.65mm"
 			(at 259.842 189.23 0)
 			(hide yes)
@@
 			)
 		)
-		(property "Footprint" "Package_SO:SOIC-8_3.9x4.9mm_P1.27mm"
+		(property "Footprint" "NX-J401-Adapter:SOIC-8_3.9x4.9mm_P1.27mm"
 			(at 293.37 123.19 0)
 			(hide yes)
@@
 	)
 	(symbol
-		(lib_id "Device:L_Iron")
+		(lib_id "NX-J401-Adapter:L_Iron")
 		(at 134.62 119.38 90)
 		(unit 1)
@@
 			)
 		)
-		(property "Footprint" "Inductor_SMD:L_0805_2012Metric"
+		(property "Footprint" "NX-J401-Adapter:L_0805_2012Metric"
 			(at 134.62 119.38 0)
 			(hide yes)
