File: circuit-boards/NX-J401-Adapter-v6/NX-J401-Adapter-v6.kicad_sch (KiCad schematic)
At the start: 28 parts, among them J1 Terminal, J10 POWER, J2 Terminal, J5 NX CONTROL & UART, J6 USB1, J7 15V, J9 CAN1, Q2 CSD19534Q5A, Q9 CSD19534Q5A, SW1 RESET, SW2 RECOVERY, U2 LM74700QDBVRQ1, U4 LM74700QDBVRQ1

Commit message: Moved the Vout connector to increase clearance
Signed-off-by: Scott Berman <sgberman1@gmail.com>
Parts:
- removed J5: NX CONTROL & UART, Connector_PinHeader_2.54mm:PinHeader_1x18_P2.54mm_Horizontal, symbol Connector:Conn_01x18_Pin
- added H7, H8, H9: MountingHole, MountingHole:MountingHole_2.5mm, symbol Mechanical:MountingHole
- added J3: NX CONTROL & UART, Connector_PinHeader_2.54mm:PinHeader_1x15_P2.54mm_Horizontal, symbol Connector:Conn_01x15_Pin
- D6, D7: DIST Digikey -> (none); DIST P/N 1080-1419-1-ND -> (none); JLCPCB P/N (none) -> C5123493; MFG Everlight -> BrtLed(Bright LED Elec); MFG P/N QTLP650D4TR/QT15-21SYGD/S530-E2/TR8 -> BL-HGK33-TRB
- J1, J2: JLCPCB P/N (none) -> XXXXXX
- renumbered H3 to H5, H4 to H6, J6 to J4, J7 to J5
Connections:
- net 3V3_BTN: now also J3.1 (Pin_1)
- net GND1: now also J3.10 (Pin_10), J3.12 (Pin_12)
- net NX_PC_LED+: now also J3.5 (Pin_5)
- net NX_PC_LED-: now also J3.4 (Pin_4)
- net UART2_RXD: now also J3.6 (Pin_6)
- net UART2_TXD: now also J3.7 (Pin_7)
- net ~{REC}: now also J3.13 (Pin_13)
- net ~{SYS_RESET}: now also J3.11 (Pin_11)

Commit message: minor fixes
Signed-off-by: Scott Berman <sgberman1@gmail.com>
Other:
- company: (none) -> SPACE COOKIES FRC TEAM 1868

Commit message: Add rails to M.2 adapter.  Minor fixes to NX J401 adapter
Signed-off-by: Scott Berman <sgberman1@gmail.com>
Parts:
- added LOGO1: SPACE COOKIES LOGO, NX-J401-Adapter:SPACE_COOKIES_LOGO_15mm, symbol Graphic:SYM_Arrow_Large
Changed lines of the file:
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@@
 		)
 	)
-	(text_box "Mating Connector:\nHousing: Molex 0436450200\nPrecrimped 24AWG wire 450mm: \n   Black: Molex 2147601225\n   Red:   Molex 2147602225"
+	(text_box "Mating Connector:\nHousing: Molex 0436450200\nPrecrimped 18AWG wire 450mm: \n   Black: Molex 2147601225\n   Red:   Molex 2147602225"
 		(exclude_from_sim no)
 		(at 16.51 48.26 0)
@@
 		)
 	)
-	(text_box "Mating Connector:\nHousing: Molex 0436450200\nPrecrimped 24AWG wire 450mm: \n   Black: Molex 2147601225\n   Red:   Molex 2147602225"
+	(text_box "Mating Connector:\nHousing: Molex 0436450200\nPrecrimped 18AWG wire 450mm: \n   Black: Molex 2147601225\n   Red:   Molex 2147602225"
 		(exclude_from_sim no)
 		(at 356.87 50.8 0)
@@
 					(unit 1)
 				)
+			)
+		)
+	)
+	(symbol
+		(lib_id "Graphic:SYM_Arrow_Large")
+		(at 74.93 237.49 0)
+		(unit 1)
+		(body_style 1)
+		(exclude_from_sim no)
+		(in_bom no)
+		(on_board yes)
+		(in_pos_files yes)
+		(dnp no)
+		(property "Reference" "LOGO1"
+			(at 74.93 235.204 0)
+			(hide yes)
+			(show_name no)
+			(do_not_autoplace no)
+			(effects
+				(font
+					(size 1.27 1.27)
+				)
+			)
+		)
+		(property "Value" "SPACE COOKIES LOGO"
+			(at 80.01 237.49 0)
+			(show_name no)
+			(do_not_autoplace no)
+			(effects
+				(font
+					(size 2.54 2.54)
+				)
+				(justify left)
+			)
+		)
+		(property "Footprint" "NX-J401-Adapter:SPACE_COOKIES_LOGO_15mm"
+			(at 74.93 237.49 0)
+			(hide yes)
+			(show_name no)
+			(do_not_autoplace no)
+			(effects
+				(font
+					(size 1.27 1.27)
+				)
+			)
+		)
+		(property "Datasheet" ""
+			(at 74.93 237.49 0)
+			(hide yes)
+			(show_name no)
+			(do_not_autoplace no)
+			(effects
+				(font
+					(size 1.27 1.27)
+				)
+			)
+		)
+		(property "Description" ""
+			(at 74.93 237.49 0)
+			(hide yes)
+			(show_name no)
+			(do_not_autoplace no)
+			(effects
+				(font
+					(size 1.27 1.27)
+				)
+			)
+		)
+		(instances
+			(project "NX-J401-Adapter-v6"
+				(path "/3c9fa76f-2b37-4666-8575-58caa65def04"
+					(reference "LOGO1")
+					(unit 1)
+				)

Commit message: Updates
Signed-off-by: Scott Berman <sgberman1@gmail.com>
Parts:
- C10, C40, C42, C5: footprint Capacitor_SMD:C_1210_3225Metric -> NX-J401-Adapter:C_1210_3225Metric; symbol Device:C_US -> NX-J401-Adapter:C_US
- C4, C41: footprint Capacitor_SMD:C_0603_1608Metric -> NX-J401-Adapter:C_0603_1608Metric; symbol Device:C_US -> NX-J401-Adapter:C_US
- D3: symbol Device:D_TVS -> NX-J401-Adapter:D_TVS
- D6, D7: footprint LED_SMD:LED_1206_3216Metric -> NX-J401-Adapter:LED_1206_3216Metric; symbol Device:LED -> NX-J401-Adapter:LED_1
- H1, H2, H5, H6, H7, H8, H9: footprint MountingHole:MountingHole_2.5mm -> NX-J401-Adapter:MountingHole_2.5mm; symbol Mechanical:MountingHole -> NX-J401-Adapter:MountingHole
- J10, J5, J9: symbol Connector_Generic:Conn_01x02 -> NX-J401-Adapter:Conn_01x02
- J3: footprint Connector_PinHeader_2.54mm:PinHeader_1x15_P2.54mm_Horizontal -> NX-J401-Adapter:PinHeader_1x15_P2.54mm_Horizontal; symbol Connector:Conn_01x15_Pin -> NX-J401-Adapter:Conn_01x15_Pin
- J4: symbol Connector_Generic:Conn_01x04 -> NX-J401-Adapter:Conn_01x04
- LOGO1: symbol Graphic:SYM_Arrow_Large -> NX-J401-Adapter:SYM_Arrow_Large
- Q2, Q9: symbol Transistor_FET:CSD19534Q5A -> NX-J401-Adapter:CSD19534Q5A
- R16: footprint Resistor_SMD:R_0603_1608Metric -> NX-J401-Adapter:R_0603_1608Metric; symbol Device:R_US -> NX-J401-Adapter:R_US
- SW1, SW2: symbol Switch:SW_Push -> NX-J401-Adapter:SW_Push
- U2, U4: footprint Package_TO_SOT_SMD:SOT-23-6 -> NX-J401-Adapter:SOT-23-6
Other:
- note added: "Power Supply Back Feed Protection"
- note added: "Reverse Polarity Protection"
Changed lines of the file:
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@@
 	(title_block
 		(title "NX J401 Adapter")
-		(date "2026-05-25")
+		(date "2026-06-02")
 		(rev "6")
 		(company "SPACE COOKIES FRC TEAM 1868")
@@
 		)
 	)
+	(text "Power Supply Back\nFeed Protection"
+		(exclude_from_sim no)
+		(at 282.194 35.306 0)
+		(effects
+			(font
+				(size 1.27 1.27)
+			)
+		)
+	)
 	(text "SLEEP/WAKE*"
 		(exclude_from_sim no)
@@
 		)
 	)
+	(text "Reverse Polarity Protection"
+		(exclude_from_sim no)
+		(at 143.764 34.544 0)
+		(effects
+			(font
+				(size 1.27 1.27)
+			)
+		)
+	)
 	(text "Auto Power On Disable"
 		(exclude_from_sim no)
@@
 	)
 	(symbol
-		(lib_id "Mechanical:MountingHole")
+		(lib_id "NX-J401-Adapter:MountingHole")
 		(at 295.91 182.88 0)
 		(unit 1)
@@
 			)
 		)
-		(property "Footprint" "MountingHole:MountingHole_2.5mm"
+		(property "Footprint" "NX-J401-Adapter:MountingHole_2.5mm"
 			(at 295.91 182.88 0)
 			(hide yes)
@@
 	)
 	(symbol
-		(lib_id "Device:C_US")
+		(lib_id "NX-J401-Adapter:C_US")
 		(at 161.29 63.5 0)
 		(unit 1)
@@
 			)
 		)
-		(property "Footprint" "Capacitor_SMD:C_1210_3225Metric"
+		(property "Footprint" "NX-J401-Adapter:C_1210_3225Metric"
 			(at 161.29 63.5 0)
 			(hide yes)
@@
 			)
 		)
-		(property "Footprint" "Package_TO_SOT_SMD:SOT-23-6"
+		(property "Footprint" "NX-J401-Adapter:SOT-23-6"
 			(at 133.985 74.93 0)
 			(hide yes)
@@
 	)
 	(symbol
-		(lib_id "Mechanical:MountingHole")
+		(lib_id "NX-J401-Adapter:MountingHole")
 		(at 326.39 187.96 0)
 		(unit 1)
@@
 			)
 		)
-		(property "Footprint" "MountingHole:MountingHole_2.5mm"
+		(property "Footprint" "NX-J401-Adapter:MountingHole_2.5mm"
 			(at 326.39 187.96 0)
 			(hide yes)
@@
 	(symbol
 		(lib_name "LED_1")
-		(lib_id "Device:LED")
+		(lib_id "NX-J401-Adapter:LED_1")
 		(at 168.91 71.12 90)
 		(unit 1)
@@
 			)
 		)
-		(property "Footprint" "LED_SMD:LED_1206_3216Metric"
+		(property "Footprint" "NX-J401-Adapter:LED_1206_3216Metric"
 			(at 168.91 71.12 0)
 			(hide yes)
@@
 	)
 	(symbol
-		(lib_id "Mechanical:MountingHole")
+		(lib_id "NX-J401-Adapter:MountingHole")
 		(at 295.91 187.96 0)
 		(unit 1)
@@
 			)
 		)
-		(property "Footprint" "MountingHole:MountingHole_2.5mm"
+		(property "Footprint" "NX-J401-Adapter:MountingHole_2.5mm"
 			(at 295.91 187.96 0)
 			(hide yes)
@@
 	)
 	(symbol
-		(lib_id "Mechanical:MountingHole")
+		(lib_id "NX-J401-Adapter:MountingHole")
 		(at 326.39 177.8 0)
 		(unit 1)
@@
 			)
 		)
-		(property "Footprint" "MountingHole:MountingHole_2.5mm"
+		(property "Footprint" "NX-J401-Adapter:MountingHole_2.5mm"
 			(at 326.39 177.8 0)
 			(hide yes)
@@
 	)
 	(symbol
-		(lib_id "Device:C_US")
+		(lib_id "NX-J401-Adapter:C_US")
 		(at 299.72 63.5 0)
 		(unit 1)
@@
 			)
 		)
-		(property "Footprint" "Capacitor_SMD:C_1210_3225Metric"
+		(property "Footprint" "NX-J401-Adapter:C_1210_3225Metric"
 			(at 299.72 63.5 0)
 			(hide yes)
@@
 	)
 	(symbol
-		(lib_id "Connector_Generic:Conn_01x02")
+		(lib_id "NX-J401-Adapter:Conn_01x02")
 		(at 78.74 66.04 180)
 		(unit 1)
@@
 	)
 	(symbol
-		(lib_id "Transistor_FET:CSD19534Q5A")
+		(lib_id "NX-J401-Adapter:CSD19534Q5A")
 		(at 143.51 48.26 270)
 		(mirror x)
@@
 	)
 	(symbol
-		(lib_id "Device:C_US")
+		(lib_id "NX-J401-Adapter:C_US")
 		(at 257.81 63.5 0)
 		(unit 1)
@@
 			)
 		)
-		(property "Footprint" "Capacitor_SMD:C_1210_3225Metric"
+		(property "Footprint" "NX-J401-Adapter:C_1210_3225Metric"
 			(at 257.81 63.5 0)
 			(hide yes)
@@
 	)
 	(symbol
-		(lib_id "Connector_Generic:Conn_01x02")
+		(lib_id "NX-J401-Adapter:Conn_01x02")
 		(at 347.98 119.38 0)
 		(mirror x)
@@
 	)
 	(symbol
-		(lib_id "Device:R_US")
+		(lib_id "NX-J401-Adapter:R_US")
 		(at 168.91 57.15 0)
 		(mirror y)
@@
 			)
 		)
-		(property "Footprint" "Resistor_SMD:R_0603_1608Metric"
+		(property "Footprint" "NX-J401-Adapter:R_0603_1608Metric"
 			(at 167.894 57.404 90)
 			(hide yes)
@@
 	)
 	(symbol
-		(lib_id "Graphic:SYM_Arrow_Large")
+		(lib_id "NX-J401-Adapter:SYM_Arrow_Large")
 		(at 74.93 237.49 0)
 		(unit 1)
@@
 			)
 		)
-		(property "Footprint" "Package_TO_SOT_SMD:SOT-23-6"
+		(property "Footprint" "NX-J401-Adapter:SOT-23-6"
 			(at 272.415 74.93 0)
 			(hide yes)
@@
 	)
 	(symbol
-		(lib_id "Device:C_US")
+		(lib_id "NX-J401-Adapter:C_US")
 		(at 269.24 57.15 0)
 		(mirror y)
@@
 			)
 		)
-		(property "Footprint" "Capacitor_SMD:C_0603_1608Metric"
+		(property "Footprint" "NX-J401-Adapter:C_0603_1608Metric"
 			(at 269.24 57.15 0)
 			(hide yes)
@@
 	)
 	(symbol
-		(lib_id "Switch:SW_Push")
+		(lib_id "NX-J401-Adapter:SW_Push")
 		(at 151.13 203.2 270)
 		(unit 1)
@@
 	)
 	(symbol
-		(lib_id "Mechanical:MountingHole")
+		(lib_id "NX-J401-Adapter:MountingHole")
 		(at 295.91 177.8 0)
 		(unit 1)
@@
 			)
 		)
-		(property "Footprint" "MountingHole:MountingHole_2.5mm"
+		(property "Footprint" "NX-J401-Adapter:MountingHole_2.5mm"
 			(at 295.91 177.8 0)
 			(hide yes)
@@
 	)
 	(symbol
-		(lib_id "Connector_Generic:Conn_01x02")
+		(lib_id "NX-J401-Adapter:Conn_01x02")
 		(at 347.98 71.12 0)
 		(mirror x)
@@
 	)
 	(symbol
-		(lib_id "Device:C_US")
+		(lib_id "NX-J401-Adapter:C_US")
 		(at 130.81 57.15 0)
 		(mirror y)
@@
 			)
 		)
-		(property "Footprint" "Capacitor_SMD:C_0603_1608Metric"
+		(property "Footprint" "NX-J401-Adapter:C_0603_1608Metric"
 			(at 130.81 57.15 0)
 			(hide yes)
@@
 	)
 	(symbol
-		(lib_id "Device:D_TVS")
+		(lib_id "NX-J401-Adapter:D_TVS")
 		(at 104.14 63.5 90)
 		(unit 1)
@@
 	)
 	(symbol
-		(lib_id "Mechanical:MountingHole")
+		(lib_id "NX-J401-Adapter:MountingHole")
 		(at 295.91 172.72 0)
 		(unit 1)
@@
 			)
 		)
-		(property "Footprint" "MountingHole:MountingHole_2.5mm"
+		(property "Footprint" "NX-J401-Adapter:MountingHole_2.5mm"
 			(at 295.91 172.72 0)
 			(hide yes)
@@
 	)
 	(symbol
-		(lib_id "Connector:Conn_01x15_Pin")
+		(lib_id "NX-J401-Adapter:Conn_01x15_Pin")
 		(at 39.37 193.04 0)
 		(unit 1)
@@
 			)
 		)
-		(property "Footprint" "Connector_PinHeader_2.54mm:PinHeader_1x15_P2.54mm_Horizontal"
+		(property "Footprint" "NX-J401-Adapter:PinHeader_1x15_P2.54mm_Horizontal"
 			(at 39.37 193.04 0)
 			(hide yes)
@@
 	)
 	(symbol
-		(lib_id "Connector_Generic:Conn_01x04")
+		(lib_id "NX-J401-Adapter:Conn_01x04")
 		(at 85.09 124.46 180)
 		(unit 1)
@@
 	)
 	(symbol
-		(lib_id "Mechanical:MountingHole")
+		(lib_id "NX-J401-Adapter:MountingHole")
 		(at 326.39 182.88 0)
 		(unit 1)
@@
 			)
 		)
-		(property "Footprint" "MountingHole:MountingHole_2.5mm"
+		(property "Footprint" "NX-J401-Adapter:MountingHole_2.5mm"
 			(at 326.39 182.88 0)
 			(hide yes)
@@
 	)
 	(symbol
-		(lib_id "Device:C_US")
+		(lib_id "NX-J401-Adapter:C_US")
 		(at 118.11 63.5 0)
 		(unit 1)
@@
 			)
 		)
-		(property "Footprint" "Capacitor_SMD:C_1210_3225Metric"
+		(property "Footprint" "NX-J401-Adapter:C_1210_3225Metric"
 			(at 118.11 63.5 0)
 			(hide yes)
@@
 	(symbol
 		(lib_name "LED_1")
-		(lib_id "Device:LED")
+		(lib_id "NX-J401-Adapter:LED_1")
 		(at 114.3 201.93 90)
 		(unit 1)
@@
 			)
 		)
-		(property "Footprint" "LED_SMD:LED_1206_3216Metric"
+		(property "Footprint" "NX-J401-Adapter:LED_1206_3216Metric"
 			(at 114.3 201.93 0)
 			(hide yes)
@@
 	)
 	(symbol
-		(lib_id "Switch:SW_Push")
+		(lib_id "NX-J401-Adapter:SW_Push")
 		(at 133.35 203.2 270)
 		(unit 1)
@@
 	)
 	(symbol
-		(lib_id "Transistor_FET:CSD19534Q5A")
+		(lib_id "NX-J401-Adapter:CSD19534Q5A")
 		(at 281.94 48.26 270)
 		(mirror x)

Commit message: Adjusted connector positioning to more closely match J401.
Signed-off-by: Scott Berman <sgberman1@gmail.com>
Parts:
- renumbered C4 to C3, C10 to C7, H7 to H2, H2 to H3, H8 to H5, H5 to H7, H6 to H8, J5 to J4, J4 to J7
Changed lines of the file:
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@@
 		(dnp no)
 		(fields_autoplaced yes)
-		(property "Reference" "H6"
+		(property "Reference" "H8"
 			(at 298.45 181.6099 0)
 			(show_name no)
@@
 			(project "NX-J401-Adapter-v6"
 				(path "/3c9fa76f-2b37-4666-8575-58caa65def04"
-					(reference "H6")
+					(reference "H8")
 					(unit 1)
 				)
@@
 		(dnp no)
 		(fields_autoplaced yes)
-		(property "Reference" "H2"
+		(property "Reference" "H3"
 			(at 298.45 186.6899 0)
 			(show_name no)
@@
 			(project "NX-J401-Adapter-v6"
 				(path "/3c9fa76f-2b37-4666-8575-58caa65def04"
-					(reference "H2")
+					(reference "H3")
 					(unit 1)
 				)
@@
 		(dnp no)
 		(fields_autoplaced yes)
-		(property "Reference" "H7"
+		(property "Reference" "H2"
 			(at 328.93 176.5299 0)
 			(show_name no)
@@
 			(project "NX-J401-Adapter-v6"
 				(path "/3c9fa76f-2b37-4666-8575-58caa65def04"
-					(reference "H7")
+					(reference "H2")
 					(unit 1)
 				)
@@
 		(in_pos_files yes)
 		(dnp no)
-		(property "Reference" "C10"
+		(property "Reference" "C7"
 			(at 259.588 61.468 90)
 			(show_name no)
@@
 			(project "NX-J401-Adapter-v6"
 				(path "/3c9fa76f-2b37-4666-8575-58caa65def04"
-					(reference "C10")
+					(reference "C7")
 					(unit 1)
 				)
@@
 		(in_pos_files yes)
 		(dnp no)
-		(property "Reference" "C4"
+		(property "Reference" "C3"
 			(at 270.764 54.61 90)
 			(show_name no)
@@
 			(project "NX-J401-Adapter-v6"
 				(path "/3c9fa76f-2b37-4666-8575-58caa65def04"
-					(reference "C4")
+					(reference "C3")
 					(unit 1)
 				)
@@
 		(dnp no)
 		(fields_autoplaced yes)
-		(property "Reference" "H5"
+		(property "Reference" "H7"
 			(at 298.45 176.5299 0)
 			(show_name no)
@@
 			(project "NX-J401-Adapter-v6"
 				(path "/3c9fa76f-2b37-4666-8575-58caa65def04"
-					(reference "H5")
+					(reference "H7")
 					(unit 1)
 				)
@@
 		(in_pos_files yes)
 		(dnp no)
-		(property "Reference" "J5"
+		(property "Reference" "J4"
 			(at 347.726 65.024 0)
 			(show_name no)
@@
 			(project "NX-J401-Adapter-v6"
 				(path "/3c9fa76f-2b37-4666-8575-58caa65def04"
-					(reference "J5")
+					(reference "J4")
 					(unit 1)
 				)
@@
 		(in_pos_files yes)
 		(dnp no)
-		(property "Reference" "J4"
+		(property "Reference" "J7"
 			(at 85.09 116.84 0)
 			(show_name no)
@@
 			(project "NX-J401-Adapter-v6"
 				(path "/3c9fa76f-2b37-4666-8575-58caa65def04"
-					(reference "J4")
+					(reference "J7")
 					(unit 1)
 				)
@@
 		(dnp no)
 		(fields_autoplaced yes)
-		(property "Reference" "H8"
+		(property "Reference" "H5"
 			(at 328.93 181.6099 0)
 			(show_name no)
@@
 			(project "NX-J401-Adapter-v6"
 				(path "/3c9fa76f-2b37-4666-8575-58caa65def04"
-					(reference "H8")
+					(reference "H5")
 					(unit 1)
 				)
