File: circuit-boards/NX-J401-Adapter-v6/canable2.kicad_sch (KiCad schematic)
At the start: 29 parts, among them J8 SWD, Q1 SI2301CDS-T1-GE3, Q5 SS8050, Q8 SI2301CDS-T1-GE3, U1 TPS613222ADBV, U3 STM32G431CBTx, U6 TJA1051T/3/1J

Commit message: Updates
Signed-off-by: Scott Berman <sgberman1@gmail.com>
Parts:
- C1, C2, C22, C3: footprint Capacitor_SMD:C_0805_2012Metric -> NX-J401-Adapter:C_0805_2012Metric; symbol Device:C_US -> NX-J401-Adapter:C_US
- C11, C21, C36, C44, C6, C7, C8, C9: footprint Capacitor_SMD:C_0603_1608Metric -> NX-J401-Adapter:C_0603_1608Metric; symbol Device:C_US -> NX-J401-Adapter:C_US
- D5: footprint Package_TO_SOT_SMD:SOT-23 -> NX-J401-Adapter:SOT-23
- D8, D9: footprint LED_SMD:LED_1206_3216Metric -> NX-J401-Adapter:LED_1206_3216Metric; symbol Device:LED -> NX-J401-Adapter:LED
- J8: footprint Connector_PinHeader_2.54mm:PinHeader_1x05_P2.54mm_Horizontal -> NX-J401-Adapter:PinHeader_1x05_P2.54mm_Horizontal; symbol Connector_Generic:Conn_01x05 -> NX-J401-Adapter:Conn_01x05
- L1: symbol Device:L_Iron -> NX-J401-Adapter:L_Iron
- Q1, Q8: footprint Package_TO_SOT_SMD:SOT-23 -> NX-J401-Adapter:SOT-23; symbol Transistor_FET:Si2319CDS -> NX-J401-Adapter:Si2319CDS
- Q5: footprint Package_TO_SOT_SMD:SOT-23 -> NX-J401-Adapter:SOT-23; symbol Transistor_BJT:SS8050 -> NX-J401-Adapter:SS8050
- R1, R2, R3, R4, R5, R7: footprint Resistor_SMD:R_0603_1608Metric -> NX-J401-Adapter:R_0603_1608Metric; symbol Device:R_US -> NX-J401-Adapter:R_US
- U1: footprint Package_TO_SOT_SMD:SOT-23-5 -> NX-J401-Adapter:SOT-23-5; symbol Regulator_Switching:TPS613222ADBV -> NX-J401-Adapter:TPS613222ADBV
- U3: footprint Package_QFP:LQFP-48_7x7mm_P0.5mm -> NX-J401-Adapter:LQFP-48_7x7mm_P0.5mm; symbol MCU_ST_STM32G4:STM32G431CBTx -> NX-J401-Adapter:STM32G431CBTx
- U6: footprint Package_SO:SO-8_3.9x4.9mm_P1.27mm -> NX-J401-Adapter:SO-8_3.9x4.9mm_P1.27mm; symbol Interface_CAN_LIN:TJA1051TK-3 -> NX-J401-Adapter:TJA1051TK-3
Other:
- note added: "Reverse Polarity Protection"
Changed lines of the file:
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@@
 	(title_block
 		(title "NX J401 Adapter")
-		(date "2026-05-25")
+		(date "2026-06-02")
 		(rev "6")
 		(company "SPACE COOKIES FRC TEAM 1868")
 	)
+	(text "Reverse Polarity Protection"
+		(exclude_from_sim no)
+		(at 76.454 30.988 0)
+		(effects
+			(font
+				(size 1.27 1.27)
+			)
+		)
+	)
 	(junction
 		(at 114.3 232.41)
@@
 	)
 	(symbol
-		(lib_id "Transistor_FET:Si2319CDS")
+		(lib_id "NX-J401-Adapter:Si2319CDS")
 		(at 246.38 35.56 270)
 		(mirror x)
@@
 			)
 		)
-		(property "Footprint" "Package_TO_SOT_SMD:SOT-23"
+		(property "Footprint" "NX-J401-Adapter:SOT-23"
 			(at 244.475 30.48 0)
 			(hide yes)
@@
 	)
 	(symbol
-		(lib_id "Connector_Generic:Conn_01x05")
+		(lib_id "NX-J401-Adapter:Conn_01x05")
 		(at 317.5 173.99 0)
 		(unit 1)
@@
 			)
 		)
-		(property "Footprint" "Connector_PinHeader_2.54mm:PinHeader_1x05_P2.54mm_Horizontal"
+		(property "Footprint" "NX-J401-Adapter:PinHeader_1x05_P2.54mm_Horizontal"
 			(at 317.5 173.99 0)
 			(hide yes)
@@
 	)
 	(symbol
-		(lib_id "Transistor_FET:Si2319CDS")
+		(lib_id "NX-J401-Adapter:Si2319CDS")
 		(at 76.2 43.18 90)
 		(unit 1)
@@
 			)
 		)
-		(property "Footprint" "Package_TO_SOT_SMD:SOT-23"
+		(property "Footprint" "NX-J401-Adapter:SOT-23"
 			(at 78.105 38.1 0)
 			(hide yes)
@@
 	)
 	(symbol
-		(lib_id "Device:C_US")
+		(lib_id "NX-J401-Adapter:C_US")
 		(at 95.25 53.34 0)
 		(unit 1)
@@
 			)
 		)
-		(property "Footprint" "Capacitor_SMD:C_0805_2012Metric"
+		(property "Footprint" "NX-J401-Adapter:C_0805_2012Metric"
 			(at 95.25 53.34 0)
 			(hide yes)
@@
 	)
 	(symbol
-		(lib_id "Device:R_US")
+		(lib_id "NX-J401-Adapter:R_US")
 		(at 231.14 195.58 0)
 		(mirror y)
@@
 			)
 		)
-		(property "Footprint" "Resistor_SMD:R_0603_1608Metric"
+		(property "Footprint" "NX-J401-Adapter:R_0603_1608Metric"
 			(at 230.124 195.834 90)
 			(hide yes)
@@
 	)
 	(symbol
-		(lib_id "Device:LED")
+		(lib_id "NX-J401-Adapter:LED")
 		(at 231.14 182.88 90)
 		(unit 1)
@@
 			)
 		)
-		(property "Footprint" "LED_SMD:LED_1206_3216Metric"
+		(property "Footprint" "NX-J401-Adapter:LED_1206_3216Metric"
 			(at 231.14 182.88 0)
 			(hide yes)
@@
 	)
 	(symbol
-		(lib_id "Device:C_US")
+		(lib_id "NX-J401-Adapter:C_US")
 		(at 124.46 214.63 0)
 		(mirror y)
@@
 			)
 		)
-		(property "Footprint" "Capacitor_SMD:C_0603_1608Metric"
+		(property "Footprint" "NX-J401-Adapter:C_0603_1608Metric"
 			(at 124.46 214.63 0)
 			(hide yes)
@@
 	)
 	(symbol
-		(lib_id "Device:R_US")
+		(lib_id "NX-J401-Adapter:R_US")
 		(at 166.37 93.98 0)
 		(mirror y)
@@
 			)
 		)
-		(property "Footprint" "Resistor_SMD:R_0603_1608Metric"
+		(property "Footprint" "NX-J401-Adapter:R_0603_1608Metric"
 			(at 165.354 94.234 90)
 			(hide yes)
@@
 	)
 	(symbol
-		(lib_id "Device:C_US")
+		(lib_id "NX-J401-Adapter:C_US")
 		(at 154.94 214.63 0)
 		(mirror y)
@@
 			)
 		)
-		(property "Footprint" "Capacitor_SMD:C_0603_1608Metric"
+		(property "Footprint" "NX-J401-Adapter:C_0603_1608Metric"
 			(at 154.94 214.63 0)
 			(hide yes)
@@
 	)
 	(symbol
-		(lib_id "Transistor_BJT:SS8050")
+		(lib_id "NX-J401-Adapter:SS8050")
 		(at 243.84 53.34 0)
 		(unit 1)
@@
 			)
 		)
-		(property "Footprint" "Package_TO_SOT_SMD:SOT-23"
+		(property "Footprint" "NX-J401-Adapter:SOT-23"
 			(at 248.92 60.706 0)
 			(hide yes)
@@
 	)
 	(symbol
-		(lib_id "Device:C_US")
+		(lib_id "NX-J401-Adapter:C_US")
 		(at 114.3 214.63 0)
 		(mirror y)
@@
 			)
 		)
-		(property "Footprint" "Capacitor_SMD:C_0603_1608Metric"
+		(property "Footprint" "NX-J401-Adapter:C_0603_1608Metric"
 			(at 114.3 214.63 0)
 			(hide yes)
@@
 	)
 	(symbol
-		(lib_id "Device:LED")
+		(lib_id "NX-J401-Adapter:LED")
 		(at 217.17 182.88 90)
 		(unit 1)
@@
 			)
 		)
-		(property "Footprint" "LED_SMD:LED_1206_3216Metric"
+		(property "Footprint" "NX-J401-Adapter:LED_1206_3216Metric"
 			(at 217.17 182.88 0)
 			(hide yes)
@@
 	)
 	(symbol
-		(lib_id "Device:R_US")
+		(lib_id "NX-J401-Adapter:R_US")
 		(at 238.76 39.37 0)
 		(mirror y)
@@
 			)
 		)
-		(property "Footprint" "Resistor_SMD:R_0603_1608Metric"
+		(property "Footprint" "NX-J401-Adapter:R_0603_1608Metric"
 			(at 237.744 39.624 90)
 			(hide yes)
@@
 	)
 	(symbol
-		(lib_id "Device:L_Iron")
+		(lib_id "NX-J401-Adapter:L_Iron")
 		(at 105.41 40.64 90)
 		(unit 1)
@@
 	)
 	(symbol
-		(lib_id "Device:C_US")
+		(lib_id "NX-J401-Adapter:C_US")
 		(at 148.59 53.34 0)
 		(unit 1)
@@
 			)
 		)
-		(property "Footprint" "Capacitor_SMD:C_0805_2012Metric"
+		(property "Footprint" "NX-J401-Adapter:C_0805_2012Metric"
 			(at 148.59 53.34 0)
 			(hide yes)
@@
 			)
 		)
-		(property "Footprint" "Package_TO_SOT_SMD:SOT-23"
+		(property "Footprint" "NX-J401-Adapter:SOT-23"
 			(at 318.77 142.24 0)
 			(hide yes)
@@
 	)
 	(symbol
-		(lib_id "Device:C_US")
+		(lib_id "NX-J401-Adapter:C_US")
 		(at 160.02 53.34 0)
 		(unit 1)
@@
 			)
 		)
-		(property "Footprint" "Capacitor_SMD:C_0805_2012Metric"
+		(property "Footprint" "NX-J401-Adapter:C_0805_2012Metric"
 			(at 160.02 53.34 0)
 			(hide yes)
@@
 	)
 	(symbol
-		(lib_id "MCU_ST_STM32G4:STM32G431CBTx")
+		(lib_id "NX-J401-Adapter:STM32G431CBTx")
 		(at 134.62 138.43 0)
 		(mirror y)
@@
 			)
 		)
-		(property "Footprint" "Package_QFP:LQFP-48_7x7mm_P0.5mm"
+		(property "Footprint" "NX-J401-Adapter:LQFP-48_7x7mm_P0.5mm"
 			(at 149.86 176.53 0)
 			(hide yes)
@@
 	)
 	(symbol
-		(lib_id "Device:R_US")
+		(lib_id "NX-J401-Adapter:R_US")
 		(at 158.75 170.18 0)
 		(mirror y)
@@
 			)
 		)
-		(property "Footprint" "Resistor_SMD:R_0603_1608Metric"
+		(property "Footprint" "NX-J401-Adapter:R_0603_1608Metric"
 			(at 157.734 170.434 90)
 			(hide yes)
@@
 	)
 	(symbol
-		(lib_id "Interface_CAN_LIN:TJA1051TK-3")
+		(lib_id "NX-J401-Adapter:TJA1051TK-3")
 		(at 283.21 133.35 0)
 		(unit 1)
@@
 			)
 		)
-		(property "Footprint" "Package_SO:SO-8_3.9x4.9mm_P1.27mm"
+		(property "Footprint" "NX-J401-Adapter:SO-8_3.9x4.9mm_P1.27mm"
 			(at 283.21 154.178 0)
 			(hide yes)
@@
 	)
 	(symbol
-		(lib_id "Device:C_US")
+		(lib_id "NX-J401-Adapter:C_US")
 		(at 166.37 104.14 0)
 		(mirror y)
@@
 			)
 		)
-		(property "Footprint" "Capacitor_SMD:C_0603_1608Metric"
+		(property "Footprint" "NX-J401-Adapter:C_0603_1608Metric"
 			(at 166.37 104.14 0)
 			(hide yes)
@@
 	)
 	(symbol
-		(lib_id "Device:R_US")
+		(lib_id "NX-J401-Adapter:R_US")
 		(at 215.9 43.18 0)
 		(mirror y)
@@
 			)
 		)
-		(property "Footprint" "Resistor_SMD:R_0603_1608Metric"
+		(property "Footprint" "NX-J401-Adapter:R_0603_1608Metric"
 			(at 214.884 43.434 90)
 			(hide yes)
@@
 	)
 	(symbol
-		(lib_id "Device:C_US")
+		(lib_id "NX-J401-Adapter:C_US")
 		(at 215.9 59.69 0)
 		(mirror y)
@@
 			)
 		)
-		(property "Footprint" "Capacitor_SMD:C_0805_2012Metric"
+		(property "Footprint" "NX-J401-Adapter:C_0805_2012Metric"
 			(at 215.9 59.69 0)
 			(hide yes)
@@
 	)
 	(symbol
-		(lib_id "Device:C_US")
+		(lib_id "NX-J401-Adapter:C_US")
 		(at 134.62 214.63 0)
 		(mirror y)
@@
 			)
 		)
-		(property "Footprint" "Capacitor_SMD:C_0603_1608Metric"
+		(property "Footprint" "NX-J401-Adapter:C_0603_1608Metric"
 			(at 134.62 214.63 0)
 			(hide yes)
@@
 	)
 	(symbol
-		(lib_id "Device:C_US")
+		(lib_id "NX-J401-Adapter:C_US")
 		(at 144.78 214.63 0)
 		(mirror y)
@@
 			)
 		)
-		(property "Footprint" "Capacitor_SMD:C_0603_1608Metric"
+		(property "Footprint" "NX-J401-Adapter:C_0603_1608Metric"
 			(at 144.78 214.63 0)
 			(hide yes)
@@
 	)
 	(symbol
-		(lib_id "Device:R_US")
+		(lib_id "NX-J401-Adapter:R_US")
 		(at 217.17 195.58 0)
 		(mirror y)
@@
 			)
 		)
-		(property "Footprint" "Resistor_SMD:R_0603_1608Metric"
+		(property "Footprint" "NX-J401-Adapter:R_0603_1608Metric"
 			(at 216.154 195.834 90)
 			(hide yes)
@@
 	)
 	(symbol
-		(lib_id "Device:C_US")
+		(lib_id "NX-J401-Adapter:C_US")
 		(at 260.35 142.24 0)
 		(mirror y)
@@
 			)
 		)
-		(property "Footprint" "Capacitor_SMD:C_0603_1608Metric"
+		(property "Footprint" "NX-J401-Adapter:C_0603_1608Metric"
 			(at 260.35 142.24 0)
 			(hide yes)
@@
 	)
 	(symbol
-		(lib_id "Regulator_Switching:TPS613222ADBV")
+		(lib_id "NX-J401-Adapter:TPS613222ADBV")
 		(at 130.81 43.18 0)
 		(unit 1)
@@
 			)
 		)
-		(property "Footprint" "Package_TO_SOT_SMD:SOT-23-5"
+		(property "Footprint" "NX-J401-Adapter:SOT-23-5"
 			(at 130.81 63.5 0)
 			(hide yes)
@@
 	)
 	(symbol
-		(lib_id "Device:C_US")
+		(lib_id "NX-J401-Adapter:C_US")
 		(at 273.05 116.84 0)
 		(mirror y)
@@
 			)
 		)
-		(property "Footprint" "Capacitor_SMD:C_0603_1608Metric"
+		(property "Footprint" "NX-J401-Adapter:C_0603_1608Metric"
 			(at 273.05 116.84 0)
 			(hide yes)

Commit message: Adjusted connector positioning to more closely match J401.
Signed-off-by: Scott Berman <sgberman1@gmail.com>
Parts:
- renumbered C3 to C1, C9 to C10, C11 to C20, C21 to C30, C22 to C31, C1 to C4, C7 to C8, C8 to C9, Q5 to Q7, R7 to R11, R5 to R6
Changed lines of the file:
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@@
 		(in_pos_files yes)
 		(dnp no)
-		(property "Reference" "C3"
+		(property "Reference" "C1"
 			(at 96.266 50.546 0)
 			(show_name no)
@@
 			(project "NX-J401-Adapter-v6"
 				(path "/3c9fa76f-2b37-4666-8575-58caa65def04/958ef65b-dc3d-4755-b7b0-3d4dc8feed9f"
-					(reference "C3")
+					(reference "C1")
 					(unit 1)
 				)
@@
 		(in_pos_files yes)
 		(dnp no)
-		(property "Reference" "C7"
+		(property "Reference" "C8"
 			(at 128.27 214.63 90)
 			(show_name no)
@@
 			(project "NX-J401-Adapter-v6"
 				(path "/3c9fa76f-2b37-4666-8575-58caa65def04/958ef65b-dc3d-4755-b7b0-3d4dc8feed9f"
-					(reference "C7")
+					(reference "C8")
 					(unit 1)
 				)
@@
 		(dnp no)
 		(fields_autoplaced yes)
-		(property "Reference" "Q5"
+		(property "Reference" "Q7"
 			(at 248.92 52.0699 0)
 			(show_name no)
@@
 			(project "NX-J401-Adapter-v6"
 				(path "/3c9fa76f-2b37-4666-8575-58caa65def04/958ef65b-dc3d-4755-b7b0-3d4dc8feed9f"
-					(reference "Q5")
+					(reference "Q7")
 					(unit 1)
 				)
@@
 		(in_pos_files yes)
 		(dnp no)
-		(property "Reference" "C9"
+		(property "Reference" "C10"
 			(at 118.11 214.63 90)
 			(show_name no)
@@
 			(project "NX-J401-Adapter-v6"
 				(path "/3c9fa76f-2b37-4666-8575-58caa65def04/958ef65b-dc3d-4755-b7b0-3d4dc8feed9f"
-					(reference "C9")
+					(reference "C10")
 					(unit 1)
 				)
@@
 		(in_pos_files yes)
 		(dnp no)
-		(property "Reference" "R5"
+		(property "Reference" "R6"
 			(at 237.236 37.846 0)
 			(show_name no)
@@
 			(project "NX-J401-Adapter-v6"
 				(path "/3c9fa76f-2b37-4666-8575-58caa65def04/958ef65b-dc3d-4755-b7b0-3d4dc8feed9f"
-					(reference "R5")
+					(reference "R6")
 					(unit 1)
 				)
@@
 		(in_pos_files yes)
 		(dnp no)
-		(property "Reference" "C1"
+		(property "Reference" "C4"
 			(at 161.036 50.546 0)
 			(show_name no)
@@
 			(project "NX-J401-Adapter-v6"
 				(path "/3c9fa76f-2b37-4666-8575-58caa65def04/958ef65b-dc3d-4755-b7b0-3d4dc8feed9f"
-					(reference "C1")
+					(reference "C4")
 					(unit 1)
 				)
@@
 		(in_pos_files yes)
 		(dnp no)
-		(property "Reference" "C21"
+		(property "Reference" "C30"
 			(at 167.132 101.854 0)
 			(show_name no)
@@
 			(project "NX-J401-Adapter-v6"
 				(path "/3c9fa76f-2b37-4666-8575-58caa65def04/958ef65b-dc3d-4755-b7b0-3d4dc8feed9f"
-					(reference "C21")
+					(reference "C30")
 					(unit 1)
 				)
@@
 		(in_pos_files yes)
 		(dnp no)
-		(property "Reference" "R7"
+		(property "Reference" "R11"
 			(at 214.376 41.656 0)
 			(show_name no)
@@
 			(project "NX-J401-Adapter-v6"
 				(path "/3c9fa76f-2b37-4666-8575-58caa65def04/958ef65b-dc3d-4755-b7b0-3d4dc8feed9f"
-					(reference "R7")
+					(reference "R11")
 					(unit 1)
 				)
@@
 		(in_pos_files yes)
 		(dnp no)
-		(property "Reference" "C22"
+		(property "Reference" "C31"
 			(at 212.09 57.658 0)
 			(show_name no)
@@
 			(project "NX-J401-Adapter-v6"
 				(path "/3c9fa76f-2b37-4666-8575-58caa65def04/958ef65b-dc3d-4755-b7b0-3d4dc8feed9f"
-					(reference "C22")
+					(reference "C31")
 					(unit 1)
 				)
@@
 		(in_pos_files yes)
 		(dnp no)
-		(property "Reference" "C8"
+		(property "Reference" "C9"
 			(at 138.43 214.63 90)
 			(show_name no)
@@
 			(project "NX-J401-Adapter-v6"
 				(path "/3c9fa76f-2b37-4666-8575-58caa65def04/958ef65b-dc3d-4755-b7b0-3d4dc8feed9f"
-					(reference "C8")
+					(reference "C9")
 					(unit 1)
 				)
@@
 		(in_pos_files yes)
 		(dnp no)
-		(property "Reference" "C11"
+		(property "Reference" "C20"
 			(at 148.59 214.63 90)
 			(show_name no)
@@
 			(project "NX-J401-Adapter-v6"
 				(path "/3c9fa76f-2b37-4666-8575-58caa65def04/958ef65b-dc3d-4755-b7b0-3d4dc8feed9f"
-					(reference "C11")
+					(reference "C20")
 					(unit 1)
 				)
