File: circuit-boards/NX-J401-Adapter-v7/NX-J401-Adapter-v7.kicad_sch (KiCad schematic)
At the start: 32 parts, among them J1 Terminal, J10 POWER, J2 Terminal, J3 NX CONTROL & UART, J4 15V, J7 USB1, J9 CAN1, Q2 CSD19534Q5A, Q9 CSD19534Q5A, SW1 RESET, SW2 RECOVERY, U2 LM74700QDBVRQ1, U4 LM74700QDBVRQ1

Commit message: Routed PCB
Signed-off-by: scott <scott@scott-Z590I-AORUS-ULTRA.bb>
Parts:
- renumbered C7 to C1, C5 to C11, C3 to C12, C42 to C45, C41 to C52, C40 to C54, D3 to D1, D6 to D2, D7 to D3, H3 to H2, H7 to H5, H8 to H6, Q2 to Q1, R16 to R23, SW1 to SW2, SW2 to SW3, U2 to U1, U4 to U7
Changed lines of the file:
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@@
 		(dnp no)
 		(fields_autoplaced yes)
-		(property "Reference" "H8"
+		(property "Reference" "H6"
 			(at 298.45 181.6099 0)
 			(show_name no)
@@
 			(project "NX-J401-Adapter-v7"
 				(path "/3c9fa76f-2b37-4666-8575-58caa65def04"
-					(reference "H8")
+					(reference "H6")
 					(unit 1)
 				)
@@
 		(in_pos_files yes)
 		(dnp no)
-		(property "Reference" "C42"
+		(property "Reference" "C45"
 			(at 163.068 61.468 90)
 			(show_name no)
@@
 			(project "NX-J401-Adapter-v7"
 				(path "/3c9fa76f-2b37-4666-8575-58caa65def04"
-					(reference "C42")
+					(reference "C45")
 					(unit 1)
 				)
@@
 		(in_pos_files yes)
 		(dnp no)
-		(property "Reference" "U4"
+		(property "Reference" "U7"
 			(at 148.844 75.184 0)
 			(show_name no)
@@
 			(project "NX-J401-Adapter-v7"
 				(path "/3c9fa76f-2b37-4666-8575-58caa65def04"
-					(reference "U4")
+					(reference "U7")
 					(unit 1)
 				)
@@
 		(in_pos_files yes)
 		(dnp no)
-		(property "Reference" "D6"
+		(property "Reference" "D2"
 			(at 171.45 70.104 90)
 			(show_name no)
@@
 			(project "NX-J401-Adapter-v7"
 				(path "/3c9fa76f-2b37-4666-8575-58caa65def04"
-					(reference "D6")
+					(reference "D2")
 					(unit 1)
 				)
@@
 		(dnp no)
 		(fields_autoplaced yes)
-		(property "Reference" "H3"
+		(property "Reference" "H2"
 			(at 298.45 186.6899 0)
 			(show_name no)
@@
 			(project "NX-J401-Adapter-v7"
 				(path "/3c9fa76f-2b37-4666-8575-58caa65def04"
-					(reference "H3")
+					(reference "H2")
 					(unit 1)
 				)
@@
 		(in_pos_files yes)
 		(dnp no)
-		(property "Reference" "C5"
+		(property "Reference" "C11"
 			(at 301.498 61.468 90)
 			(show_name no)
@@
 			(project "NX-J401-Adapter-v7"
 				(path "/3c9fa76f-2b37-4666-8575-58caa65def04"
-					(reference "C5")
+					(reference "C11")
 					(unit 1)
 				)
@@
 		(in_pos_files yes)
 		(dnp no)
-		(property "Reference" "C7"
+		(property "Reference" "C1"
 			(at 259.588 61.468 90)
 			(show_name no)
@@
 			(project "NX-J401-Adapter-v7"
 				(path "/3c9fa76f-2b37-4666-8575-58caa65def04"
-					(reference "C7")
+					(reference "C1")
 					(unit 1)
 				)
@@
 		(in_pos_files yes)
 		(dnp no)
-		(property "Reference" "R16"
+		(property "Reference" "R23"
 			(at 166.37 57.15 90)
 			(show_name no)
@@
 			(project "NX-J401-Adapter-v7"
 				(path "/3c9fa76f-2b37-4666-8575-58caa65def04"
-					(reference "R16")
+					(reference "R23")
 					(unit 1)
 				)
@@
 		(in_pos_files yes)
 		(dnp no)
-		(property "Reference" "U2"
+		(property "Reference" "U1"
 			(at 287.274 75.184 0)
 			(show_name no)
@@
 			(project "NX-J401-Adapter-v7"
 				(path "/3c9fa76f-2b37-4666-8575-58caa65def04"
-					(reference "U2")
+					(reference "U1")
 					(unit 1)
 				)
@@
 		(in_pos_files yes)
 		(dnp no)
-		(property "Reference" "C3"
+		(property "Reference" "C12"
 			(at 270.764 54.61 90)
 			(show_name no)
@@
 			(project "NX-J401-Adapter-v7"
 				(path "/3c9fa76f-2b37-4666-8575-58caa65def04"
-					(reference "C3")
+					(reference "C12")
 					(unit 1)
 				)
@@
 		(dnp no)
 		(fields_autoplaced yes)
-		(property "Reference" "SW1"
+		(property "Reference" "SW2"
 			(at 154.94 201.93 90)
 			(show_name no)
@@
 			(project "NX-J401-Adapter-v7"
 				(path "/3c9fa76f-2b37-4666-8575-58caa65def04"
-					(reference "SW1")
+					(reference "SW2")
 					(unit 1)
 				)
@@
 		(dnp no)
 		(fields_autoplaced yes)
-		(property "Reference" "H7"
+		(property "Reference" "H5"
 			(at 298.45 176.5299 0)
 			(show_name no)
@@
 			(project "NX-J401-Adapter-v7"
 				(path "/3c9fa76f-2b37-4666-8575-58caa65def04"
-					(reference "H7")
+					(reference "H5")
 					(unit 1)
 				)
@@
 		(in_pos_files yes)
 		(dnp no)
-		(property "Reference" "C41"
+		(property "Reference" "C52"
 			(at 132.334 54.61 90)
 			(show_name no)
@@
 			(project "NX-J401-Adapter-v7"
 				(path "/3c9fa76f-2b37-4666-8575-58caa65def04"
-					(reference "C41")
+					(reference "C52")
 					(unit 1)
 				)
@@
 		(in_pos_files yes)
 		(dnp no)
-		(property "Reference" "D3"
+		(property "Reference" "D1"
 			(at 106.68 62.2299 90)
 			(show_name no)
@@
 			(project "NX-J401-Adapter-v7"
 				(path "/3c9fa76f-2b37-4666-8575-58caa65def04"
-					(reference "D3")
+					(reference "D1")
 					(unit 1)
 				)
@@
 		(in_pos_files yes)
 		(dnp no)
-		(property "Reference" "C40"
+		(property "Reference" "C54"
 			(at 119.888 61.468 90)
 			(show_name no)
@@
 			(project "NX-J401-Adapter-v7"
 				(path "/3c9fa76f-2b37-4666-8575-58caa65def04"
-					(reference "C40")
+					(reference "C54")
 					(unit 1)
 				)
@@
 		(in_pos_files yes)
 		(dnp no)
-		(property "Reference" "D7"
+		(property "Reference" "D3"
 			(at 116.84 200.914 90)
 			(show_name no)
@@
 			(project "NX-J401-Adapter-v7"
 				(path "/3c9fa76f-2b37-4666-8575-58caa65def04"
-					(reference "D7")
+					(reference "D3")
 					(unit 1)
 				)
@@
 		(dnp no)
 		(fields_autoplaced yes)
-		(property "Reference" "SW2"
+		(property "Reference" "SW3"
 			(at 137.16 201.93 90)
 			(show_name no)
@@
 			(project "NX-J401-Adapter-v7"
 				(path "/3c9fa76f-2b37-4666-8575-58caa65def04"
-					(reference "SW2")
+					(reference "SW3")
 					(unit 1)
 				)
@@
 		(in_pos_files yes)
 		(dnp no)
-		(property "Reference" "Q2"
+		(property "Reference" "Q1"
 			(at 281.94 39.37 90)
 			(show_name no)
@@
 			(project "NX-J401-Adapter-v7"
 				(path "/3c9fa76f-2b37-4666-8575-58caa65def04"
-					(reference "Q2")
+					(reference "Q1")
 					(unit 1)
 				)
