File: circuit-boards/NX-J401-Adapter-v7/NX-J401-Adapter-v7.kicad_sch (KiCad schematic)
At the start: 32 parts, among them J1 Terminal, J10 POWER, J2 Terminal, J3 NX CONTROL & UART, J4 15V, J7 USB1, J9 CAN1, Q1 CSD19534Q5A, Q9 CSD19534Q5A, SW1 RESET, SW2 RECOVERY, U1 LM74700QDBVRQ1, U7 LM74700QDBVRQ1

Commit message: PCB update
Signed-off-by: Scott Berman <sgberman1@gmail.com>
Parts:
- LP1, LP2, LP3, LP4: value (none) -> Light Pipe; JLCPCB P/N (none) -> XXXXXX
- SW1, SW2: JLCPCB P/N (none) -> XXXXXX
Changed lines of the file:
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@@
 	(title_block
 		(title "NX J401 Adapter")
-		(date "2026-06-02")
-		(rev "6")
+		(date "2026-08-01")
+		(rev "7")
 		(company "SPACE COOKIES FRC TEAM 1868")
 	)
@@
 			)
 		)
-		(property "Value" ""
+		(property "Value" "Light Pipe"
 			(at 175.26 220.98 0)
 			(show_name no)
@@
 			)
 		)
+		(property "JLCPCB P/N" "XXXXXX"
+			(at 175.26 220.98 0)
+			(hide yes)
+			(show_name no)
+			(do_not_autoplace no)
+			(effects
+				(font
+					(size 1.27 1.27)
+				)
+			)
+		)
 		(instances
 			(project "NX-J401-Adapter-v7"
@@
 			)
 		)
-		(property "Value" ""
+		(property "Value" "Light Pipe"
 			(at 175.26 247.65 0)
 			(show_name no)
@@
 			)
 		)
+		(property "JLCPCB P/N" "XXXXXX"
+			(at 175.26 247.65 0)
+			(hide yes)
+			(show_name no)
+			(do_not_autoplace no)
+			(effects
+				(font
+					(size 1.27 1.27)
+				)
+			)
+		)
 		(instances
 			(project "NX-J401-Adapter-v7"
@@
 			)
 		)
-		(property "Value" ""
+		(property "Value" "Light Pipe"
 			(at 175.26 238.76 0)
 			(show_name no)
@@
 			)
 		)
+		(property "JLCPCB P/N" "XXXXXX"
+			(at 175.26 238.76 0)
+			(hide yes)
+			(show_name no)
+			(do_not_autoplace no)
+			(effects
+				(font
+					(size 1.27 1.27)
+				)
+			)
+		)
 		(instances
 			(project "NX-J401-Adapter-v7"
@@
 			)
 		)
+		(property "JLCPCB P/N" "XXXXXX"
+			(at 151.13 203.2 90)
+			(hide yes)
+			(show_name no)
+			(do_not_autoplace no)
+			(effects
+				(font
+					(size 1.27 1.27)
+				)
+			)
+		)
 		(pin "1"
 		)
@@
 			)
 		)
-		(property "Value" ""
+		(property "Value" "Light Pipe"
 			(at 175.26 229.87 0)
 			(show_name no)
@@
 			)
 		)
+		(property "JLCPCB P/N" "XXXXXX"
+			(at 175.26 229.87 0)
+			(hide yes)
+			(show_name no)
+			(do_not_autoplace no)
+			(effects
+				(font
+					(size 1.27 1.27)
+				)
+			)
+		)
 		(instances
 			(project "NX-J401-Adapter-v7"
@@
 			(hide yes)
 			(show_name no)
+			(do_not_autoplace no)
+			(effects
+				(font
+					(size 1.27 1.27)
+				)
+			)
+		)
+		(property "JLCPCB P/N" "XXXXXX"
+			(at 133.35 203.2 90)
+			(hide yes)
+			(show_name no)

Commit message: Add mounting holes near Vout and tooling holes
Signed-off-by: Scott Berman <sgberman1@gmail.com>
Parts:
- added H10, H11, H12, H13: 1.152mm ToolingHole, MountingHole:ToolingHole_1.152mm, symbol NX-J401-Adapter:MountingHole
- added H7, H8, H9: MountingHole, NX-J401-Adapter:MountingHole_2.5mm, symbol NX-J401-Adapter:MountingHole

Commit message: Update break away pcb sections
Signed-off-by: Scott Berman <scott.berman@bluerivertech.com>
Parts:
- C1, C12, C45, C54: MFG P/N GRM32ER71H106KA12L -> GRM32ER71H106KA12L
- D1: MFG P/N SMDJ24CA -> SMDJ24CA
Changed lines of the file:
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@@
 			)
 		)
-		(property "MFG P/N" " GRM32ER71H106KA12L"
+		(property "MFG P/N" "GRM32ER71H106KA12L"
 			(at 161.29 63.5 0)
 			(hide yes)
@@
 			)
 		)
-		(property "MFG P/N" " GRM32ER71H106KA12L"
+		(property "MFG P/N" "GRM32ER71H106KA12L"
 			(at 299.72 63.5 0)
 			(hide yes)
@@
 			)
 		)
-		(property "MFG P/N" " GRM32ER71H106KA12L"
+		(property "MFG P/N" "GRM32ER71H106KA12L"
 			(at 257.81 63.5 0)
 			(hide yes)
@@
 			)
 		)
-		(property "MFG P/N" " SMDJ24CA"
+		(property "MFG P/N" "SMDJ24CA"
 			(at 100.33 63.5 0)
 			(show_name no)
@@
 			)
 		)
-		(property "MFG P/N" " GRM32ER71H106KA12L"
+		(property "MFG P/N" "GRM32ER71H106KA12L"
 			(at 118.11 63.5 0)
 			(hide yes)
