File: circuit-boards/NX-J401-Adapter-v7/NX-J401-Adapter-v7.kicad_pcb (KiCad board)
At the start: 4 copper layers, 119.6 x 99.2 mm, 142 parts, among them J1 Terminal, J10 POWER, J11 USB_C_Receptacle_USB2.0_14P, J2 Terminal, J3 NX CONTROL & UART, J4 15V, J5 NX CONTROL & UART, J6 NX CONTROL & UART, J7 USB1, J8 SWD, J9 CAN1, Q1 CSD19534Q5A, Q2 SI2301CDS-T1-GE3, Q3 CSD17578Q5A, Q4 CSD17578Q5A, Q5 SS8050, Q6 CSD19534Q5A, Q7 SI2301CDS-T1-GE3, Q8 CSD19534Q5A, Q9 CSD19534Q5A, SW1 RESET, SW2 RECOVERY, U1 LM74700QDBVRQ1, U2 TPS613222ADBV, U3 STM32G431CBTx, U4 LM5176PWPR, U5 ISO6721BDR, U6 FT232RNL, U7 LM74700QDBVRQ1, U8 TJA1051T/3/1J

Commit message: Update break away pcb sections
Signed-off-by: Scott Berman <scott.berman@bluerivertech.com>
Parts:
- moved H13 18.0 mm to (266.6, 159.8)
- moved H12 18.0 mm to (269.2, 68.2)
- moved LOGO2 9.91 mm to (271.5, 134.7)
Other:
- outline, holes or cut-outs redrawn
- board text added: "BACK"
- board text added: "FRONT"
- board text added: "NOTES: 1. Depanelize using Hakko DP-25-N"
