File: circuit-boards/NX-J401-Adapter-v7/NX-Button-Interface.kicad_sch (KiCad schematic)
At the start: 5 parts, among them J5 NX CONTROL & UART, J6 NX CONTROL & UART

Commit message: Routed PCB
Signed-off-by: scott <scott@scott-Z590I-AORUS-ULTRA.bb>
Parts:
- renumbered H4 to H3, H6 to H4
Changed lines of the file:
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@@
 		(dnp no)
 		(fields_autoplaced yes)
-		(property "Reference" "H4"
+		(property "Reference" "H3"
 			(at 219.71 101.5999 0)
 			(show_name no)
@@
 			(project "NX-J401-Adapter-v7"
 				(path "/3c9fa76f-2b37-4666-8575-58caa65def04/f8ff9f31-2365-4daa-ba47-54bf7f47daed"
-					(reference "H4")
+					(reference "H3")
 					(unit 1)
 				)
@@
 		(dnp no)
 		(fields_autoplaced yes)
-		(property "Reference" "H6"
+		(property "Reference" "H4"
 			(at 219.71 107.9499 0)
 			(show_name no)
@@
 			(project "NX-J401-Adapter-v7"
 				(path "/3c9fa76f-2b37-4666-8575-58caa65def04/f8ff9f31-2365-4daa-ba47-54bf7f47daed"
-					(reference "H6")
+					(reference "H4")
 					(unit 1)
 				)
