File: circuit-boards/NX-J401-Adapter-v7/buck-boost-power-supply.kicad_sch (KiCad schematic)
At the start: 55 parts, among them Q3 CSD19534Q5A, Q4 CSD17578Q5A, Q5 CSD19534Q5A, Q6 CSD17578Q5A

Commit message: Routed PCB
Signed-off-by: scott <scott@scott-Z590I-AORUS-ULTRA.bb>
Parts:
- renumbered C11 to C10, C17 to C14, C27 to C15, C16 to C18, C26 to C19, C28 to C2, C15 to C23, C25 to C24, C52 to C26, C37 to C27, C51 to C28, C35 to C29, C18 to C3, C50 to C31, C49 to C33, C48 to C35, C34 to C36, C33 to C37, C47 to C39, C29 to C4, C32 to C40, C14 to C43, C24 to C44, C13 to C49, C19 to C5, C23 to C50, C43 to C6, C22 to C7, C12 to C8, C21 to C9, D2 to D6, D1 to D7, D4 to D8, L2 to L1, Q6 to Q3, Q3 to Q6, Q5 to Q8, R9 to R13, R5 to R14, R20 to R15, R19 to R16, R18 to R17, R8 to R18, R15 to R19, R17 to R20, R14 to R21, R7 to R22, R23 to R3, R22 to R5, R21 to R6, R13 to R7, R12 to R8, U5 to U4

Commit message: PCB update
Signed-off-by: Scott Berman <sgberman1@gmail.com>
Parts:
- R3: JLCPCB P/N C137697 -> C227834; MFG P/N RC0603FR-075K9L -> AC0603FR-07357KL
- U4: value (none) -> LM5176PWPR
Changed lines of the file:
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@@
 	(title_block
 		(title "NX J401 Adapter")
-		(date "2026-06-02")
-		(rev "6")
+		(date "2026-08-01")
+		(rev "7")
 		(company "SPACE COOKIES FRC TEAM 1868")
 	)
@@
 			)
 		)
-		(property "Value" ""
+		(property "Value" "LM5176PWPR"
 			(at 144.78 148.59 0)
+			(hide yes)
 			(show_name no)
 			(do_not_autoplace no)
@@
 			)
 		)
-		(property "MFG P/N" "RC0603FR-075K9L"
+		(property "MFG P/N" "AC0603FR-07357KL"
 			(at 250.19 140.97 90)
 			(hide yes)
@@
 			)
 		)
-		(property "JLCPCB P/N" "C137697"
+		(property "JLCPCB P/N" "C227834"
 			(at 250.19 140.97 90)
 			(hide yes)

Commit message: Update break away pcb sections
Signed-off-by: Scott Berman <scott.berman@bluerivertech.com>
Parts:
- C10, C14, C15, C18, C19, C2, C23, C24, C3, C4, C43, C44, C49, C5, C50, C6, C7, C8, C9: MFG P/N GRM32ER71H106KA12L -> GRM32ER71H106KA12L
Changed lines of the file:
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@@
 			)
 		)
-		(property "MFG P/N" " GRM32ER71H106KA12L"
+		(property "MFG P/N" "GRM32ER71H106KA12L"
 			(at 313.69 67.31 0)
 			(hide yes)
@@
 			)
 		)
-		(property "MFG P/N" " GRM32ER71H106KA12L"
+		(property "MFG P/N" "GRM32ER71H106KA12L"
 			(at 97.79 67.31 0)
 			(hide yes)
@@
 			)
 		)
-		(property "MFG P/N" " GRM32ER71H106KA12L"
+		(property "MFG P/N" "GRM32ER71H106KA12L"
 			(at 135.89 67.31 0)
 			(hide yes)
@@
 			)
 		)
-		(property "MFG P/N" " GRM32ER71H106KA12L"
+		(property "MFG P/N" "GRM32ER71H106KA12L"
 			(at 120.65 67.31 0)
 			(hide yes)
@@
 			)
 		)
-		(property "MFG P/N" " GRM32ER71H106KA12L"
+		(property "MFG P/N" "GRM32ER71H106KA12L"
 			(at 275.59 67.31 0)
 			(hide yes)
@@
 			)
 		)
-		(property "MFG P/N" " GRM32ER71H106KA12L"
+		(property "MFG P/N" "GRM32ER71H106KA12L"
 			(at 90.17 67.31 0)
 			(hide yes)
@@
 			)
 		)
-		(property "MFG P/N" " GRM32ER71H106KA12L"
+		(property "MFG P/N" "GRM32ER71H106KA12L"
 			(at 267.97 67.31 0)
 			(hide yes)
@@
 			)
 		)
-		(property "MFG P/N" " GRM32ER71H106KA12L"
+		(property "MFG P/N" "GRM32ER71H106KA12L"
 			(at 290.83 67.31 0)
 			(hide yes)
@@
 			)
 		)
-		(property "MFG P/N" " GRM32ER71H106KA12L"
+		(property "MFG P/N" "GRM32ER71H106KA12L"
 			(at 298.45 67.31 0)
 			(hide yes)
@@
 			)
 		)
-		(property "MFG P/N" " GRM32ER71H106KA12L"
+		(property "MFG P/N" "GRM32ER71H106KA12L"
 			(at 128.27 67.31 0)
 			(hide yes)
@@
 			)
 		)
-		(property "MFG P/N" " GRM32ER71H106KA12L"
+		(property "MFG P/N" "GRM32ER71H106KA12L"
 			(at 143.51 67.31 0)
 			(hide yes)
@@
 			)
 		)
-		(property "MFG P/N" " GRM32ER71H106KA12L"
+		(property "MFG P/N" "GRM32ER71H106KA12L"
 			(at 260.35 67.31 0)
 			(hide yes)
@@
 			)
 		)
-		(property "MFG P/N" " GRM32ER71H106KA12L"
+		(property "MFG P/N" "GRM32ER71H106KA12L"
 			(at 306.07 67.31 0)
 			(hide yes)
@@
 			)
 		)
-		(property "MFG P/N" " GRM32ER71H106KA12L"
+		(property "MFG P/N" "GRM32ER71H106KA12L"
 			(at 105.41 67.31 0)
 			(hide yes)
@@
 			)
 		)
-		(property "MFG P/N" " GRM32ER71H106KA12L"
+		(property "MFG P/N" "GRM32ER71H106KA12L"
 			(at 151.13 67.31 0)
 			(hide yes)
@@
 			)
 		)
-		(property "MFG P/N" " GRM32ER71H106KA12L"
+		(property "MFG P/N" "GRM32ER71H106KA12L"
 			(at 283.21 67.31 0)
 			(hide yes)
@@
 			)
 		)
-		(property "MFG P/N" " GRM32ER71H106KA12L"
+		(property "MFG P/N" "GRM32ER71H106KA12L"
 			(at 328.93 67.31 0)
 			(hide yes)
@@
 			)
 		)
-		(property "MFG P/N" " GRM32ER71H106KA12L"
+		(property "MFG P/N" "GRM32ER71H106KA12L"
 			(at 113.03 67.31 0)
 			(hide yes)
@@
 			)
 		)
-		(property "MFG P/N" " GRM32ER71H106KA12L"
+		(property "MFG P/N" "GRM32ER71H106KA12L"
 			(at 321.31 67.31 0)
 			(hide yes)
