File: circuit-boards/NX-J401-Adapter-v7/usb-serial.kicad_sch (KiCad schematic)
At the start: 14 parts, among them J11 USB_C_Receptacle_USB2.0_14P, U7 ISO6721BDR, U8 FT232RNL

Commit message: Routed PCB
Signed-off-by: scott <scott@scott-Z590I-AORUS-ULTRA.bb>
Parts:
- renumbered C39 to C38, C38 to C41, C46 to C42, C53 to C46, C45 to C47, C54 to C51, C56 to C55, C55 to C56, U7 to U5, U8 to U6
Changed lines of the file:
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@@
 		(in_pos_files yes)
 		(dnp no)
-		(property "Reference" "C39"
+		(property "Reference" "C38"
 			(at 325.12 108.2039 0)
 			(show_name no)
@@
 			(project "NX-J401-Adapter-v7"
 				(path "/3c9fa76f-2b37-4666-8575-58caa65def04/7f338915-7b6e-40c1-9733-742b14680646"
-					(reference "C39")
+					(reference "C38")
 					(unit 1)
 				)
@@
 		(in_pos_files yes)
 		(dnp no)
-		(property "Reference" "C53"
+		(property "Reference" "C46"
 			(at 204.47 128.5239 0)
 			(show_name no)
@@
 			(project "NX-J401-Adapter-v7"
 				(path "/3c9fa76f-2b37-4666-8575-58caa65def04/7f338915-7b6e-40c1-9733-742b14680646"
-					(reference "C53")
+					(reference "C46")
 					(unit 1)
 				)
@@
 		(in_pos_files yes)
 		(dnp no)
-		(property "Reference" "C46"
+		(property "Reference" "C42"
 			(at 118.618 131.572 90)
 			(show_name no)
@@
 			(project "NX-J401-Adapter-v7"
 				(path "/3c9fa76f-2b37-4666-8575-58caa65def04/7f338915-7b6e-40c1-9733-742b14680646"
-					(reference "C46")
+					(reference "C42")
 					(unit 1)
 				)
@@
 		(in_pos_files yes)
 		(dnp no)
-		(property "Reference" "C55"
+		(property "Reference" "C56"
 			(at 140.716 189.23 0)
 			(show_name no)
@@
 			(project "NX-J401-Adapter-v7"
 				(path "/3c9fa76f-2b37-4666-8575-58caa65def04/7f338915-7b6e-40c1-9733-742b14680646"
-					(reference "C55")
+					(reference "C56")
 					(unit 1)
 				)
@@
 		(in_pos_files yes)
 		(dnp no)
-		(property "Reference" "C45"
+		(property "Reference" "C47"
 			(at 155.956 130.556 0)
 			(show_name no)
@@
 			(project "NX-J401-Adapter-v7"
 				(path "/3c9fa76f-2b37-4666-8575-58caa65def04/7f338915-7b6e-40c1-9733-742b14680646"
-					(reference "C45")
+					(reference "C47")
 					(unit 1)
 				)
@@
 		(in_pos_files yes)
 		(dnp no)
-		(property "Reference" "C38"
+		(property "Reference" "C41"
 			(at 275.59 95.5039 0)
 			(show_name no)
@@
 			(project "NX-J401-Adapter-v7"
 				(path "/3c9fa76f-2b37-4666-8575-58caa65def04/7f338915-7b6e-40c1-9733-742b14680646"
-					(reference "C38")
+					(reference "C41")
 					(unit 1)
 				)
@@
 		(in_pos_files yes)
 		(dnp no)
-		(property "Reference" "C54"
+		(property "Reference" "C51"
 			(at 205.74 190.7539 0)
 			(show_name no)
@@
 			(project "NX-J401-Adapter-v7"
 				(path "/3c9fa76f-2b37-4666-8575-58caa65def04/7f338915-7b6e-40c1-9733-742b14680646"
-					(reference "C54")
+					(reference "C51")
 					(unit 1)
 				)
@@
 		(in_pos_files yes)
 		(dnp no)
-		(property "Reference" "C56"
+		(property "Reference" "C55"
 			(at 130.556 189.23 0)
 			(show_name no)
@@
 			(project "NX-J401-Adapter-v7"
 				(path "/3c9fa76f-2b37-4666-8575-58caa65def04/7f338915-7b6e-40c1-9733-742b14680646"
-					(reference "C56")
+					(reference "C55")
 					(unit 1)
 				)
@@
 		(dnp no)
 		(fields_autoplaced yes)
-		(property "Reference" "U8"
+		(property "Reference" "U6"
 			(at 242.1733 139.7 0)
 			(show_name no)
@@
 			(project "NX-J401-Adapter-v7"
 				(path "/3c9fa76f-2b37-4666-8575-58caa65def04/7f338915-7b6e-40c1-9733-742b14680646"
-					(reference "U8")
+					(reference "U6")
 					(unit 1)
 				)
@@
 		(dnp no)
 		(fields_autoplaced yes)
-		(property "Reference" "U7"
+		(property "Reference" "U5"
 			(at 293.37 118.11 0)
 			(show_name no)
@@
 			(project "NX-J401-Adapter-v7"
 				(path "/3c9fa76f-2b37-4666-8575-58caa65def04/7f338915-7b6e-40c1-9733-742b14680646"
-					(reference "U7")
-					(unit 1)
-				)
+					(reference "U5")
+					(unit 1)
+				)
