File: circuit-boards/NX-J401-Adapter-v7/_restore_backup_2026-07-26T14-48-17-220/NX-J401-Adapter-v7.kicad_sch (KiCad schematic)
At the start: 32 parts, among them J1 Terminal, J10 POWER, J2 Terminal, J3 NX CONTROL & UART, J4 15V, J7 USB1, J9 CAN1, Q1 CSD19534Q5A, Q9 CSD19534Q5A, SW1 RESET, SW2 RECOVERY, U1 LM74700QDBVRQ1, U7 LM74700QDBVRQ1

Commit message: Removed boot0 switch to clear J401 40 pin header
Signed-off-by: scott <scott@scott-Z590I-AORUS-ULTRA.bb>
Parts:
- renumbered C12 to C11, C11 to C12, SW1 to SW2, SW2 to SW3
Changed lines of the file:
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@@
 		(in_pos_files yes)
 		(dnp no)
-		(property "Reference" "C12"
+		(property "Reference" "C11"
 			(at 301.498 61.468 90)
 			(show_name no)
@@
 			(project "NX-J401-Adapter-v7"
 				(path "/3c9fa76f-2b37-4666-8575-58caa65def04"
-					(reference "C12")
+					(reference "C11")
 					(unit 1)
 				)
@@
 		(in_pos_files yes)
 		(dnp no)
-		(property "Reference" "C11"
+		(property "Reference" "C12"
 			(at 270.764 54.61 90)
 			(show_name no)
@@
 			(project "NX-J401-Adapter-v7"
 				(path "/3c9fa76f-2b37-4666-8575-58caa65def04"
-					(reference "C11")
+					(reference "C12")
 					(unit 1)
 				)
@@
 		(dnp no)
 		(fields_autoplaced yes)
-		(property "Reference" "SW1"
+		(property "Reference" "SW2"
 			(at 154.94 201.93 90)
 			(show_name no)
@@
 			(project "NX-J401-Adapter-v7"
 				(path "/3c9fa76f-2b37-4666-8575-58caa65def04"
-					(reference "SW1")
+					(reference "SW2")
 					(unit 1)
 				)
@@
 		(dnp no)
 		(fields_autoplaced yes)
-		(property "Reference" "SW2"
+		(property "Reference" "SW3"
 			(at 137.16 201.93 90)
 			(show_name no)
@@
 			(project "NX-J401-Adapter-v7"
 				(path "/3c9fa76f-2b37-4666-8575-58caa65def04"
-					(reference "SW2")
+					(reference "SW3")
 					(unit 1)
 				)
