File: circuit-boards/NX-J401-Adapter-v7/_restore_backup_2026-07-26T14-48-17-220/canable2.kicad_sch (KiCad schematic)
At the start: 29 parts, among them J8 SWD, Q2 SI2301CDS-T1-GE3, Q5 SS8050, Q7 SI2301CDS-T1-GE3, U2 TPS613222ADBV, U3 STM32G431CBTx, U8 TJA1051T/3/1J

Commit message: Removed boot0 switch to clear J401 40 pin header
Signed-off-by: scott <scott@scott-Z590I-AORUS-ULTRA.bb>
Parts:
- removed J8: SWD, NX-J401-Adapter:PinHeader_1x05_P2.54mm_Horizontal, symbol NX-J401-Adapter:Conn_01x05
- added J8: SWD, NX-J401-Adapter:PinHeader_1x03_P2.54mm_Horizontal, symbol Connector_Generic:Conn_01x03
- added SW1: CAN BOOT, NX-J401-Adapter:SW_TL1105VF100Q_EWI, symbol NX-J401-Adapter:SW_Push
Connections:
- net 3V3: now also SW1.1
- net BOOT0: now also SW1.2
- net GND_CAN: now also J8.1 (Pin_1)
- net SWCLK: now also J8.3 (Pin_3)
- net SWDIO: now also J8.2 (Pin_2)
Other:
- note removed: "3V3_CAN delays bringing CAN RX (BOOT0) high until NPN turns on. ~10sec."
