File: circuit-boards/TVS-Adapter-v1/TVS-Adapter-v1.kicad_pcb (KiCad board)
At the start: 4 copper layers, 119.6 x 99.2 mm, 160 parts, among them J1 Terminal, J10 POWER, J11 USB_C_Receptacle_USB2.0_14P, J2 Terminal, J3 NX CONTROL & UART, J4 15V, J5 NX CONTROL & UART, J6 NX CONTROL & UART, J7 USB1, J8 SWD, J9 CAN1, Q1 CSD19534Q5A, Q10 SI2301CDS-T1-GE3, Q11 CSD19534Q5A, Q12 CSD19534Q5A, Q13 CSD19534Q5A, Q2 SI2301CDS-T1-GE3, Q3 SS8050, Q4 SI2301CDS-T1-GE3, Q5 CSD17578Q5A, Q6 SS8050, Q7 SI2301CDS-T1-GE3, Q8 CSD17578Q5A, Q9 SS8050, SW1 RESET, SW2 RECOVERY, U1 LM74700QDBVRQ1, U2 TPS613222ADBV, U3 STM32G431CBTx, U4 LM5176PWPR, U5 ISO6741DWR, U6 FT232RNL, U7 LM74700QDBVRQ1, U8 TJA1051T/3/1J

Commit message: Updates from Claude review
Signed-off-by: Scott Berman <scott.berman@bluerivertech.com>
Parts:
- D7: value BAV199LT1G -> BAT54KFILM; footprint Package_TO_SOT_SMD:SOT-23 -> NX-J401-Adapter:D_SOD-523
- turned D7 to 90 degrees
Connections:
- C32 pad 1: Net-(Q9-B) -> Net-(D7-A)
- D7 pad 1: Net-(Q9-B) -> /CANable2.0/3V3
- D7 pad 2: /CANable2.0/3V3 -> Net-(D7-A)
- Q9 pad 1: Net-(Q9-B) -> Net-(D7-A)
- R13 pad 2: Net-(Q9-B) -> Net-(D7-A)
Routing:
- net Net-(D7-A): track 0.00 -> 12.8 mm
- net Net-(Q9-B): track 12.1 -> 0.00 mm
- net /CANable2.0/3V3: track 36.1 -> 34.2 mm
- net /VIN_PS: vias 4 -> 15
- net /V_OUT: vias 0 -> 13
- added copper zone on F.Cu, net /V_OUT
Other:
- board text added: "NOTES: 1. Depanelize using Hakko DP-25-N 2. program CBUS2 and CBUS3 to CBitBangI/O with FT_PROG or ftdi_eeprom before fitting R1/R2, and leave {dblquote}pull down I/O pins in USB suspend{dblquote} off."
- board text removed: "NOTES: 1. Depanelize using Hakko DP-25-N"
