File: circuit-boards/TVS-Adapter-v1/NX-Button-Interface.kicad_sch (KiCad schematic)
At the start: 5 parts, among them J5 NX CONTROL & UART, J6 NX CONTROL & UART

Commit message: Add reset and recovery control from FT232
Signed-off-by: Scott Berman <sgberman1@gmail.com>
Other:
- title: The Vision System Adapter -> TVS Adapter
Changed lines of the file:
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@@
 	(paper "B")
 	(title_block
-		(title "The Vision System Adapter")
-		(date "2026-10-10")
-		(rev "7")
+		(title "TVS Adapter")
+		(date "2026-10-14")
+		(rev "1")
 		(company "SPACE COOKIES FRC TEAM 1868")
 	)

Commit message: Add pullups to reset-recovery outputs
Signed-off-by: Scott Berman <sgberman1@gmail.com>
Other:
- title: TVS Adapter -> The Vision System Adapter
Changed lines of the file:
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@@
 	(paper "B")
 	(title_block
-		(title "TVS Adapter")
+		(title "The Vision System Adapter")
 		(date "2026-10-14")
 		(rev "1")

Commit message: Update with cleaned up silk and fab drawings
Signed-off-by: Scott Berman <sgberman1@gmail.com>
Parts:
- renumbered H3 to H6, H4 to H9
Changed lines of the file:
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@@
 		(dnp no)
 		(fields_autoplaced yes)
-		(property "Reference" "H3"
+		(property "Reference" "H6"
 			(at 219.71 101.5999 0)
 			(show_name no)
@@
 			(project "TVS-Adapter-v1"
 				(path "/3c9fa76f-2b37-4666-8575-58caa65def04/f8ff9f31-2365-4daa-ba47-54bf7f47daed"
-					(reference "H3")
+					(reference "H6")
 					(unit 1)
 				)
@@
 		(dnp no)
 		(fields_autoplaced yes)
-		(property "Reference" "H4"
+		(property "Reference" "H9"
 			(at 219.71 107.9499 0)
 			(show_name no)
@@
 			(project "TVS-Adapter-v1"
 				(path "/3c9fa76f-2b37-4666-8575-58caa65def04/f8ff9f31-2365-4daa-ba47-54bf7f47daed"
-					(reference "H4")
+					(reference "H9")
 					(unit 1)
 				)

Commit message: Fixed most issues from review pass 4
Signed-off-by: scottb <sgberman1@gmail.com>
Connections:
- net 3V3_BTN: now also J5.15 (Pin_15), J6.15 (Pin_15); no longer J5.1 (Pin_1), J6.1 (Pin_1)
- net GND_BTN: now also J5.4 (Pin_4), J5.6 (Pin_6), J6.4 (Pin_4), J6.6 (Pin_6); no longer J5.10 (Pin_10), J5.12 (Pin_12), J6.10 (Pin_10), J6.12 (Pin_12)
- net NX_PC_LED+: now also J5.11 (Pin_11), J6.11 (Pin_11); no longer J5.5 (Pin_5), J6.5 (Pin_5)
- net NX_PC_LED-: now also J5.12 (Pin_12), J6.12 (Pin_12); no longer J5.4 (Pin_4), J6.4 (Pin_4)
- net UART2_RXD: now also J5.10 (Pin_10), J6.10 (Pin_10); no longer J5.6 (Pin_6), J6.6 (Pin_6)
- net UART2_TXD: now also J5.9 (Pin_9), J6.9 (Pin_9); no longer J5.7 (Pin_7), J6.7 (Pin_7)
- net ~{REC}: now also J5.3 (Pin_3), J6.3 (Pin_3); no longer J5.13 (Pin_13), J6.13 (Pin_13)
- net ~{SYS_RESET}: now also J5.5 (Pin_5), J6.5 (Pin_5); no longer J5.11 (Pin_11), J6.11 (Pin_11)
Other:
- moved on the sheet: J5
Changed lines of the file:
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@@
+	)
+	(no_connect
+		(at 132.08 105.41)
+	)
+	(no_connect
+		(at 161.29 135.89)
+	)
+	(no_connect
+		(at 132.08 102.87)
+	)
+	(no_connect
+		(at 132.08 120.65)
+	)
+	(no_connect
+		(at 161.29 133.35)
+	)
+	(no_connect
+		(at 132.08 133.35)
+	)
+	(no_connect
+		(at 161.29 120.65)
+	)
+	(no_connect
+		(at 132.08 118.11)
+	)
+	(no_connect
+		(at 161.29 105.41)
+	)
+	(no_connect
+		(at 132.08 135.89)
+	)
+	(no_connect
+		(at 161.29 118.11)
 	)
 	(no_connect
 		(at 161.29 102.87)
 	)
-	(no_connect
-		(at 132.08 135.89)
-	)
-	(no_connect
-		(at 132.08 118.11)
-	)
-	(no_connect
-		(at 132.08 133.35)
-	)
-	(no_connect
-		(at 161.29 105.41)
-	)
-	(no_connect
-		(at 132.08 120.65)
-	)
-	(no_connect
-		(at 161.29 133.35)
-	)
-	(no_connect
-		(at 161.29 118.11)
-	)
-	(no_connect
-		(at 132.08 102.87)
-	)
-	(no_connect
-		(at 161.29 120.65)
-	)
-	(no_connect
-		(at 161.29 135.89)
-	)
-	(no_connect
-		(at 132.08 105.41)
-	)
 	(wire
 		(pts
@@
 	(wire
 		(pts
+			(xy 132.08 110.49) (xy 161.29 110.49)
+		)
+		(stroke
+			(width 0)
+			(type default)
+		)
+	)
+	(wire
+		(pts
 			(xy 132.08 123.19) (xy 161.29 123.19)
 		)
@@
 	(wire
 		(pts
+			(xy 132.08 128.27) (xy 161.29 128.27)
+		)
+		(stroke
+			(width 0)
+			(type default)
+		)
+	)
+	(wire
+		(pts
 			(xy 132.08 130.81) (xy 161.29 130.81)
 		)
@@
 	(wire
 		(pts
-			(xy 132.08 110.49) (xy 161.29 110.49)
-		)
-		(stroke
-			(width 0)
-			(type default)
-		)
-	)
-	(wire
-		(pts
-			(xy 132.08 128.27) (xy 161.29 128.27)
+			(xy 132.08 107.95) (xy 161.29 107.95)
 		)
 		(stroke
@@
 		(pts
 			(xy 132.08 125.73) (xy 161.29 125.73)
-		)
-		(stroke
-			(width 0)
-			(type default)
-		)
-	)
-	(wire
-		(pts
-			(xy 132.08 107.95) (xy 161.29 107.95)
 		)
 		(stroke
@@
 	(symbol
 		(lib_id "NX-J401-Adapter:Conn_01x15_Socket")
-		(at 127 118.11 0)
-		(mirror y)
+		(at 127 118.11 180)
 		(unit 1)
 		(body_style 1)
@@
 		(in_pos_files yes)
 		(dnp no)
-		(fields_autoplaced yes)
 		(property "Reference" "J5"
-			(at 127.635 95.25 0)
+			(at 128.27 96.52 0)
 			(show_name no)
 			(do_not_autoplace no)
@@
 		)
 		(property "Value" "NX CONTROL & UART"
-			(at 127.635 97.79 0)
+			(at 127 138.43 0)
 			(show_name no)
 			(do_not_autoplace no)
@@
 		(lib_id "NX-J401-Adapter:Conn_01x15_Socket")
 		(at 166.37 118.11 0)
+		(mirror x)
 		(unit 1)
 		(body_style 1)
@@
 		(dnp no)
 		(property "Reference" "J6"
-			(at 165.735 95.25 0)
+			(at 166.37 96.52 0)
 			(show_name no)
 			(do_not_autoplace no)
@@
 		)
 		(property "Value" "NX CONTROL & UART"
-			(at 165.735 97.79 0)
-			(show_name no)
-			(do_not_autoplace no)
+			(at 166.37 138.43 0)
+			(show_name no)
+			(do_not_autoplace no)
