File: circuit-boards/TVS-Adapter-v1/TVS-Adapter-v1.kicad_sch (KiCad schematic)
At the start: 41 parts, among them J1 Terminal, J10 POWER, J2 Terminal, J3 NX CONTROL & UART, J4 15V, J7 USB1, J9 CAN1, Q1 CSD19534Q5A, Q9 CSD19534Q5A, SW1 RESET, SW2 RECOVERY, U1 LM74700QDBVRQ1, U7 LM74700QDBVRQ1

Commit message: Add reset and recovery control.  PCB incomplete WIP
Signed-off-by: scott <scott@scott-Z590I-AORUS-ULTRA.bb>
Other:
- sheet USB Serial ports: added ~{FORCE_RECOVERY}, ~{RESET}; removed none
Changed lines of the file:
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@@
 	)
 	(junction
+		(at 151.13 187.96)
+		(diameter 0)
+		(color 0 0 0 0)
+	)
+	(junction
+		(at 133.35 190.5)
+		(diameter 0)
+		(color 0 0 0 0)
+	)
+	(junction
 		(at 166.37 45.72)
 		(diameter 0)
@@
 	(wire
 		(pts
+			(xy 133.35 190.5) (xy 180.34 190.5)
+		)
+		(stroke
+			(width 0)
+			(type default)
+		)
+	)
+	(wire
+		(pts
 			(xy 99.06 195.58) (xy 93.98 195.58)
 		)
@@
 	(wire
 		(pts
+			(xy 151.13 187.96) (xy 180.34 187.96)
+		)
+		(stroke
+			(width 0)
+			(type default)
+		)
+	)
+	(wire
+		(pts
 			(xy 299.72 45.72) (xy 299.72 59.69)
 		)
@@
 	(sheet
 		(at 180.34 175.26)
-		(size 68.58 16.51)
+		(size 68.58 19.05)
 		(exclude_from_sim no)
 		(in_bom yes)
@@
 			(effects
 				(font
+					(size 1.27 1.27)
+				)
+				(justify left)
+			)
+		)
+		(pin "~{FORCE_RECOVERY}" output
+			(at 180.34 190.5 180)
+			(effects
+				(font
+					(size 1.27 1.27)
+				)
+				(justify left)
+			)
+		)
+		(pin "~{RESET}" output
+			(at 180.34 187.96 180)
+			(effects
+				(font

Commit message: Add reset and recovery control from FT232
Signed-off-by: Scott Berman <sgberman1@gmail.com>
Other:
- title: The Vision System Adapter -> TVS Adapter
Changed lines of the file:
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@@
 	(paper "B")
 	(title_block
-		(title "The Vision System Adapter")
-		(date "2026-10-10")
-		(rev "7")
+		(title "TVS Adapter")
+		(date "2026-10-14")
+		(rev "1")
 		(company "SPACE COOKIES FRC TEAM 1868")
 	)

Commit message: Add pullups to reset-recovery outputs
Signed-off-by: Scott Berman <sgberman1@gmail.com>
Other:
- title: TVS Adapter -> The Vision System Adapter
Changed lines of the file:
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@@
 	(paper "B")
 	(title_block
-		(title "TVS Adapter")
+		(title "The Vision System Adapter")
 		(date "2026-10-14")
 		(rev "1")

Commit message: Update with cleaned up silk and fab drawings
Signed-off-by: Scott Berman <sgberman1@gmail.com>
Parts:
- renumbered C11 to C13, C12 to C14, C45 to C47, C52 to C55, C54 to C57, H10 to H1, H5 to H10, H6 to H11, H11 to H12, H12 to H2, H1 to H3, H2 to H4, H7 to H5, H8 to H7, H9 to H8, Q9 to Q13, R26 to R23, R28 to R26, R27 to R28
Changed lines of the file:
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@@
 		(in_pos_files yes)
 		(dnp no)
-		(property "Reference" "R28"
+		(property "Reference" "R26"
 			(at 157.48 59.182 90)
 			(show_name no)
@@
 			(project "TVS-Adapter-v1"
 				(path "/3c9fa76f-2b37-4666-8575-58caa65def04"
-					(reference "R28")
+					(reference "R26")
 					(unit 1)
 				)
@@
 		(dnp no)
 		(fields_autoplaced yes)
-		(property "Reference" "H6"
+		(property "Reference" "H11"
 			(at 298.45 181.6099 0)
 			(show_name no)
@@
 			(project "TVS-Adapter-v1"
 				(path "/3c9fa76f-2b37-4666-8575-58caa65def04"
-					(reference "H6")
+					(reference "H11")
 					(unit 1)
 				)
@@
 		(dnp no)
 		(fields_autoplaced yes)
-		(property "Reference" "H12"
+		(property "Reference" "H2"
 			(at 350.52 185.4199 0)
 			(show_name no)
@@
 			(project "TVS-Adapter-v1"
 				(path "/3c9fa76f-2b37-4666-8575-58caa65def04"
-					(reference "H12")
+					(reference "H2")
 					(unit 1)
 				)
@@
 		(in_pos_files yes)
 		(dnp no)
-		(property "Reference" "C45"
+		(property "Reference" "C47"
 			(at 152.908 61.468 90)
 			(show_name no)
@@
 			(project "TVS-Adapter-v1"
 				(path "/3c9fa76f-2b37-4666-8575-58caa65def04"
-					(reference "C45")
+					(reference "C47")
 					(unit 1)
 				)
@@
 		(dnp no)
 		(fields_autoplaced yes)
-		(property "Reference" "H10"
+		(property "Reference" "H1"
 			(at 350.52 172.7199 0)
 			(show_name no)
@@
 			(project "TVS-Adapter-v1"
 				(path "/3c9fa76f-2b37-4666-8575-58caa65def04"
-					(reference "H10")
+					(reference "H1")
 					(unit 1)
 				)
@@
 		(dnp no)
 		(fields_autoplaced yes)
-		(property "Reference" "H2"
+		(property "Reference" "H4"
 			(at 298.45 186.6899 0)
 			(show_name no)
@@
 			(project "TVS-Adapter-v1"
 				(path "/3c9fa76f-2b37-4666-8575-58caa65def04"
-					(reference "H2")
+					(reference "H4")
 					(unit 1)
 				)
@@
 		(in_pos_files yes)
 		(dnp no)
-		(property "Reference" "C12"
+		(property "Reference" "C14"
 			(at 301.498 61.468 90)
 			(show_name no)
@@
 			(project "TVS-Adapter-v1"
 				(path "/3c9fa76f-2b37-4666-8575-58caa65def04"
-					(reference "C12")
+					(reference "C14")
 					(unit 1)
 				)
@@
 		(in_pos_files yes)
 		(dnp no)
-		(property "Reference" "Q9"
+		(property "Reference" "Q13"
 			(at 133.35 39.37 90)
 			(show_name no)
@@
 			(project "TVS-Adapter-v1"
 				(path "/3c9fa76f-2b37-4666-8575-58caa65def04"
-					(reference "Q9")
+					(reference "Q13")
 					(unit 1)
 				)
@@
 		(in_pos_files yes)
 		(dnp no)
-		(property "Reference" "C11"
+		(property "Reference" "C13"
 			(at 270.764 54.61 90)
 			(show_name no)
@@
 			(project "TVS-Adapter-v1"
 				(path "/3c9fa76f-2b37-4666-8575-58caa65def04"
-					(reference "C11")
+					(reference "C13")
 					(unit 1)
 				)
@@
 		(in_pos_files yes)
 		(dnp no)
-		(property "Reference" "R27"
+		(property "Reference" "R28"
 			(at 165.1 59.182 90)
 			(show_name no)
@@
 			(project "TVS-Adapter-v1"
 				(path "/3c9fa76f-2b37-4666-8575-58caa65def04"
-					(reference "R27")
+					(reference "R28")
 					(unit 1)
 				)
@@
 		(dnp no)
 		(fields_autoplaced yes)
-		(property "Reference" "H8"
+		(property "Reference" "H7"
 			(at 298.45 203.1999 0)
 			(show_name no)
@@
 			(project "TVS-Adapter-v1"
 				(path "/3c9fa76f-2b37-4666-8575-58caa65def04"
-					(reference "H8")
+					(reference "H7")
 					(unit 1)
 				)
@@
 		(dnp no)
 		(fields_autoplaced yes)
-		(property "Reference" "H5"
+		(property "Reference" "H10"
 			(at 298.45 176.5299 0)
 			(show_name no)
@@
 			(project "TVS-Adapter-v1"
 				(path "/3c9fa76f-2b37-4666-8575-58caa65def04"
-					(reference "H5")
+					(reference "H10")
 					(unit 1)
 				)
@@
 		(dnp no)
 		(fields_autoplaced yes)
-		(property "Reference" "H7"
+		(property "Reference" "H5"
 			(at 298.45 198.1199 0)
 			(show_name no)
@@
 			(project "TVS-Adapter-v1"
 				(path "/3c9fa76f-2b37-4666-8575-58caa65def04"
-					(reference "H7")
+					(reference "H5")
 					(unit 1)
 				)
@@
 		(in_pos_files yes)
 		(dnp no)
-		(property "Reference" "C52"
+		(property "Reference" "C55"
 			(at 122.174 54.61 90)
 			(show_name no)
@@
 			(project "TVS-Adapter-v1"
 				(path "/3c9fa76f-2b37-4666-8575-58caa65def04"
-					(reference "C52")
+					(reference "C55")
 					(unit 1)
 				)
@@
 		(dnp no)
 		(fields_autoplaced yes)
-		(property "Reference" "H11"
+		(property "Reference" "H12"
 			(at 350.52 179.0699 0)
 			(show_name no)
@@
 			(project "TVS-Adapter-v1"
 				(path "/3c9fa76f-2b37-4666-8575-58caa65def04"
-					(reference "H11")
+					(reference "H12")
 					(unit 1)
 				)
@@
 		(dnp no)
 		(fields_autoplaced yes)
-		(property "Reference" "H1"
+		(property "Reference" "H3"
 			(at 298.45 171.4499 0)
 			(show_name no)
@@
 			(project "TVS-Adapter-v1"
 				(path "/3c9fa76f-2b37-4666-8575-58caa65def04"
-					(reference "H1")
+					(reference "H3")
 					(unit 1)
 				)
@@
 		(in_pos_files yes)
 		(dnp no)
-		(property "Reference" "R26"
+		(property "Reference" "R23"
 			(at 171.45 59.182 90)
 			(show_name no)
@@
 			(project "TVS-Adapter-v1"
 				(path "/3c9fa76f-2b37-4666-8575-58caa65def04"
-					(reference "R26")
+					(reference "R23")
 					(unit 1)
 				)
@@
 		(dnp no)
 		(fields_autoplaced yes)
-		(property "Reference" "H9"
+		(property "Reference" "H8"
 			(at 298.45 208.2799 0)
 			(show_name no)
@@
 			(project "TVS-Adapter-v1"
 				(path "/3c9fa76f-2b37-4666-8575-58caa65def04"
-					(reference "H9")
+					(reference "H8")
 					(unit 1)
 				)
@@
 		(in_pos_files yes)
 		(dnp no)
-		(property "Reference" "C54"
+		(property "Reference" "C57"
 			(at 109.728 61.468 90)
 			(show_name no)
@@
 			(project "TVS-Adapter-v1"
 				(path "/3c9fa76f-2b37-4666-8575-58caa65def04"
-					(reference "C54")
+					(reference "C57")
 					(unit 1)
 				)

Commit message: Updating open collector output circuit of USB console, flash controller
Signed-off-by: Scott Berman <sgberman1@gmail.com>
Parts:
- renumbered C47 to C48, R23 to R25, R26 to R28, R28 to R30
Changed lines of the file:
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@@
 	(title_block
 		(title "The Vision System Adapter")
-		(date "2026-10-14")
+		(date "2026-10-17")
 		(rev "1")
 		(company "SPACE COOKIES FRC TEAM 1868")
@@
 		(in_pos_files yes)
 		(dnp no)
-		(property "Reference" "R26"
+		(property "Reference" "R28"
 			(at 157.48 59.182 90)
 			(show_name no)
@@
 			(project "TVS-Adapter-v1"
 				(path "/3c9fa76f-2b37-4666-8575-58caa65def04"
-					(reference "R26")
+					(reference "R28")
 					(unit 1)
 				)
@@
 		(in_pos_files yes)
 		(dnp no)
-		(property "Reference" "C47"
+		(property "Reference" "C48"
 			(at 152.908 61.468 90)
 			(show_name no)
@@
 			(project "TVS-Adapter-v1"
 				(path "/3c9fa76f-2b37-4666-8575-58caa65def04"
-					(reference "C47")
+					(reference "C48")
 					(unit 1)
 				)
@@
 		(in_pos_files yes)
 		(dnp no)
-		(property "Reference" "R28"
+		(property "Reference" "R30"
 			(at 165.1 59.182 90)
 			(show_name no)
@@
 			(project "TVS-Adapter-v1"
 				(path "/3c9fa76f-2b37-4666-8575-58caa65def04"
-					(reference "R28")
+					(reference "R30")
 					(unit 1)
 				)
@@
 		(in_pos_files yes)
 		(dnp no)
-		(property "Reference" "R23"
+		(property "Reference" "R25"
 			(at 171.45 59.182 90)
 			(show_name no)
@@
 			(project "TVS-Adapter-v1"
 				(path "/3c9fa76f-2b37-4666-8575-58caa65def04"
-					(reference "R23")
+					(reference "R25")
 					(unit 1)
 				)

Commit message: Fixed most issues from review pass 4
Signed-off-by: scottb <sgberman1@gmail.com>
Parts:
- J3: MFG Molex -> Adam Tech
Connections:
- net 3V3_BTN: now also J3.15 (Pin_15); no longer J3.1 (Pin_1)
- net GND1: now also J3.4 (Pin_4), J3.6 (Pin_6); no longer J3.10 (Pin_10), J3.12 (Pin_12)
- net NX_PC_LED-: now also J3.12 (Pin_12); no longer J3.4 (Pin_4)
- net UART2_RXD: now also J3.10 (Pin_10); no longer J3.6 (Pin_6)
- net UART2_TXD: now also J3.9 (Pin_9); no longer J3.7 (Pin_7)
- net ~{REC}: now also J3.3 (Pin_3); no longer J3.13 (Pin_13)
- net ~{SYS_RESET}: now also J3.5 (Pin_5); no longer J3.11 (Pin_11)
- net NX_PC_LED+ renamed VDD_5V_SYS
- net VDD_5V_SYS: now also J3.11 (Pin_11); no longer J3.5 (Pin_5)
Other:
- sheet USB Serial ports: added +5V J401, 3V3 J401; removed 3V3
