File: circuit-boards/TVS-Adapter-v1/buck-boost-power-supply.kicad_sch (KiCad schematic)
At the start: 57 parts, among them Q3 CSD17578Q5A, Q4 CSD17578Q5A, Q6 CSD19534Q5A, Q8 CSD19534Q5A, U4 LM5176PWPR

Commit message: Add reset and recovery control from FT232
Signed-off-by: Scott Berman <sgberman1@gmail.com>
Other:
- title: The Vision System Adapter -> TVS Adapter
Changed lines of the file:
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@@
 	(paper "B")
 	(title_block
-		(title "The Vision System Adapter")
-		(date "2026-10-10")
-		(rev "7")
+		(title "TVS Adapter")
+		(date "2026-10-14")
+		(rev "1")
 		(company "SPACE COOKIES FRC TEAM 1868")
 	)

Commit message: Add pullups to reset-recovery outputs
Signed-off-by: Scott Berman <sgberman1@gmail.com>
Other:
- title: TVS Adapter -> The Vision System Adapter
Changed lines of the file:
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@@
 	(paper "B")
 	(title_block
-		(title "TVS Adapter")
+		(title "The Vision System Adapter")
 		(date "2026-10-14")
 		(rev "1")

Commit message: Update with cleaned up silk and fab drawings
Signed-off-by: Scott Berman <sgberman1@gmail.com>
Parts:
- renumbered C9 to C10, C10 to C11, C58 to C12, C14 to C16, C15 to C17, C18 to C20, C19 to C21, C23 to C25, C24 to C26, C26 to C28, C27 to C29, C28 to C30, C29 to C31, C31 to C33, C33 to C35, C35 to C37, C36 to C39, C37 to C40, C39 to C41, C40 to C42, C43 to C45, C44 to C46, C49 to C52, C50 to C53, C7 to C6, C8 to C7, C59 to C8, C6 to C9, D7 to D8, D8 to D9, Q6 to Q11, Q8 to Q12, Q3 to Q5, Q4 to Q8, R8 to R10, R10 to R14, R13 to R17, R14 to R18, R15 to R19, R16 to R20, R17 to R21, R18 to R22, R19 to R24, R20 to R25, R21 to R27, R22 to R29, R3 to R5, R5 to R7, R6 to R8, R7 to R9

Commit message: Updating open collector output circuit of USB console, flash controller
Signed-off-by: Scott Berman <sgberman1@gmail.com>
Parts:
- C12, C8: JLCPCB P/N XXXXX -> XXXXXX
- renumbered C45 to C46, C46 to C47, R8 to R10, R9 to R11, R10 to R12, R14 to R16, R17 to R19, R18 to R20, R19 to R21, R20 to R22, R21 to R23, R22 to R24, R24 to R26, R25 to R27, R27 to R29, R29 to R31, R7 to R9
Changed lines of the file:
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@@
 	(title_block
 		(title "The Vision System Adapter")
-		(date "2026-10-14")
+		(date "2026-10-17")
 		(rev "1")
 		(company "SPACE COOKIES FRC TEAM 1868")
@@
 		(dnp no)
 		(fields_autoplaced yes)
-		(property "Reference" "R18"
+		(property "Reference" "R20"
 			(at 205.74 93.9799 0)
 			(show_name no)
@@
 			(project "TVS-Adapter-v1"
 				(path "/3c9fa76f-2b37-4666-8575-58caa65def04/048331f9-005d-457c-bfd7-5224f9f99d07"
-					(reference "R18")
+					(reference "R20")
 					(unit 1)
 				)
@@
 		(in_pos_files yes)
 		(dnp no)
-		(property "Reference" "R10"
+		(property "Reference" "R12"
 			(at 113.284 216.154 90)
 			(show_name no)
@@
 			(project "TVS-Adapter-v1"
 				(path "/3c9fa76f-2b37-4666-8575-58caa65def04/048331f9-005d-457c-bfd7-5224f9f99d07"
-					(reference "R10")
+					(reference "R12")
 					(unit 1)
 				)
@@
 			)
 		)
-		(property "JLCPCB P/N" "XXXXX"
+		(property "JLCPCB P/N" "XXXXXX"
 			(at 48.26 67.31 0)
 			(hide yes)
@@
 		(in_pos_files yes)
 		(dnp no)
-		(property "Reference" "R22"
+		(property "Reference" "R24"
 			(at 171.45 168.91 90)
 			(show_name no)
@@
 			(project "TVS-Adapter-v1"
 				(path "/3c9fa76f-2b37-4666-8575-58caa65def04/048331f9-005d-457c-bfd7-5224f9f99d07"
-					(reference "R22")
+					(reference "R24")
 					(unit 1)
 				)
@@
 		(in_pos_files yes)
 		(dnp no)
-		(property "Reference" "R19"
+		(property "Reference" "R21"
 			(at 88.138 199.39 0)
 			(show_name no)
@@
 			(project "TVS-Adapter-v1"
 				(path "/3c9fa76f-2b37-4666-8575-58caa65def04/048331f9-005d-457c-bfd7-5224f9f99d07"
-					(reference "R19")
+					(reference "R21")
 					(unit 1)
 				)
@@
 		(in_pos_files yes)
 		(dnp no)
-		(property "Reference" "R9"
+		(property "Reference" "R11"
 			(at 120.142 215.9 90)
 			(show_name no)
@@
 			(project "TVS-Adapter-v1"
 				(path "/3c9fa76f-2b37-4666-8575-58caa65def04/048331f9-005d-457c-bfd7-5224f9f99d07"
-					(reference "R9")
+					(reference "R11")
 					(unit 1)
 				)
@@
 		(in_pos_files yes)
 		(dnp no)
-		(property "Reference" "R24"
+		(property "Reference" "R26"
 			(at 74.168 157.48 0)
 			(show_name no)
@@
 			(project "TVS-Adapter-v1"
 				(path "/3c9fa76f-2b37-4666-8575-58caa65def04/048331f9-005d-457c-bfd7-5224f9f99d07"
-					(reference "R24")
+					(reference "R26")
 					(unit 1)
 				)
@@
 		(in_pos_files yes)
 		(dnp no)
-		(property "Reference" "R8"
+		(property "Reference" "R10"
 			(at 51.308 201.93 0)
 			(show_name no)
@@
 			(project "TVS-Adapter-v1"
 				(path "/3c9fa76f-2b37-4666-8575-58caa65def04/048331f9-005d-457c-bfd7-5224f9f99d07"
-					(reference "R8")
+					(reference "R10")
 					(unit 1)
 				)
@@
 		(in_pos_files yes)
 		(dnp no)
-		(property "Reference" "R21"
+		(property "Reference" "R23"
 			(at 85.598 137.414 0)
 			(show_name no)
@@
 			(project "TVS-Adapter-v1"
 				(path "/3c9fa76f-2b37-4666-8575-58caa65def04/048331f9-005d-457c-bfd7-5224f9f99d07"
-					(reference "R21")
+					(reference "R23")
 					(unit 1)
 				)
@@
 		(in_pos_files yes)
 		(dnp no)
-		(property "Reference" "C46"
+		(property "Reference" "C47"
 			(at 91.948 65.278 90)
 			(show_name no)
@@
 			(project "TVS-Adapter-v1"
 				(path "/3c9fa76f-2b37-4666-8575-58caa65def04/048331f9-005d-457c-bfd7-5224f9f99d07"
-					(reference "C46")
+					(reference "C47")
 					(unit 1)
 				)
@@
 		(in_pos_files yes)
 		(dnp no)
-		(property "Reference" "C45"
+		(property "Reference" "C46"
 			(at 130.048 65.278 90)
 			(show_name no)
@@
 			(project "TVS-Adapter-v1"
 				(path "/3c9fa76f-2b37-4666-8575-58caa65def04/048331f9-005d-457c-bfd7-5224f9f99d07"
-					(reference "C45")
+					(reference "C46")
 					(unit 1)
 				)
@@
 		(in_pos_files yes)
 		(dnp no)
-		(property "Reference" "R14"
+		(property "Reference" "R16"
 			(at 171.45 177.8 90)
 			(show_name no)
@@
 			(project "TVS-Adapter-v1"
 				(path "/3c9fa76f-2b37-4666-8575-58caa65def04/048331f9-005d-457c-bfd7-5224f9f99d07"
-					(reference "R14")
+					(reference "R16")
 					(unit 1)
 				)
@@
 		(in_pos_files yes)
 		(dnp no)
-		(property "Reference" "R17"
+		(property "Reference" "R19"
 			(at 171.45 189.23 90)
 			(show_name no)
@@
 			(project "TVS-Adapter-v1"
 				(path "/3c9fa76f-2b37-4666-8575-58caa65def04/048331f9-005d-457c-bfd7-5224f9f99d07"
-					(reference "R17")
+					(reference "R19")
 					(unit 1)
 				)
@@
 		(in_pos_files yes)
 		(dnp no)
-		(property "Reference" "R25"
+		(property "Reference" "R27"
 			(at 113.538 137.414 0)
 			(show_name no)
@@
 			(project "TVS-Adapter-v1"
 				(path "/3c9fa76f-2b37-4666-8575-58caa65def04/048331f9-005d-457c-bfd7-5224f9f99d07"
-					(reference "R25")
+					(reference "R27")
 					(unit 1)
 				)
@@
 		(in_pos_files yes)
 		(dnp no)
-		(property "Reference" "R27"
+		(property "Reference" "R29"
 			(at 74.168 139.7 0)
 			(show_name no)
@@
 			(project "TVS-Adapter-v1"
 				(path "/3c9fa76f-2b37-4666-8575-58caa65def04/048331f9-005d-457c-bfd7-5224f9f99d07"
-					(reference "R27")
+					(reference "R29")
 					(unit 1)
 				)
@@
 		(in_pos_files yes)
 		(dnp no)
-		(property "Reference" "R29"
+		(property "Reference" "R31"
 			(at 171.45 157.48 90)
 			(show_name no)
@@
 			(project "TVS-Adapter-v1"
 				(path "/3c9fa76f-2b37-4666-8575-58caa65def04/048331f9-005d-457c-bfd7-5224f9f99d07"
-					(reference "R29")
+					(reference "R31")
 					(unit 1)
 				)
@@
 		(in_pos_files yes)
 		(dnp no)
-		(property "Reference" "R20"
+		(property "Reference" "R22"
 			(at 77.978 199.39 0)
 			(show_name no)
@@
 			(project "TVS-Adapter-v1"
 				(path "/3c9fa76f-2b37-4666-8575-58caa65def04/048331f9-005d-457c-bfd7-5224f9f99d07"
-					(reference "R20")
+					(reference "R22")
 					(unit 1)
 				)
@@
 			)
 		)
-		(property "JLCPCB P/N" "XXXXX"
+		(property "JLCPCB P/N" "XXXXXX"
 			(at 57.15 67.31 0)
 			(hide yes)
@@
 		(in_pos_files yes)
 		(dnp no)
-		(property "Reference" "R7"
+		(property "Reference" "R9"
 			(at 251.968 152.4 0)
 			(show_name no)
@@
 			(project "TVS-Adapter-v1"
 				(path "/3c9fa76f-2b37-4666-8575-58caa65def04/048331f9-005d-457c-bfd7-5224f9f99d07"
-					(reference "R7")
+					(reference "R9")
 					(unit 1)
 				)

Commit message: Fixed most issues from review pass 4
Signed-off-by: scottb <sgberman1@gmail.com>
Parts:
- R22: value 205K-1%-0603 -> 93.1k-1%-0603; JLCPCB P/N C22949 -> C228101; MFG P/N 0603WAF2053T5E -> AC0603FR-0793K1L
Changed lines of the file:
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@@
 			)
 		)
-		(column_widths 12.7 11.43)
+		(column_widths 12.7 21.59)
 		(row_heights 2.54 2.54 2.54 2.54 2.54 2.54)
 		(cells
@@
 				(exclude_from_sim no)
 				(at 147.32 222.25 0)
-				(size 11.43 2.54)
+				(size 21.59 2.54)
 				(margins 0.9525 0.9525 0.9525 0.9525)
 				(span 1 1)
@@
 				)
 			)
-			(table_cell "5V"
+			(table_cell "6V / 5V Transient"
 				(exclude_from_sim no)
 				(at 147.32 224.79 0)
-				(size 11.43 2.54)
+				(size 21.59 2.54)
 				(margins 0.9525 0.9525 0.9525 0.9525)
 				(span 1 1)
@@
 				(exclude_from_sim no)
 				(at 147.32 227.33 0)
-				(size 11.43 2.54)
+				(size 21.59 2.54)
 				(margins 0.9525 0.9525 0.9525 0.9525)
 				(span 1 1)
@@
 				(exclude_from_sim no)
 				(at 147.32 229.87 0)
-				(size 11.43 2.54)
+				(size 21.59 2.54)
 				(margins 0.9525 0.9525 0.9525 0.9525)
 				(span 1 1)
@@
 				(exclude_from_sim no)
 				(at 147.32 232.41 0)
-				(size 11.43 2.54)
+				(size 21.59 2.54)
 				(margins 0.9525 0.9525 0.9525 0.9525)
 				(span 1 1)
@@
 				(exclude_from_sim no)
 				(at 147.32 234.95 0)
-				(size 11.43 2.54)
+				(size 21.59 2.54)
 				(margins 0.9525 0.9525 0.9525 0.9525)
 				(span 1 1)
@@
 			)
 		)
-		(property "Value" "205K-1%-0603"
+		(property "Value" "93.1k-1%-0603"
 			(at 73.152 199.39 90)
 			(show_name no)
@@
 			)
 		)
-		(property "MFG P/N" "0603WAF2053T5E"
+		(property "MFG P/N" "AC0603FR-0793K1L"
 			(at 76.2 199.39 90)
 			(hide yes)
@@
 			)
 		)
-		(property "JLCPCB P/N" "C22949"
+		(property "JLCPCB P/N" "C228101"
 			(at 76.2 199.39 90)
 			(hide yes)
