File: circuit-boards/TVS-Adapter-v1/canable2.kicad_sch (KiCad schematic)
At the start: 30 parts, among them J8 SWD, Q2 SI2301CDS-T1-GE3, Q5 SS8050, Q7 SI2301CDS-T1-GE3, U2 TPS613222ADBV, U3 STM32G431CBTx, U8 TJA1051T/3/1J

Commit message: Add reset and recovery control from FT232
Signed-off-by: Scott Berman <sgberman1@gmail.com>
Other:
- title: The Vision System Adapter -> TVS Adapter
Changed lines of the file:
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@@
 	(paper "B")
 	(title_block
-		(title "The Vision System Adapter")
-		(date "2026-10-10")
-		(rev "7")
+		(title "TVS Adapter")
+		(date "2026-10-14")
+		(rev "1")
 		(company "SPACE COOKIES FRC TEAM 1868")
 	)

Commit message: Add pullups to reset-recovery outputs
Signed-off-by: Scott Berman <sgberman1@gmail.com>
Other:
- title: TVS Adapter -> The Vision System Adapter
Changed lines of the file:
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@@
 	(paper "B")
 	(title_block
-		(title "TVS Adapter")
+		(title "The Vision System Adapter")
 		(date "2026-10-14")
 		(rev "1")

Commit message: Update with cleaned up silk and fab drawings
Signed-off-by: Scott Berman <sgberman1@gmail.com>
Parts:
- renumbered C13 to C15, C16 to C18, C17 to C19, C20 to C22, C21 to C23, C22 to C24, C25 to C27, C30 to C32, C32 to C34, C34 to C36, C48 to C50, C53 to C56, D9 to D10, D10 to D7, Q7 to Q10, Q5 to Q9, R9 to R11, R11 to R15, R12 to R16, R1 to R3, R2 to R4, R4 to R6
Changed lines of the file:
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@@
 		(in_pos_files yes)
 		(dnp no)
-		(property "Reference" "Q7"
+		(property "Reference" "Q10"
 			(at 246.38 26.67 90)
 			(show_name no)
@@
 			(project "TVS-Adapter-v1"
 				(path "/3c9fa76f-2b37-4666-8575-58caa65def04/958ef65b-dc3d-4755-b7b0-3d4dc8feed9f"
-					(reference "Q7")
+					(reference "Q10")
 					(unit 1)
 				)
@@
 		(in_pos_files yes)
 		(dnp no)
-		(property "Reference" "C13"
+		(property "Reference" "C15"
 			(at 96.266 50.546 0)
 			(show_name no)
@@
 			(project "TVS-Adapter-v1"
 				(path "/3c9fa76f-2b37-4666-8575-58caa65def04/958ef65b-dc3d-4755-b7b0-3d4dc8feed9f"
-					(reference "C13")
+					(reference "C15")
 					(unit 1)
 				)
@@
 		(in_pos_files yes)
 		(dnp no)
-		(property "Reference" "R1"
+		(property "Reference" "R3"
 			(at 228.6 195.58 90)
 			(show_name no)
@@
 			(project "TVS-Adapter-v1"
 				(path "/3c9fa76f-2b37-4666-8575-58caa65def04/958ef65b-dc3d-4755-b7b0-3d4dc8feed9f"
-					(reference "R1")
+					(reference "R3")
 					(unit 1)
 				)
@@
 		(in_pos_files yes)
 		(dnp no)
-		(property "Reference" "C20"
+		(property "Reference" "C22"
 			(at 128.27 214.63 90)
 			(show_name no)
@@
 			(project "TVS-Adapter-v1"
 				(path "/3c9fa76f-2b37-4666-8575-58caa65def04/958ef65b-dc3d-4755-b7b0-3d4dc8feed9f"
-					(reference "C20")
+					(reference "C22")
 					(unit 1)
 				)
@@
 		(in_pos_files yes)
 		(dnp no)
-		(property "Reference" "R4"
+		(property "Reference" "R6"
 			(at 168.148 93.98 0)
 			(show_name no)
@@
 			(project "TVS-Adapter-v1"
 				(path "/3c9fa76f-2b37-4666-8575-58caa65def04/958ef65b-dc3d-4755-b7b0-3d4dc8feed9f"
-					(reference "R4")
+					(reference "R6")
 					(unit 1)
 				)
@@
 		(in_pos_files yes)
 		(dnp no)
-		(property "Reference" "C32"
+		(property "Reference" "C34"
 			(at 158.75 214.63 90)
 			(show_name no)
@@
 			(project "TVS-Adapter-v1"
 				(path "/3c9fa76f-2b37-4666-8575-58caa65def04/958ef65b-dc3d-4755-b7b0-3d4dc8feed9f"
-					(reference "C32")
+					(reference "C34")
 					(unit 1)
 				)
@@
 		(dnp no)
 		(fields_autoplaced yes)
-		(property "Reference" "Q5"
+		(property "Reference" "Q9"
 			(at 248.92 52.0699 0)
 			(show_name no)
@@
 			(project "TVS-Adapter-v1"
 				(path "/3c9fa76f-2b37-4666-8575-58caa65def04/958ef65b-dc3d-4755-b7b0-3d4dc8feed9f"
-					(reference "Q5")
+					(reference "Q9")
 					(unit 1)
 				)
@@
 		(in_pos_files yes)
 		(dnp no)
-		(property "Reference" "C22"
+		(property "Reference" "C24"
 			(at 118.11 214.63 90)
 			(show_name no)
@@
 			(project "TVS-Adapter-v1"
 				(path "/3c9fa76f-2b37-4666-8575-58caa65def04/958ef65b-dc3d-4755-b7b0-3d4dc8feed9f"
-					(reference "C22")
+					(reference "C24")
 					(unit 1)
 				)
@@
 		(in_pos_files yes)
 		(dnp no)
-		(property "Reference" "R12"
+		(property "Reference" "R16"
 			(at 237.236 37.846 0)
 			(show_name no)
@@
 			(project "TVS-Adapter-v1"
 				(path "/3c9fa76f-2b37-4666-8575-58caa65def04/958ef65b-dc3d-4755-b7b0-3d4dc8feed9f"
-					(reference "R12")
+					(reference "R16")
 					(unit 1)
 				)
@@
 		(in_pos_files yes)
 		(dnp no)
-		(property "Reference" "C16"
+		(property "Reference" "C18"
 			(at 149.606 50.546 0)
 			(show_name no)
@@
 			(project "TVS-Adapter-v1"
 				(path "/3c9fa76f-2b37-4666-8575-58caa65def04/958ef65b-dc3d-4755-b7b0-3d4dc8feed9f"
-					(reference "C16")
+					(reference "C18")
 					(unit 1)
 				)
@@
 		(dnp no)
 		(fields_autoplaced yes)
-		(property "Reference" "D9"
+		(property "Reference" "D10"
 			(at 318.77 143.5099 90)
 			(show_name no)
@@
 			(project "TVS-Adapter-v1"
 				(path "/3c9fa76f-2b37-4666-8575-58caa65def04/958ef65b-dc3d-4755-b7b0-3d4dc8feed9f"
-					(reference "D9")
+					(reference "D10")
 					(unit 1)
 				)
@@
 		(in_pos_files yes)
 		(dnp no)
-		(property "Reference" "C17"
+		(property "Reference" "C19"
 			(at 161.036 50.546 0)
 			(show_name no)
@@
 			(project "TVS-Adapter-v1"
 				(path "/3c9fa76f-2b37-4666-8575-58caa65def04/958ef65b-dc3d-4755-b7b0-3d4dc8feed9f"
-					(reference "C17")
+					(reference "C19")
 					(unit 1)
 				)
@@
 		(in_pos_files yes)
 		(dnp no)
-		(property "Reference" "R11"
+		(property "Reference" "R15"
 			(at 160.528 170.18 0)
 			(show_name no)
@@
 			(project "TVS-Adapter-v1"
 				(path "/3c9fa76f-2b37-4666-8575-58caa65def04/958ef65b-dc3d-4755-b7b0-3d4dc8feed9f"
-					(reference "R11")
+					(reference "R15")
 					(unit 1)
 				)
@@
 		(in_pos_files yes)
 		(dnp no)
-		(property "Reference" "C25"
+		(property "Reference" "C27"
 			(at 167.132 101.854 0)
 			(show_name no)
@@
 			(project "TVS-Adapter-v1"
 				(path "/3c9fa76f-2b37-4666-8575-58caa65def04/958ef65b-dc3d-4755-b7b0-3d4dc8feed9f"
-					(reference "C25")
+					(reference "C27")
 					(unit 1)
 				)
@@
 		(in_pos_files yes)
 		(dnp no)
-		(property "Reference" "R9"
+		(property "Reference" "R11"
 			(at 205.486 41.656 0)
 			(show_name no)
@@
 			(project "TVS-Adapter-v1"
 				(path "/3c9fa76f-2b37-4666-8575-58caa65def04/958ef65b-dc3d-4755-b7b0-3d4dc8feed9f"
-					(reference "R9")
+					(reference "R11")
 					(unit 1)
 				)
@@
 		(in_pos_files yes)
 		(dnp no)
-		(property "Reference" "C30"
+		(property "Reference" "C32"
 			(at 203.2 57.658 0)
 			(show_name no)
@@
 			(project "TVS-Adapter-v1"
 				(path "/3c9fa76f-2b37-4666-8575-58caa65def04/958ef65b-dc3d-4755-b7b0-3d4dc8feed9f"
-					(reference "C30")
+					(reference "C32")
 					(unit 1)
 				)
@@
 		(in_pos_files yes)
 		(dnp no)
-		(property "Reference" "C21"
+		(property "Reference" "C23"
 			(at 138.43 214.63 90)
 			(show_name no)
@@
 			(project "TVS-Adapter-v1"
 				(path "/3c9fa76f-2b37-4666-8575-58caa65def04/958ef65b-dc3d-4755-b7b0-3d4dc8feed9f"
-					(reference "C21")
+					(reference "C23")
 					(unit 1)
 				)
@@
 		(in_pos_files yes)
 		(dnp no)
-		(property "Reference" "C34"
+		(property "Reference" "C36"
 			(at 148.59 214.63 90)
 			(show_name no)
@@
 			(project "TVS-Adapter-v1"
 				(path "/3c9fa76f-2b37-4666-8575-58caa65def04/958ef65b-dc3d-4755-b7b0-3d4dc8feed9f"
-					(reference "C34")
+					(reference "C36")
 					(unit 1)
 				)
@@
 		(in_pos_files yes)
 		(dnp no)
-		(property "Reference" "R2"
+		(property "Reference" "R4"
 			(at 214.63 195.58 90)
 			(show_name no)
@@
 			(project "TVS-Adapter-v1"
 				(path "/3c9fa76f-2b37-4666-8575-58caa65def04/958ef65b-dc3d-4755-b7b0-3d4dc8feed9f"
-					(reference "R2")
+					(reference "R4")
 					(unit 1)
 				)
@@
 		(in_pos_files yes)
 		(dnp no)
-		(property "Reference" "C48"
+		(property "Reference" "C50"
 			(at 256.54 141.2239 0)
 			(show_name no)
@@
 			(project "TVS-Adapter-v1"
 				(path "/3c9fa76f-2b37-4666-8575-58caa65def04/958ef65b-dc3d-4755-b7b0-3d4dc8feed9f"
-					(reference "C48")
+					(reference "C50")
 					(unit 1)
 				)
@@
 		(in_pos_files yes)
 		(dnp no)
-		(property "Reference" "D10"
+		(property "Reference" "D7"
 			(at 218.44 43.1799 90)
 			(show_name no)
@@
 			(project "TVS-Adapter-v1"
 				(path "/3c9fa76f-2b37-4666-8575-58caa65def04/958ef65b-dc3d-4755-b7b0-3d4dc8feed9f"
-					(reference "D10")
+					(reference "D7")
 					(unit 1)
 				)
@@
 		(in_pos_files yes)
 		(dnp no)
-		(property "Reference" "C53"
+		(property "Reference" "C56"
 			(at 269.24 115.8239 0)
 			(show_name no)
@@
 			(project "TVS-Adapter-v1"
 				(path "/3c9fa76f-2b37-4666-8575-58caa65def04/958ef65b-dc3d-4755-b7b0-3d4dc8feed9f"
-					(reference "C53")
+					(reference "C56")
 					(unit 1)
 				)

Commit message: Updating open collector output circuit of USB console, flash controller
Signed-off-by: Scott Berman <sgberman1@gmail.com>
Parts:
- renumbered R11 to R13, R15 to R17, R16 to R18
Changed lines of the file:
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@@
 	(title_block
 		(title "The Vision System Adapter")
-		(date "2026-10-14")
+		(date "2026-10-17")
 		(rev "1")
 		(company "SPACE COOKIES FRC TEAM 1868")
@@
 		(in_pos_files yes)
 		(dnp no)
-		(property "Reference" "R16"
+		(property "Reference" "R18"
 			(at 237.236 37.846 0)
 			(show_name no)
@@
 			(project "TVS-Adapter-v1"
 				(path "/3c9fa76f-2b37-4666-8575-58caa65def04/958ef65b-dc3d-4755-b7b0-3d4dc8feed9f"
-					(reference "R16")
+					(reference "R18")
 					(unit 1)
 				)
@@
 		(in_pos_files yes)
 		(dnp no)
-		(property "Reference" "R15"
+		(property "Reference" "R17"
 			(at 160.528 170.18 0)
 			(show_name no)
@@
 			(project "TVS-Adapter-v1"
 				(path "/3c9fa76f-2b37-4666-8575-58caa65def04/958ef65b-dc3d-4755-b7b0-3d4dc8feed9f"
-					(reference "R15")
+					(reference "R17")
 					(unit 1)
 				)
@@
 		(in_pos_files yes)
 		(dnp no)
-		(property "Reference" "R11"
+		(property "Reference" "R13"
 			(at 205.486 41.656 0)
 			(show_name no)
@@
 			(project "TVS-Adapter-v1"
 				(path "/3c9fa76f-2b37-4666-8575-58caa65def04/958ef65b-dc3d-4755-b7b0-3d4dc8feed9f"
-					(reference "R11")
+					(reference "R13")
 					(unit 1)
 				)

Commit message: Updates from Claude review
Signed-off-by: Scott Berman <scott.berman@bluerivertech.com>
Parts:
- removed D7: BAV199LT1G, Package_TO_SOT_SMD:SOT-23, symbol Diode:BAV99
- added D7: BAT54KFILM, NX-J401-Adapter:D_SOD-523, symbol NX-J401-Adapter:B260A-13-F
Connections:
- net 3V3: now also D7.1 (K)
- net at C32.1, Q9.1 (B), R13.2: now also D7.2 (A)

Commit message: Fixed most issues from review pass 4
Signed-off-by: scottb <sgberman1@gmail.com>
Parts:
- removed J8: SWD, NX-J401-Adapter:PinHeader_1x05_P2.54mm_Horizontal, symbol NX-J401-Adapter:Conn_01x05
- added C65: 22uF-10%-16V-0805, NX-J401-Adapter:C_0805_2012Metric, symbol NX-J401-Adapter:C_US
- added J12: SWD, Connector_PinHeader_2.54mm:PinHeader_1x06_P2.54mm_Horizontal, symbol Connector_Generic:Conn_01x06
Connections:
- net 3V3: now also C65.1, J12.6 (Pin_6)
- net BOOT0: now also J12.5 (Pin_5)
- net GND_CAN: now also C65.2, J12.1 (Pin_1)
- net NRST: now also J12.2 (Pin_2)
- net SWCLK: now also J12.4 (Pin_4)
- net SWDIO: now also J12.3 (Pin_3)
Other:
- note removed: "3V3_CAN delays bringing CAN RX (BOOT0) high until NPN turns on. ~10sec."
Changed lines of the file:
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@@
 		(company "SPACE COOKIES FRC TEAM 1868")
 	)
-	(text "3V3_CAN delays bringing CAN RX (BOOT0)\nhigh until NPN turns on. ~10sec."
+	(text "Reverse Polarity Protection"
 		(exclude_from_sim no)
-		(at 285.75 48.26 0)
+		(at 76.454 30.988 0)
 		(effects
 			(font
 				(size 1.27 1.27)
 			)
-			(justify left)
 		)
 	)
-	(text "Reverse Polarity Protection"
+	(text_box "NOTES:\n- CANABLE circuit interfaces with the M.2 Key-E adapter plugged into the J401.  Input power must be no greater than 3.6V\n- 3V3_CAN delays bringing CAN RX (BOOT0)\nhigh until NPN turns on. ~10sec."
 		(exclude_from_sim no)
-		(at 76.454 30.988 0)
+		(at 306.07 27.94 0)
+		(size 52.07 19.05)
+		(margins 0.9525 0.9525 0.9525 0.9525)
+		(stroke
+			(width 0)
+			(type solid)
+		)
+		(fill
+			(type color)
+			(color 0 0 0 0.1019607843)
+		)
 		(effects
 			(font
 				(size 1.27 1.27)
 			)
+			(justify left top)
 		)
 	)
@@
 	)
 	(junction
+		(at 154.94 200.66)
+		(diameter 0)
+		(color 0 0 0 0)
+	)
+	(junction
 		(at 160.02 40.64)
 		(diameter 0)
@@
 		(color 0 0 0 0)
 	)
+	(junction
+		(at 154.94 232.41)
+		(diameter 0)
+		(color 0 0 0 0)
+	)
 	(no_connect
 		(at 152.4 166.37)
@@
 	(wire
 		(pts
-			(xy 311.15 173.99) (xy 312.42 173.99)
+			(xy 311.15 171.45) (xy 312.42 171.45)
 		)
 		(stroke
@@
 	(wire
 		(pts
+			(xy 154.94 200.66) (xy 165.1 200.66)
+		)
+		(stroke
+			(width 0)
+			(type default)
+		)
+	)
+	(wire
+		(pts
 			(xy 166.37 90.17) (xy 154.94 90.17)
 		)
@@
 	(wire
 		(pts
+			(xy 165.1 200.66) (xy 165.1 210.82)
+		)
+		(stroke
+			(width 0)
+			(type default)
+		)
+	)
+	(wire
+		(pts
 			(xy 95.25 68.58) (xy 130.81 68.58)
 		)
@@
 	(wire
 		(pts
+			(xy 165.1 218.44) (xy 165.1 232.41)
+		)
+		(stroke
+			(width 0)
+			(type default)
+		)
+	)
+	(wire
+		(pts
 			(xy 213.36 53.34) (xy 238.76 53.34)
 		)
@@
 	(wire
 		(pts
+			(xy 311.15 173.99) (xy 312.42 173.99)
+		)
+		(stroke
+			(width 0)
+			(type default)
+		)
+	)
+	(wire
+		(pts
 			(xy 124.46 200.66) (xy 124.46 210.82)
 		)
@@
 	(wire
 		(pts
+			(xy 165.1 232.41) (xy 154.94 232.41)
+		)
+		(stroke
+			(width 0)
+			(type default)
+		)
+	)
+	(wire
+		(pts
 			(xy 283.21 107.95) (xy 283.21 123.19)
 		)
@@
 	)
 	(label "GND_CAN"
-		(at 311.15 173.99 180)
+		(at 311.15 171.45 180)
 		(effects
 			(font
@@
 		)
 	)
+	(label "NRST"
+		(at 311.15 173.99 180)
+		(effects
+			(font
+				(size 1.27 1.27)
+			)
+			(justify right bottom)
+		)
+	)
 	(label "SWDIO"
 		(at 104.14 138.43 180)
@@
 	)
 	(symbol
+		(lib_id "NX-J401-Adapter:C_US")
+		(at 165.1 214.63 0)
+		(unit 1)
+		(body_style 1)
+		(exclude_from_sim no)
+		(in_bom yes)
+		(on_board yes)
+		(in_pos_files yes)
+		(dnp no)
+		(property "Reference" "C65"
+			(at 168.91 214.63 90)
+			(show_name no)
+			(do_not_autoplace no)
+			(effects
+				(font
+					(size 1.27 1.27)
+				)
+			)
+		)
+		(property "Value" "22uF-10%-16V-0805"
+			(at 161.544 214.884 90)
+			(show_name no)
+			(do_not_autoplace no)
+			(effects
+				(font
+					(size 1.27 1.27)
+				)
+			)
+		)
+		(property "Footprint" "NX-J401-Adapter:C_0805_2012Metric"
+			(at 165.1 214.63 0)
+			(hide yes)
+			(show_name no)
+			(do_not_autoplace no)
+			(effects
+				(font
+					(size 1.27 1.27)
+				)
+			)
+		)
+		(property "Datasheet" ""
+			(at 165.1 214.63 0)
+			(hide yes)
+			(show_name no)
+			(do_not_autoplace no)
+			(effects
+				(font
+					(size 1.27 1.27)
+				)
+			)
+		)
+		(property "Description" "16V 22uF X5R ±10% 0805 Multilayer Ceramic Capacitors MLCC - SMD/SMT ROHS"
+			(at 165.1 214.63 0)
+			(hide yes)
+			(show_name no)
+			(do_not_autoplace no)
+			(effects
+				(font
+					(size 1.27 1.27)
+				)
+			)
+		)
+		(property "MFG" "Samsung Electro-Mechanics"
+			(at 165.1 214.63 0)
+			(hide yes)
+			(show_name no)
+			(do_not_autoplace no)
+			(effects
+				(font
+					(size 1.27 1.27)
+				)
+			)
+		)
+		(property "MFG P/N" "CL21A226KOQNNNE"
+			(at 165.1 214.63 0)
+			(hide yes)
+			(show_name no)
+			(do_not_autoplace no)
+			(effects
+				(font
+					(size 1.27 1.27)
+				)
+			)
+		)
+		(property "JLCPCB P/N" "C296720"
+			(at 165.1 214.63 0)
+			(hide yes)
+			(show_name no)
+			(do_not_autoplace no)
+			(effects
+				(font
+					(size 1.27 1.27)
+				)
+			)
+		)
+		(property "KiLib_Generator" "SMD_2terminal_chip_molded"
+			(at 165.1 214.63 0)
+			(hide yes)
+			(show_name no)
+			(do_not_autoplace no)
+			(effects
+				(font
+					(size 1.27 1.27)
+				)
+			)
+		)
+		(pin "1"
+		)
+		(pin "2"
+		)
+		(instances
+			(project "TVS-Adapter-v1"
+				(path "/3c9fa76f-2b37-4666-8575-58caa65def04/958ef65b-dc3d-4755-b7b0-3d4dc8feed9f"
+					(reference "C65")
+					(unit 1)
+				)
+			)
+		)
+	)
+	(symbol
 		(lib_id "NX-J401-Adapter:PESD1CAN")
 		(at 318.77 142.24 270)
@@
 	)
 	(symbol
-		(lib_id "NX-J401-Adapter:Conn_01x05")
-		(at 317.5 179.07 0)
+		(lib_id "Connector_Generic:Conn_01x06")
+		(at 317.5 176.53 0)
 		(unit 1)
 		(body_style 1)
@@
 		(in_pos_files yes)
 		(dnp no)
-		(property "Reference" "J8"
-			(at 320.04 177.7999 0)
+		(property "Reference" "J12"
+			(at 320.04 176.5299 0)
 			(show_name no)
 			(do_not_autoplace no)
@@
 		)
 		(property "Value" "SWD"
-			(at 320.04 180.3399 0)
+			(at 320.04 179.0699 0)
 			(show_name no)
 			(do_not_autoplace no)
@@
 			)
 		)
-		(property "Footprint" "NX-J401-Adapter:PinHeader_1x05_P2.54mm_Horizontal"
-			(at 317.5 179.07 0)
+		(property "Footprint" "Connector_PinHeader_2.54mm:PinHeader_1x06_P2.54mm_Horizontal"
+			(at 317.5 176.53 0)
 			(hide yes)
 			(show_name no)
@@
 		)
 		(property "Datasheet" ""
-			(at 317.5 179.07 0)
+			(at 317.5 176.53 0)
 			(hide yes)
 			(show_name no)
@@
 			)
 		)
-		(property "Description" "Generic connector, single row, 01x05, script generated (kicad-library-utils/schlib/autogen/connector/)"
-			(at 317.5 179.07 0)
+		(property "Description" "Generic connector, single row, 01x06, script generated (kicad-library-utils/schlib/autogen/connector/)"
+			(at 317.5 176.53 0)
 			(hide yes)
 			(show_name no)
@@
 		)
 		(property "MFG" "Adam Tech"
-			(at 320.294 186.182 0)
+			(at 327.66 185.42 0)
 			(show_name no)
 			(do_not_autoplace no)
@@
 					(size 1.27 1.27)
 				)
-				(justify left)
 			)
 		)
-		(property "MFG P/N" "PH1RB-05-UA"
-			(at 320.294 183.896 0)
+		(property "MFG P/N" "PH1RB-06-UA"
+			(at 327.66 182.88 0)
 			(show_name no)
 			(do_not_autoplace no)
@@
 					(size 1.27 1.27)
 				)
-				(justify left)
 			)
 		)
 		(property "DIST" "Digikey"
-			(at 317.5 179.07 0)
+			(at 317.5 176.53 0)
 			(hide yes)
 			(show_name no)
@@
 			)
 		)
-		(property "DIST P/N" "2057-PH1RB-05-UA-ND"
-			(at 317.5 179.07 0)
+		(property "DIST P/N" "2057-PH1RB-06-UA-ND"
+			(at 317.5 176.53 0)
 			(hide yes)
 			(show_name no)
@@
 		)
 		(property "JLCPCB P/N" "XXXXXX"
-			(at 317.5 179.07 0)
-			(hide yes)
-			(show_name no)
-			(do_not_autoplace no)
-			(effects
-				(font
-					(size 1.27 1.27)
-				)
-			)
-		)
-		(property "KiLib_Generator" "connector/pin_header_socket"
-			(at 317.5 179.07 0)
+			(at 317.5 176.53 0)
 			(hide yes)
 			(show_name no)
@@
 			)
 		)
-		(pin "2"
+		(pin "6"
 		)
 		(pin "1"
@@
 		(pin "3"
 		)
+		(pin "2"
+		)
 		(instances
 			(project "TVS-Adapter-v1"
 				(path "/3c9fa76f-2b37-4666-8575-58caa65def04/958ef65b-dc3d-4755-b7b0-3d4dc8feed9f"
-					(reference "J8")
+					(reference "J12")
 					(unit 1)
 				)
