File: circuit-boards/TVS-Adapter-v1/usb-serial.kicad_sch (KiCad schematic)
At the start: 15 parts, among them J11 USB_C_Receptacle_USB2.0_14P, U5 ISO6721BDR, U6 FT232RNL

Commit message: Add reset and recovery control.  PCB incomplete WIP
Signed-off-by: scott <scott@scott-Z590I-AORUS-ULTRA.bb>
Parts:
- removed C38, C41: 0.1uF-50V-10%-0603, NX-J401-Adapter:C_0603_1608Metric, symbol NX-J401-Adapter:C_US
- removed U5: ISO6721BDR, NX-J401-Adapter:SOIC-8_3.9x4.9mm_P1.27mm, symbol NX-J401-Adapter:ISO6721BDR
- added C60, C63, C64, C65: 0.1uF-50V-10%-0603, NX-J401-Adapter:C_0603_1608Metric, symbol NX-J401-Adapter:C_US
- added Q10, Q11, Q12, Q13: BSS123LT1G, Package_TO_SOT_SMD:SOT-23, symbol Transistor_FET:BSS123
- added R23, R31: 0R-1%-0603, NX-J401-Adapter:R_0603_1608Metric, symbol NX-J401-Adapter:R_US
- added R29, R30, R32, R33: 5.1k-1%-0603, NX-J401-Adapter:R_0603_1608Metric, symbol NX-J401-Adapter:R_US
- added U10: ISO6741DWR, Package_SO:SOIC-16W_7.5x10.3mm_P1.27mm, symbol Isolator:ISO6741
- added U12, U13: SN74LVC1G86DBVR, Package_TO_SOT_SMD:SOT-23-5, symbol 74xGxx:74LVC1G86
Connections:
- net 3V3: now also C60.1, R29.2, R30.2, U10.10 (EN2), U10.16 (V_{CC2})
- net 3V3_USB: now also C63.1, C64.1, C65.1, R32.2, R33.2, U10.1 (V_{CC1}), U10.7 (EN1), U12.5 (VCC), U13.5 (VCC)
- net GND1: now also C60.2, Q10.2 (S), Q11.2 (S), Q12.2 (S), Q13.2 (S), U10.15 (GND2), U10.9 (GND2)
- net GND_USB: now also C63.2, C64.2, C65.2, R23.1, R31.1, U10.2 (GND1), U10.8 (GND1), U12.3 (GND), U13.3 (GND)
- net RXD: now also U10.11 (IND)
- net TXD: now also U10.12 (OUTC)
- net at U6.1 (TXD): now also U10.5 (INC)
- net at U6.2 (~{DTR}): now also U13.1
- net at U6.3 (~{RTS}): now also U12.1
- net at U6.5 (RXD): now also U10.6 (OUTD)
- new net: R31.2, R33.1, U13.2
- new net: Q10.1 (G), U10.13 (OUTB)
- new net: Q12.1 (G), U10.14 (OUTA)
- new net: U10.3 (INA), U12.4
- new net: U10.4 (INB), U13.4
- new net: Q10.3 (D), Q11.1 (G), R29.1
- new net: Q12.3 (D), Q13.1 (G), R30.1
- new net: R23.2, R32.1, U12.2
- new net ~{FORCE_RECOVERY}: Q13.3 (D)
- new net ~{RESET}: Q11.3 (D)
- no-connect marks 16 -> 14
Other:
- moved on the sheet: C42, C46, C47, C51, C55, C56, C57, J11, L3, R24, R25, U6

Commit message: Add reset and recovery control from FT232
Signed-off-by: Scott Berman <sgberman1@gmail.com>
Parts:
- removed C64, C65: 0.1uF-50V-10%-0603, NX-J401-Adapter:C_0603_1608Metric, symbol NX-J401-Adapter:C_US
- removed Q10, Q11, Q12: BSS123LT1G, Package_TO_SOT_SMD:SOT-23, symbol Transistor_FET:BSS123
- removed R32, R33: 5.1k-1%-0603, NX-J401-Adapter:R_0603_1608Metric, symbol NX-J401-Adapter:R_US
- removed U12, U13: SN74LVC1G86DBVR, Package_TO_SOT_SMD:SOT-23-5, symbol 74xGxx:74LVC1G86
- added Q14, Q15, Q16: BSS138, Package_TO_SOT_SMD:SOT-23, symbol Transistor_FET:BSS123
- Q13: value BSS123LT1G -> BSS138; JLCPCB P/N C78755 -> C52895; MFG P/N BSS123LT1G -> BSS138
Connections:
- net GND1: now also Q14.2 (S), Q15.2 (S), Q16.2 (S)
- net GND_USB: no longer R23.1, R31.1
- net ~{FORCE_RECOVERY}: now also R23.2; no longer Q13.3 (D)
- net ~{RESET}: now also R31.2
- net at U10.13 (OUTB): now also Q15.1 (G)
- net at U10.14 (OUTA): now also Q14.1 (G)
- net at U10.3 (INA): now also U6.13 (CBUS2)
- net at U10.4 (INB): now also U6.14 (CBUS3)
- net at R29.1: now also Q15.3 (D), Q16.1 (G)
- net at Q13.1 (G), R30.1: now also Q14.3 (D)
- new net: Q16.3 (D), R31.1
- new net: Q13.3 (D), R23.1
Other:
- title: The Vision System Adapter -> TVS Adapter
- moved on the sheet: C42, C46, C47, C51, C55, C56, C57, C60, C63, J11, L3, Q13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

Commit message: Add pullups to reset-recovery outputs
Signed-off-by: Scott Berman <sgberman1@gmail.com>
Parts:
- added R32, R33: 5.1k-1%-0603, NX-J401-Adapter:R_0603_1608Metric, symbol NX-J401-Adapter:R_US
Connections:
- net 3V3_USB: now also R32.2, R33.2
- net at U10.3 (INA), U6.13 (CBUS2): now also R32.1
- net at U10.4 (INB), U6.14 (CBUS3): now also R33.1
Other:
- title: TVS Adapter -> The Vision System Adapter

Commit message: Update with cleaned up silk and fab drawings
Signed-off-by: Scott Berman <sgberman1@gmail.com>
Parts:
- R1: renamed from R23; footprint NX-J401-Adapter:R_0603_1608Metric -> Resistor_SMD:R_0603_1608Metric_Pad0.98x0.95mm_HandSolder
- R2: renamed from R31; footprint NX-J401-Adapter:R_0603_1608Metric -> Resistor_SMD:R_0603_1608Metric_Pad0.98x0.95mm_HandSolder
- renumbered C60 to C38, C63 to C43, C42 to C44, C46 to C48, C47 to C49, C57 to C51, C51 to C54, C55 to C58, C56 to C59, Q13 to Q3, Q16 to Q4, Q14 to Q6, Q15 to Q7, R30 to R12, R29 to R13, R33 to R30, R32 to R31, R24 to R32, R25 to R33, U10 to U5
Changed lines of the file:
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@@
 		(in_pos_files yes)
 		(dnp yes)
-		(property "Reference" "R31"
+		(property "Reference" "R2"
 			(at 364.49 127 90)
 			(show_name no)
@@
 			)
 		)
-		(property "Footprint" "NX-J401-Adapter:R_0603_1608Metric"
+		(property "Footprint" "Resistor_SMD:R_0603_1608Metric_Pad0.98x0.95mm_HandSolder"
 			(at 367.284 129.286 90)
 			(hide yes)
@@
 			(project "TVS-Adapter-v1"
 				(path "/3c9fa76f-2b37-4666-8575-58caa65def04/7f338915-7b6e-40c1-9733-742b14680646"
-					(reference "R31")
+					(reference "R2")
 					(unit 1)
 				)
@@
 		(in_pos_files yes)
 		(dnp no)
-		(property "Reference" "R25"
+		(property "Reference" "R33"
 			(at 89.408 156.21 90)
 			(show_name no)
@@
 			(project "TVS-Adapter-v1"
 				(path "/3c9fa76f-2b37-4666-8575-58caa65def04/7f338915-7b6e-40c1-9733-742b14680646"
-					(reference "R25")
+					(reference "R33")
 					(unit 1)
 				)
@@
 		(in_pos_files yes)
 		(dnp no)
-		(property "Reference" "C46"
+		(property "Reference" "C48"
 			(at 157.48 125.9839 0)
 			(show_name no)
@@
 			(project "TVS-Adapter-v1"
 				(path "/3c9fa76f-2b37-4666-8575-58caa65def04/7f338915-7b6e-40c1-9733-742b14680646"
-					(reference "C46")
+					(reference "C48")
 					(unit 1)
 				)
@@
 		(in_pos_files yes)
 		(dnp no)
-		(property "Reference" "U10"
+		(property "Reference" "U5"
 			(at 279.4 135.89 0)
 			(show_name no)
@@
 			(project "TVS-Adapter-v1"
 				(path "/3c9fa76f-2b37-4666-8575-58caa65def04/7f338915-7b6e-40c1-9733-742b14680646"
-					(reference "U10")
+					(reference "U5")
 					(unit 1)
 				)
@@
 		(in_pos_files yes)
 		(dnp no)
-		(property "Reference" "Q14"
+		(property "Reference" "Q6"
 			(at 322.58 111.76 0)
 			(show_name no)
@@
 			(project "TVS-Adapter-v1"
 				(path "/3c9fa76f-2b37-4666-8575-58caa65def04/7f338915-7b6e-40c1-9733-742b14680646"
-					(reference "Q14")
+					(reference "Q6")
 					(unit 1)
 				)
@@
 		(in_pos_files yes)
 		(dnp no)
-		(property "Reference" "C42"
+		(property "Reference" "C44"
 			(at 93.218 129.032 90)
 			(show_name no)
@@
 			(project "TVS-Adapter-v1"
 				(path "/3c9fa76f-2b37-4666-8575-58caa65def04/7f338915-7b6e-40c1-9733-742b14680646"
-					(reference "C42")
+					(reference "C44")
 					(unit 1)
 				)
@@
 		(in_pos_files yes)
 		(dnp no)
-		(property "Reference" "Q13"
+		(property "Reference" "Q3"
 			(at 350.52 111.76 0)
 			(show_name no)
@@
 			(project "TVS-Adapter-v1"
 				(path "/3c9fa76f-2b37-4666-8575-58caa65def04/7f338915-7b6e-40c1-9733-742b14680646"
-					(reference "Q13")
+					(reference "Q3")
 					(unit 1)
 				)
@@
 		(in_pos_files yes)
 		(dnp yes)
-		(property "Reference" "R23"
+		(property "Reference" "R1"
 			(at 364.49 106.68 90)
 			(show_name no)
@@
 			)
 		)
-		(property "Footprint" "NX-J401-Adapter:R_0603_1608Metric"
+		(property "Footprint" "Resistor_SMD:R_0603_1608Metric_Pad0.98x0.95mm_HandSolder"
 			(at 367.284 108.966 90)
 			(hide yes)
@@
 			(project "TVS-Adapter-v1"
 				(path "/3c9fa76f-2b37-4666-8575-58caa65def04/7f338915-7b6e-40c1-9733-742b14680646"
-					(reference "R23")
+					(reference "R1")
 					(unit 1)
 				)
@@
 		(in_pos_files yes)
 		(dnp no)
-		(property "Reference" "C56"
+		(property "Reference" "C59"
 			(at 115.316 186.69 0)
 			(show_name no)
@@
 			(project "TVS-Adapter-v1"
 				(path "/3c9fa76f-2b37-4666-8575-58caa65def04/7f338915-7b6e-40c1-9733-742b14680646"
-					(reference "C56")
+					(reference "C59")
 					(unit 1)
 				)
@@
 		(in_pos_files yes)
 		(dnp no)
-		(property "Reference" "C63"
+		(property "Reference" "C43"
 			(at 254 123.4439 0)
 			(show_name no)
@@
 			(project "TVS-Adapter-v1"
 				(path "/3c9fa76f-2b37-4666-8575-58caa65def04/7f338915-7b6e-40c1-9733-742b14680646"
-					(reference "C63")
+					(reference "C43")
 					(unit 1)
 				)
@@
 		(in_pos_files yes)
 		(dnp no)
-		(property "Reference" "C47"
+		(property "Reference" "C49"
 			(at 130.556 128.016 0)
 			(show_name no)
@@
 			(project "TVS-Adapter-v1"
 				(path "/3c9fa76f-2b37-4666-8575-58caa65def04/7f338915-7b6e-40c1-9733-742b14680646"
-					(reference "C47")
+					(reference "C49")
 					(unit 1)
 				)
@@
 		(in_pos_files yes)
 		(dnp no)
-		(property "Reference" "C51"
+		(property "Reference" "C54"
 			(at 151.13 188.2139 0)
 			(show_name no)
@@
 			(project "TVS-Adapter-v1"
 				(path "/3c9fa76f-2b37-4666-8575-58caa65def04/7f338915-7b6e-40c1-9733-742b14680646"
-					(reference "C51")
+					(reference "C54")
 					(unit 1)
 				)
@@
 		(in_pos_files yes)
 		(dnp no)
-		(property "Reference" "Q16"
+		(property "Reference" "Q4"
 			(at 350.52 132.08 0)
 			(show_name no)
@@
 			(project "TVS-Adapter-v1"
 				(path "/3c9fa76f-2b37-4666-8575-58caa65def04/7f338915-7b6e-40c1-9733-742b14680646"
-					(reference "Q16")
+					(reference "Q4")
 					(unit 1)
 				)
@@
 		(in_pos_files yes)
 		(dnp no)
-		(property "Reference" "C55"
+		(property "Reference" "C58"
 			(at 105.156 186.69 0)
 			(show_name no)
@@
 			(project "TVS-Adapter-v1"
 				(path "/3c9fa76f-2b37-4666-8575-58caa65def04/7f338915-7b6e-40c1-9733-742b14680646"
-					(reference "C55")
+					(reference "C58")
 					(unit 1)
 				)
@@
 		(in_pos_files yes)
 		(dnp no)
-		(property "Reference" "R24"
+		(property "Reference" "R32"
 			(at 89.408 149.86 90)
 			(show_name no)
@@
 			(project "TVS-Adapter-v1"
 				(path "/3c9fa76f-2b37-4666-8575-58caa65def04/7f338915-7b6e-40c1-9733-742b14680646"
-					(reference "R24")
+					(reference "R32")
 					(unit 1)
 				)
@@
 		(in_pos_files yes)
 		(dnp no)
-		(property "Reference" "C57"
+		(property "Reference" "C51"
 			(at 143.51 124.46 0)
 			(show_name no)
@@
 			(project "TVS-Adapter-v1"
 				(path "/3c9fa76f-2b37-4666-8575-58caa65def04/7f338915-7b6e-40c1-9733-742b14680646"
-					(reference "C57")
+					(reference "C51")
 					(unit 1)
 				)
@@
 		(in_pos_files yes)
 		(dnp no)
-		(property "Reference" "R29"
+		(property "Reference" "R13"
 			(at 335.28 100.33 0)
 			(show_name no)
@@
 			(project "TVS-Adapter-v1"
 				(path "/3c9fa76f-2b37-4666-8575-58caa65def04/7f338915-7b6e-40c1-9733-742b14680646"
-					(reference "R29")
+					(reference "R13")
 					(unit 1)
 				)
@@
 		(in_pos_files yes)
 		(dnp no)
-		(property "Reference" "R32"
+		(property "Reference" "R31"
 			(at 214.63 129.54 0)
 			(show_name no)
@@
 			(project "TVS-Adapter-v1"
 				(path "/3c9fa76f-2b37-4666-8575-58caa65def04/7f338915-7b6e-40c1-9733-742b14680646"
-					(reference "R32")
+					(reference "R31")
 					(unit 1)
 				)
@@
 		(in_pos_files yes)
 		(dnp no)
-		(property "Reference" "R30"
+		(property "Reference" "R12"
 			(at 325.12 100.33 0)
 			(show_name no)
@@
 			(project "TVS-Adapter-v1"
 				(path "/3c9fa76f-2b37-4666-8575-58caa65def04/7f338915-7b6e-40c1-9733-742b14680646"
-					(reference "R30")
+					(reference "R12")
 					(unit 1)
 				)
@@
 		(in_pos_files yes)
 		(dnp no)
-		(property "Reference" "Q15"
+		(property "Reference" "Q7"
 			(at 321.31 132.08 0)
 			(show_name no)
@@
 			(project "TVS-Adapter-v1"
 				(path "/3c9fa76f-2b37-4666-8575-58caa65def04/7f338915-7b6e-40c1-9733-742b14680646"
-					(reference "Q15")
+					(reference "Q7")
 					(unit 1)
 				)
@@
 		(in_pos_files yes)
 		(dnp no)
-		(property "Reference" "C60"
+		(property "Reference" "C38"
 			(at 283.21 123.4439 0)
 			(show_name no)
@@
 			(project "TVS-Adapter-v1"
 				(path "/3c9fa76f-2b37-4666-8575-58caa65def04/7f338915-7b6e-40c1-9733-742b14680646"
-					(reference "C60")
+					(reference "C38")
 					(unit 1)
 				)
@@
 		(in_pos_files yes)
 		(dnp no)
-		(property "Reference" "R33"
+		(property "Reference" "R30"
 			(at 222.758 129.794 0)
 			(show_name no)
@@
 			(project "TVS-Adapter-v1"
 				(path "/3c9fa76f-2b37-4666-8575-58caa65def04/7f338915-7b6e-40c1-9733-742b14680646"
-					(reference "R33")
+					(reference "R30")
 					(unit 1)
 				)

Commit message: Updating open collector output circuit of USB console, flash controller
Signed-off-by: Scott Berman <sgberman1@gmail.com>
Parts:
- removed Q3, Q4, Q6, Q7: BSS138, Package_TO_SOT_SMD:SOT-23, symbol Transistor_FET:BSS123
- removed R12, R13: 5.1k-1%-0603, NX-J401-Adapter:R_0603_1608Metric, symbol NX-J401-Adapter:R_US
- added Q3, Q6: SS8050, NX-J401-Adapter:SOT-23, symbol NX-J401-Adapter:SS8050
- added Q4, Q7: SI2301CDS-T1-GE3, NX-J401-Adapter:SOT-23, symbol NX-J401-Adapter:Si2319CDS
- added R14, R7: 13K-1%-0603, NX-J401-Adapter:R_0603_1608Metric, symbol NX-J401-Adapter:R_US
- added R15, R8: 2K-1%-0603, NX-J401-Adapter:R_0603_1608Metric, symbol NX-J401-Adapter:R_US
- U5: JLCPCB P/N ISO6741DWR -> C5216432
- renumbered C48 to C45, R30 to R32, R31 to R33, R32 to R34, R33 to R35
Connections:
- net 3V3: now also Q4.2 (S), Q7.2 (S)
- net GND1: now also Q3.2 (E), Q6.2 (E), R14.1, R7.1
- net at R2.1: now also Q3.3 (C)
- net at U5.13 (OUTB): now also Q4.1 (G)
- net at U5.14 (OUTA): now also Q7.1 (G)
- net at R1.1: now also Q6.3 (C)
- new net: Q3.1 (B), R8.1
- new net: Q4.3 (D), R7.2, R8.2
- new net: Q7.3 (D), R14.2, R15.2
- new net: Q6.1 (B), R15.1
Other:
- moved on the sheet: R1, R2

Commit message: Updates from Claude review
Signed-off-by: Scott Berman <scott.berman@bluerivertech.com>
Parts:
- Q3, Q4, Q6, Q7: DIST (none) -> Digkey; DIST P/N (none) -> 1727-3817-1-ND
- U5: KiLib_Generator (none) -> package/gullwing
Other:
- note added: "NOTE: Program CBUS2 and CBUS3 to CBitBangI/O with FT_PROG or ftdi_eeprom before installing R1/R2."
- moved on the sheet: C38, C43, U5

Commit message: Fixed most issues from review pass 4
Signed-off-by: scottb <sgberman1@gmail.com>
Parts:
- removed Q3, Q6: SS8050, NX-J401-Adapter:SOT-23, symbol NX-J401-Adapter:SS8050
- removed Q4, Q7: SI2301CDS-T1-GE3, NX-J401-Adapter:SOT-23, symbol NX-J401-Adapter:Si2319CDS
- removed R14, R7: 13K-1%-0603, NX-J401-Adapter:R_0603_1608Metric, symbol NX-J401-Adapter:R_US
- removed R15, R8: 2K-1%-0603, NX-J401-Adapter:R_0603_1608Metric, symbol NX-J401-Adapter:R_US
- added C60, C61: 1uF-50V-10%-0603, NX-J401-Adapter:C_0603_1608Metric, symbol NX-J401-Adapter:C_US
- added C62, C63, C64: 0.1uF-50V-10%-0603, NX-J401-Adapter:C_0603_1608Metric, symbol NX-J401-Adapter:C_US
- added Q14: SS8050, NX-J401-Adapter:SOT-23, symbol NX-J401-Adapter:SS8050
- added R36, R37, R38: 5.1k-1%-0603, NX-J401-Adapter:R_0603_1608Metric, symbol NX-J401-Adapter:R_US
- added U10, U11, U12: SN74LVC1G125DBVR, Package_TO_SOT_SMD:SOT-23-5, symbol 74xGxx:SN74LVC1G125DBV
- added U9: TLV70233DBVR, Package_TO_SOT_SMD:SOT-23-5, symbol Regulator_Linear:TLV70233_SOT23-5
- U6: JLCPCB P/N C8690 -> C5246810
Connections:
- net 3V3: now also C60.1, C62.1, C63.1, C64.1, R36.2, U10.5 (VCC), U11.5 (VCC), U12.5 (VCC), U9.5 (OUT)
- net GND1: now also C60.2, C61.2, C62.2, C63.2, C64.2, Q14.2 (E), R37.1, U10.2, U10.3 (GND), U11.2, U11.3 (GND), U12.3 (GND), U9.2 (GND)
- net TXD: now also U12.4; no longer U5.12 (OUTC)
- net at R2.1: now also U11.4
- net at U5.13 (OUTB): now also U11.1
- net at U5.14 (OUTA): now also U10.1
- net at R1.1: now also U10.4
- new net: U12.2, U5.12 (OUTC)
- new net: Q14.3 (C), R36.1, U12.1
- new net: Q14.1 (B), R38.2
- new net +5V J401: C61.1, U9.1 (IN), U9.3 (EN)
- new net 3V3 J401: R37.2, R38.1
Other:
- moved on the sheet: R1, R2
